Commit message: Changed left_arm by la_arm and right_arm by ra_arm Changed l_ by lh_ and r_ by rh_ to follow shadow naming

File: agni_description/flobi/flobi-eye.urdf.xacro (robot description, xacro)
@@ -10,5 +10,5 @@
 	<!-- prefix -->
   <macro name="flobi-eye" params="prefix name parent *origin">
-     <joint name="${prefix}floby_eyes_${name}_lr_joint" type="revolute">
+     <joint name="${prefix}flobi_eyes_${name}_lr_joint" type="revolute">
       <insert_block name="origin" />
       <axis xyz="0 0 -1"/>
@@ -27,5 +27,5 @@
       </inertial>
     </link>
-     <joint name="${prefix}floby_eyes_${name}_ud_joint" type="revolute">
+     <joint name="${prefix}flobi_eyes_${name}_ud_joint" type="revolute">
       <origin xyz="0 0 ${flobi_elem_eyes_z_offset}" rpy="0 0 0"/>
       <axis xyz="0 -1 0"/>

File: agni_description/flobi/flobiv2.urdf.xacro (robot description, xacro)
@@ -11,5 +11,5 @@
 		<property name="flobi_elem_eye_mass" value="0.2"/>
 		<link name="flobi_base_link" />
-		<joint name="floby_base_joint" type="fixed">
+		<joint name="flobi_base_joint" type="fixed">
       <origin xyz="0 0 0.0" rpy="0 0 0"/>
       <parent link="flobi_base_link"/>
@@ -38,5 +38,5 @@
       </collision>
     </link>
-    <joint name="floby_neck_pan_joint" type="revolute">
+    <joint name="flobi_neck_pan_joint" type="revolute">
       <origin xyz="0 0 0.10" rpy="0 0 0"/>
       <axis xyz="0 0 1"/>
@@ -55,5 +55,5 @@
       </inertial>
     </link>
-    <joint name="floby_neck_tilt_joint" type="revolute">
+    <joint name="flobi_neck_tilt_joint" type="revolute">
       <origin xyz="0 0 0.0" rpy="0 0 0"/>
       <axis xyz="0 1 0"/>
@@ -72,5 +72,5 @@
       </inertial>
     </link>
-    <joint name="floby_neck_roll_joint" type="revolute">
+    <joint name="flobi_neck_roll_joint" type="revolute">
       <origin xyz="0 0 0.0" rpy="0 0 0"/>
       <axis xyz="1 0 0"/>
@@ -103,5 +103,5 @@
       </collision>
     </link>
-     <joint name="floby_eyes_left_lr_joint" type="revolute">
+     <joint name="flobi_eyes_left_lr_joint" type="revolute">
       <origin xyz="0.072 0.0337 0.055" rpy="0 0 0"/>
       <axis xyz="0 0 1"/>
@@ -120,5 +120,5 @@
       </inertial>
     </link>
-     <joint name="floby_eyes_left_ud_joint" type="revolute">
+     <joint name="flobi_eyes_left_ud_joint" type="revolute">
       <origin xyz="0 0 0.0" rpy="0 0 0"/>
       <axis xyz="0 1 0"/>
@@ -151,5 +151,5 @@
       </collision>
     </link>
-    <joint name="floby_eyes_right_lr_joint" type="revolute">
+    <joint name="flobi_eyes_right_lr_joint" type="revolute">
       <origin xyz="0.072 -0.0337 0.055" rpy="0 0 0"/>
       <axis xyz="0 0 1"/>
@@ -168,5 +168,5 @@
       </inertial>
     </link>
-     <joint name="floby_eye_right_ud_joint" type="revolute">
+     <joint name="flobi_eye_right_ud_joint" type="revolute">
       <origin xyz="0 0 0.0" rpy="0 0 0"/>
       <axis xyz="0 1 0"/>

File: agni_description/flobi/flobiv3.urdf.xacro (robot description, xacro)
@@ -11,5 +11,5 @@
 	<!-- if neutral is 0 then gender is considered, 0 for male, 1 for female -->
   <macro name="flobi" params="prefix neutral gender parent *origin">
-		<joint name="${prefix}floby_base_joint" type="fixed">
+		<joint name="${prefix}flobi_base_joint" type="fixed">
       <insert_block name="origin" />
       <parent link="${parent}"/>
@@ -38,5 +38,5 @@
     </link>
      -->
-    <joint name="${prefix}floby_neck_pan_joint" type="revolute">
+    <joint name="${prefix}flobi_neck_pan_joint" type="revolute">
       <origin xyz="0 0 0.0" rpy="0 0 0"/>
       <axis xyz="0 0 -1"/>
@@ -55,5 +55,5 @@
       </inertial>
     </link>
-    <joint name="${prefix}floby_neck_tilt_joint" type="revolute">
+    <joint name="${prefix}flobi_neck_tilt_joint" type="revolute">
       <origin xyz="0 0 ${flobi_elem_neck_beam_length}" rpy="0 0 0"/>
       <axis xyz="0 -1 0"/>
@@ -72,5 +72,5 @@
       </inertial>
     </link>
-    <joint name="${prefix}floby_neck_roll_joint" type="revolute">
+    <joint name="${prefix}flobi_neck_roll_joint" type="revolute">
       <origin xyz="0 0 ${flobi_elem_neck_tilt_length}" rpy="0 0 0"/>
       <axis xyz="1 0 0"/>

File: agni_description/kuka/lwr_controllers.gazebo.xacro (robot description, xacro)
@@ -12,11 +12,11 @@
 				<baseLink>left_arm_base_link</baseLink>
 				<toolLink>left_arm_hand_mount</toolLink>
-				<left_arm_0_joint>0.0</left_arm_0_joint>
-				<left_arm_1_joint>0</left_arm_1_joint>
-				<left_arm_2_joint>0.0</left_arm_2_joint>
-				<left_arm_3_joint>0</left_arm_3_joint>
-				<left_arm_4_joint>0</left_arm_4_joint>
-				<left_arm_5_joint>0</left_arm_5_joint>
-				<left_arm_6_joint>0</left_arm_6_joint>
+				<la_arm_0_joint>0.0</la_arm_0_joint>
+				<la_arm_1_joint>0</la_arm_1_joint>
+				<la_arm_2_joint>0.0</la_arm_2_joint>
+				<la_arm_3_joint>0</la_arm_3_joint>
+				<la_arm_4_joint>0</la_arm_4_joint>
+				<la_arm_5_joint>0</la_arm_5_joint>
+				<la_arm_6_joint>0</la_arm_6_joint>
 			</plugin>
 		</gazebo>
@@ -33,11 +33,11 @@
 				<baseLink>right_arm_base_link</baseLink>
 				<toolLink>right_arm_hand_mount</toolLink>
-				<right_arm_0_joint>0.0</right_arm_0_joint>
-				<right_arm_1_joint>0</right_arm_1_joint>
-				<right_arm_2_joint>0.0</right_arm_2_joint>
-				<right_arm_3_joint>0</right_arm_3_joint>
-				<right_arm_4_joint>0</right_arm_4_joint>
-				<right_arm_5_joint>0</right_arm_5_joint>
-				<right_arm_6_joint>0</right_arm_6_joint>
+				<ra_arm_0_joint>0.0</ra_arm_0_joint>
+				<ra_arm_1_joint>0</ra_arm_1_joint>
+				<ra_arm_2_joint>0.0</ra_arm_2_joint>
+				<ra_arm_3_joint>0</ra_arm_3_joint>
+				<ra_arm_4_joint>0</ra_arm_4_joint>
+				<ra_arm_5_joint>0</ra_arm_5_joint>
+				<ra_arm_6_joint>0</ra_arm_6_joint>
 			</plugin>
 		</gazebo>

File: agni_description/robots/la_kuka_gazebo.urdf.xacro (robot description, xacro)
@@ -5,5 +5,5 @@
   <xacro:include filename="$(find agni_description)/kuka/lwr_controllers.gazebo.xacro"/>
   <!-- KUKA arm -->
-  <xacro:kuka_lwr_arm name="left_" reflect="-1" tool_name=""/>
+  <xacro:kuka_lwr_arm name="la_" reflect="-1" tool_name=""/>
   <xacro:left_lwr_arm_gazebo_controller namespace="la" port="49938"/>
 </robot>

File: agni_description/robots/la_pa10_gazebo.urdf.xacro (robot description, xacro)
@@ -5,5 +5,5 @@
   <xacro:include filename="$(find agni_description)/pa10/pa10_shadow_controller_manager.xacro"/>
   <!-- PA10 arm -->
-  <xacro:pa10a_arm name="left_"/>
+  <xacro:pa10a_arm name="la_"/>
   <!-- pa10 controllers HERE
   <xacro:pa10_gazebo_controller_manager namespace="ra"/> ros-hydro-gazebo-ros-control missing-->

File: agni_description/robots/left_kuka_shadow.urdf.xacro (robot description, xacro)
@@ -13,9 +13,9 @@
   <xacro:macro name="leftkukashadow" params="parent *origin prefix controller">
     <!-- KUKA arm -->
-    <xacro:kuka_lwr_arm name="left_" reflect="-1" tool_name=""/>
-    <joint name="left_frame_placement" type="fixed">
+    <xacro:kuka_lwr_arm name="la_" reflect="-1" tool_name=""/>
+    <joint name="la_frame_placement" type="fixed">
        <insert_block name="origin" />
       <parent link="${parent}"/>
-      <child link="left_arm_base_link"/>
+      <child link="la_arm_base_link"/>
     </joint>
     <xacro:if value="${controller}">
@@ -26,9 +26,9 @@
     <xacro:if value="${prefix}">
       <!-- Shadow Hands -->
-      <xacro:shadowhand muscletrans="false" muscle="false" bio="false" ubi="true" eli="false" reflect="-1.0" prefix="l_"  />
+      <xacro:shadowhand muscletrans="false" muscle="false" bio="false" ubi="true" eli="false" reflect="-1.0" prefix="lh_"  />
       <!-- Link arm and hand -->
-      <joint name="left_arm_hand_mount" type="fixed">
-        <parent link="left_arm_hand_mount"/>
-        <child link="l_forearm"/>
+      <joint name="la_arm_hand_mount" type="fixed">
+        <parent link="la_arm_hand_mount"/>
+        <child link="lh_forearm"/>
         <origin xyz="0 0 0.0151" rpy="0 0 0" />
       </joint>
@@ -38,6 +38,6 @@
       <!-- Shadow Hands -->
       <!-- Link arm and hand -->
-      <joint name="left_arm_hand_mount" type="fixed">
-        <parent link="left_arm_hand_mount"/>
+      <joint name="la_arm_hand_mount" type="fixed">
+        <parent link="la_arm_hand_mount"/>
         <child link="forearm"/>
         <origin xyz="0 0 0.0151" rpy="0 0 0" />

File: agni_description/robots/left_pa10_shadow.urdf.xacro (robot description, xacro)
@@ -13,9 +13,9 @@
   <xacro:macro name="leftpa10shadow" params="parent *origin prefix controller">
     <!-- KUKA arm -->
-    <xacro:pa10a_arm name="left_"/>
-    <joint name="left_frame_placement" type="fixed">
+    <xacro:pa10a_arm name="la_"/>
+    <joint name="la_frame_placement" type="fixed">
        <insert_block name="origin" />
       <parent link="${parent}"/>
-      <child link="left_arm_base_link"/>
+      <child link="la_arm_base_link"/>
     </joint>
     <xacro:if value="${controller}">
@@ -28,9 +28,9 @@
     <xacro:if value="${prefix}">
       <!-- Shadow Hands -->
-      <xacro:shadowhand muscletrans="false" muscle="false" bio="false" ubi="true" eli="false" reflect="-1.0" prefix="l_"  />
+      <xacro:shadowhand muscletrans="false" muscle="false" bio="false" ubi="true" eli="false" reflect="-1.0" prefix="lh_"  />
       <!-- Link arm and hand -->
-      <joint name="left_arm_hand_mount" type="fixed">
-        <parent link="left_arm_hand_mount"/>
-        <child link="l_forearm"/>
+      <joint name="la_arm_hand_mount" type="fixed">
+        <parent link="la_arm_hand_mount"/>
+        <child link="lh_forearm"/>
         <origin xyz="0 0 0.0151" rpy="0 0 1.5707" />
       </joint>
@@ -40,6 +40,6 @@
       <!-- Shadow Hands -->
       <!-- Link arm and hand -->
-      <joint name="left_arm_hand_mount" type="fixed">
-        <parent link="left_arm_hand_mount"/>
+      <joint name="la_arm_hand_mount" type="fixed">
+        <parent link="la_arm_hand_mount"/>
         <child link="forearm"/>
         <origin xyz="0 0 0.0151" rpy="0 0 1.5707" />

File: agni_description/robots/pa10_right.urdf.xacro (robot description, xacro)
@@ -6,8 +6,8 @@
   <xacro:include filename="$(find sr_description)/hand/xacro/full_hand_muscle.urdf.xacro" />
   <!-- arms -->
-  <xacro:pa10_arm name="right_"/>
+  <xacro:pa10_arm name="ra_"/>
   <!-- Shadow Hands -->
-  <joint name="right_arm_hand_mount" type="fixed">
-    <parent link="right_arm_7_link"/>
+  <joint name="ra_arm_hand_mount" type="fixed">
+    <parent link="ra_arm_7_link"/>
     <child link="forearm"/>
     <origin xyz="0 0 0" rpy="0 0 0" />

File: agni_description/robots/ra_kuka_gazebo.urdf.xacro (robot description, xacro)
@@ -5,5 +5,5 @@
   <xacro:include filename="$(find agni_description)/kuka/lwr_controllers.gazebo.xacro"/>
   <!-- KUKA arm -->
-  <xacro:kuka_lwr_arm name="right_" reflect="1" tool_name=""/>
+  <xacro:kuka_lwr_arm name="ra_" reflect="1" tool_name=""/>
   <xacro:right_lwr_arm_gazebo_controller namespace="ra" port="49940"/>
 </robot>

File: agni_description/robots/ra_pa10_gazebo.urdf.xacro (robot description, xacro)
@@ -5,5 +5,5 @@
   <xacro:include filename="$(find agni_description)/pa10/pa10_shadow_controller_manager.xacro"/>
   <!-- PA10 arm -->
-  <xacro:pa10c_arm name="right_"/>
+  <xacro:pa10c_arm name="ra_"/>
   <!-- pa10 controllers HERE
   <xacro:pa10_gazebo_controller_manager namespace="ra"/> ros-hydro-gazebo-ros-control missing-->

File: agni_description/robots/right_kuka_shadow.urdf.xacro (robot description, xacro)
@@ -13,22 +13,22 @@
   <xacro:macro name="rightkukashadow" params="parent *origin prefix controller">
     <!-- KUKA arm -->
-    <xacro:kuka_lwr_arm name="right_" reflect="1" tool_name=""/>
-    <joint name="right_frame_placement" type="fixed">
+    <xacro:kuka_lwr_arm name="ra_" reflect="1" tool_name=""/>
+    <joint name="ra_frame_placement" type="fixed">
        <insert_block name="origin" />
       <parent link="${parent}"/>
-      <child link="right_arm_base_link"/>
+      <child link="ra_arm_base_link"/>
     </joint>
     <xacro:if value="${controller}">
-    <!-- add controllers -->
-    <xacro:right_lwr_arm_gazebo_controller namespace="ra" port="49940"/>
+      <!-- add controllers -->
+      <xacro:right_lwr_arm_gazebo_controller namespace="ra" port="49940"/>
       <xacro:shadow_gazebo_controller_manager namespace="rh" />
     </xacro:if>
     <xacro:if value="${prefix}">
       <!-- Shadow Hands -->
-      <xacro:shadowhand muscletrans="false" muscle="false" bio="false" ubi="true" eli="false" reflect="1.0" prefix="r_"  />
+      <xacro:shadowhand muscletrans="false" muscle="false" bio="false" ubi="true" eli="false" reflect="1.0" prefix="rh_"  />
       <!-- Link arm and hand -->
-      <joint name="right_arm_hand_mount" type="fixed">
-        <parent link="right_arm_hand_mount"/>
-        <child link="r_forearm"/>
+      <joint name="ra_arm_hand_mount" type="fixed">
+        <parent link="ra_arm_hand_mount"/>
+        <child link="rh_forearm"/>
         <origin xyz="0 0 0.0151" rpy="0 0 0" />
       </joint>
@@ -38,6 +38,6 @@
       <!-- Shadow Hands -->
       <!-- Link arm and hand -->
-      <joint name="right_arm_hand_mount" type="fixed">
-        <parent link="right_arm_hand_mount"/>
+      <joint name="ra_arm_hand_mount" type="fixed">
+        <parent link="ra_arm_hand_mount"/>
         <child link="forearm"/>
         <origin xyz="0 0 0.0151" rpy="0 0 0" />

File: agni_description/robots/right_pa10_shadow.urdf.xacro (robot description, xacro)
@@ -13,9 +13,9 @@
   <xacro:macro name="rightpa10shadow" params="parent *origin prefix controller">
     <!-- KUKA arm -->
-    <xacro:pa10c_arm name="right_"/>
-    <joint name="right_frame_placement" type="fixed">
+    <xacro:pa10c_arm name="ra_"/>
+    <joint name="ra_frame_placement" type="fixed">
        <insert_block name="origin" />
       <parent link="${parent}"/>
-      <child link="right_arm_base_link"/>
+      <child link="ra_arm_base_link"/>
     </joint>
     <xacro:if value="${controller}">
@@ -28,9 +28,9 @@
     <xacro:if value="${prefix}">
       <!-- Shadow Hands -->
-      <xacro:shadowhand muscletrans="false" muscle="false" bio="false" ubi="true" eli="false" reflect="1.0" prefix="r_"  />
+      <xacro:shadowhand muscletrans="false" muscle="false" bio="false" ubi="true" eli="false" reflect="1.0" prefix="rh_"  />
       <!-- Link arm and hand -->
-      <joint name="right_arm_hand_mount" type="fixed">
-        <parent link="right_arm_hand_mount"/>
-        <child link="r_forearm"/>
+      <joint name="ra_arm_hand_mount" type="fixed">
+        <parent link="ra_arm_hand_mount"/>
+        <child link="rh_forearm"/>
         <origin xyz="0 0 0.0151" rpy="0 0 1.5707" />
       </joint>
@@ -40,6 +40,6 @@
       <!-- Shadow Hands -->
       <!-- Link arm and hand -->
-      <joint name="right_arm_hand_mount" type="fixed">
-        <parent link="right_arm_hand_mount"/>
+      <joint name="ra_arm_hand_mount" type="fixed">
+        <parent link="ra_arm_hand_mount"/>
         <child link="forearm"/>
         <origin xyz="0 0 0.0151" rpy="0 0 1.5707" />
