Commit message: Added controllers in pa10 (shadow version due to prob in ros_control) Added args to set the gazebo default arm posture (not working yet) Fixed pa10a urdf (forearm rotated 180 deg)

File: agni_description/robots/la_pa10_gazebo.urdf.xacro (robot description, xacro)
@@ -3,7 +3,9 @@
 		 xmlns:xacro="http://www.ros.org/wiki/xacro">
   <xacro:include filename="$(find agni_description)/pa10/pa10-a.urdf.xacro"/>
-  <!-- <xacro:include filename="$(find agni_description)/pa10/lwr_controllers.gazebo.xacro"/> -->
+  <xacro:include filename="$(find agni_description)/pa10/pa10_shadow_controller_manager.xacro"/>
   <!-- PA10 arm -->
-  <xacro:pa10_arm name="left_"/>
-  <!-- pa10 controllers HERE -->
+  <xacro:pa10a_arm name="left_"/>
+  <!-- pa10 controllers HERE
+  <xacro:pa10_gazebo_controller_manager namespace="ra"/> ros-hydro-gazebo-ros-control missing-->
+  <xacro:pa10_shadow_gazebo_controller_manager namespace="la"/>
 </robot>

File: agni_description/robots/left_pa10_shadow.urdf.xacro (robot description, xacro)
@@ -3,5 +3,5 @@
      xmlns:xacro="http://www.ros.org/wiki/xacro">
   <xacro:include filename="$(find agni_description)/pa10/pa10-a.urdf.xacro"/>
-  <!-- <xacro:include filename="$(find agni_description)/pa10/lwr_controllers.gazebo.xacro"/> -->
+  <xacro:include filename="$(find agni_description)/pa10/pa10_shadow_controller_manager.xacro"/>
   <xacro:include filename="$(find agni_description)/urdf/sr_gazebo.urdf.xacro" />
   <xacro:include filename="$(find sr_description)/hand/xacro/full_hand.urdf.xacro" />
@@ -21,19 +21,21 @@
     <xacro:if value="${controller}">
     <!-- add controllers -->
-       <!-- pa10 controllers HERE -->
+      <!-- pa10 controllers HERE
+      <xacro:pa10_gazebo_controller_manager namespace="ra"/> ros-hydro-gazebo-ros-control missing-->
+      <xacro:pa10_shadow_gazebo_controller_manager namespace="la"/>
       <xacro:shadow_gazebo_controller_manager namespace="lh" />
     </xacro:if>
     <xacro:if value="${prefix}">
       <!-- Shadow Hands -->
-      <xacro:shadowhand muscletrans="false" muscle="false" bio="false" ubi="true" eli="false" reflect="1.0" prefix="l_"  />
+      <xacro:shadowhand muscletrans="false" muscle="false" bio="false" ubi="true" eli="false" reflect="-1.0" prefix="l_"  />
       <!-- Link arm and hand -->
       <joint name="left_arm_hand_mount" type="fixed">
         <parent link="left_arm_hand_mount"/>
         <child link="l_forearm"/>
-        <origin xyz="0 0 0.0151" rpy="0 0 0" />
+        <origin xyz="0 0 0.0151" rpy="0 0 1.5707" />
       </joint>
     </xacro:if>
     <xacro:unless value="${prefix}">
-      <xacro:shadowhand muscletrans="false" muscle="false" bio="false" ubi="true" eli="false" reflect="1.0" prefix=""  />
+      <xacro:shadowhand muscletrans="false" muscle="false" bio="false" ubi="true" eli="false" reflect="-1.0" prefix=""  />
       <!-- Shadow Hands -->
       <!-- Link arm and hand -->
@@ -41,5 +43,5 @@
         <parent link="left_arm_hand_mount"/>
         <child link="forearm"/>
-        <origin xyz="0 0 0.0151" rpy="0 0 0" />
+        <origin xyz="0 0 0.0151" rpy="0 0 1.5707" />
       </joint>
     </xacro:unless>

File: agni_description/robots/ra_pa10_gazebo.urdf.xacro (robot description, xacro)
@@ -3,7 +3,9 @@
 		 xmlns:xacro="http://www.ros.org/wiki/xacro">
   <xacro:include filename="$(find agni_description)/pa10/pa10-c.urdf.xacro"/>
-  <!-- <xacro:include filename="$(find agni_description)/pa10/lwr_controllers.gazebo.xacro"/> -->
+  <xacro:include filename="$(find agni_description)/pa10/pa10_shadow_controller_manager.xacro"/>
   <!-- PA10 arm -->
-  <xacro:pa10_arm name="right_"/>
-  <!-- pa10 controllers HERE -->
+  <xacro:pa10c_arm name="right_"/>
+  <!-- pa10 controllers HERE
+  <xacro:pa10_gazebo_controller_manager namespace="ra"/> ros-hydro-gazebo-ros-control missing-->
+  <xacro:pa10_shadow_gazebo_controller_manager namespace="ra"/>
 </robot>

File: agni_description/robots/right_pa10_shadow.urdf.xacro (robot description, xacro)
@@ -3,5 +3,5 @@
      xmlns:xacro="http://www.ros.org/wiki/xacro">
   <xacro:include filename="$(find agni_description)/pa10/pa10-c.urdf.xacro"/>
-  <!-- <xacro:include filename="$(find agni_description)/pa10/lwr_controllers.gazebo.xacro"/> -->
+  <xacro:include filename="$(find agni_description)/pa10/pa10_shadow_controller_manager.xacro"/>
   <xacro:include filename="$(find agni_description)/urdf/sr_gazebo.urdf.xacro" />
   <xacro:include filename="$(find sr_description)/hand/xacro/full_hand.urdf.xacro" />
@@ -21,6 +21,8 @@
     <xacro:if value="${controller}">
     <!-- add controllers -->
-       <!-- pa10 controllers HERE -->
       <xacro:shadow_gazebo_controller_manager namespace="rh" />
+      <!-- pa10 controllers HERE
+      <xacro:pa10_gazebo_controller_manager namespace="ra"/> ros-hydro-gazebo-ros-control missing-->
+      <xacro:pa10_shadow_gazebo_controller_manager namespace="ra"/>
     </xacro:if>
     <xacro:if value="${prefix}">
@@ -31,5 +33,5 @@
         <parent link="right_arm_hand_mount"/>
         <child link="r_forearm"/>
-        <origin xyz="0 0 0.0151" rpy="0 0 0" />
+        <origin xyz="0 0 0.0151" rpy="0 0 1.5707" />
       </joint>
     </xacro:if>
@@ -41,5 +43,5 @@
         <parent link="right_arm_hand_mount"/>
         <child link="forearm"/>
-        <origin xyz="0 0 0.0151" rpy="0 0 0" />
+        <origin xyz="0 0 0.0151" rpy="0 0 1.5707" />
       </joint>
     </xacro:unless>
