Commit message: Changed arm names prefix to la/ra Changed shape generator scale to 1.5

File: agni_description/robots/left_pa10_shadow.urdf.xacro (robot description, xacro)
@@ -13,9 +13,9 @@
   <xacro:macro name="leftpa10shadow" params="parent *origin prefix controller">
     <!-- KUKA arm -->
-    <xacro:pa10a_arm name="left_"/>
-    <joint name="left_frame_placement" type="fixed">
+    <xacro:pa10a_arm name="la_"/>
+    <joint name="la_frame_placement" type="fixed">
        <insert_block name="origin" />
       <parent link="${parent}"/>
-      <child link="left_arm_base_link"/>
+      <child link="la_arm_base_link"/>
     </joint>
     <xacro:if value="${controller}">
@@ -30,6 +30,6 @@
       <xacro:shadowhand muscletrans="false" muscle="false" bio="false" ubi="true" eli="false" reflect="-1.0" prefix="l_"  />
       <!-- Link arm and hand -->
-      <joint name="left_arm_hand_mount" type="fixed">
-        <parent link="left_arm_hand_mount"/>
+      <joint name="la_arm_hand_mount" type="fixed">
+        <parent link="la_arm_hand_mount"/>
         <child link="l_forearm"/>
         <origin xyz="0 0 0.0151" rpy="0 0 1.5707" />
@@ -40,6 +40,6 @@
       <!-- Shadow Hands -->
       <!-- Link arm and hand -->
-      <joint name="left_arm_hand_mount" type="fixed">
-        <parent link="left_arm_hand_mount"/>
+      <joint name="la_arm_hand_mount" type="fixed">
+        <parent link="la_arm_hand_mount"/>
         <child link="forearm"/>
         <origin xyz="0 0 0.0151" rpy="0 0 1.5707" />

File: agni_description/robots/right_pa10_shadow.urdf.xacro (robot description, xacro)
@@ -13,9 +13,9 @@
   <xacro:macro name="rightpa10shadow" params="parent *origin prefix controller">
     <!-- KUKA arm -->
-    <xacro:pa10c_arm name="right_"/>
-    <joint name="right_frame_placement" type="fixed">
+    <xacro:pa10c_arm name="ra_"/>
+    <joint name="ra_frame_placement" type="fixed">
        <insert_block name="origin" />
       <parent link="${parent}"/>
-      <child link="right_arm_base_link"/>
+      <child link="ra_arm_base_link"/>
     </joint>
     <xacro:if value="${controller}">
@@ -30,6 +30,6 @@
       <xacro:shadowhand muscletrans="false" muscle="false" bio="false" ubi="true" eli="false" reflect="1.0" prefix="r_"  />
       <!-- Link arm and hand -->
-      <joint name="right_arm_hand_mount" type="fixed">
-        <parent link="right_arm_hand_mount"/>
+      <joint name="ra_arm_hand_mount" type="fixed">
+        <parent link="ra_arm_hand_mount"/>
         <child link="r_forearm"/>
         <origin xyz="0 0 0.0151" rpy="0 0 1.5707" />
@@ -40,6 +40,6 @@
       <!-- Shadow Hands -->
       <!-- Link arm and hand -->
-      <joint name="right_arm_hand_mount" type="fixed">
-        <parent link="right_arm_hand_mount"/>
+      <joint name="ra_arm_hand_mount" type="fixed">
+        <parent link="ra_arm_hand_mount"/>
         <child link="forearm"/>
         <origin xyz="0 0 0.0151" rpy="0 0 1.5707" />
