Commit message: Migrated arm_and_hand to new generic loader Generic arm_hand_gazebo xacro generic Unified kuka_gazebo and pa10_gazebo xacros Fixed controller loading kuka_anytool (ports were incorrect) Fixed missing controllers in shadow_motor end-effector Fixed frame loading for spawner Clean-up of unnecessary files

File: agni_description/robots/kuka_anytool.urdf.xacro (robot description, xacro)
@@ -26,9 +26,14 @@
     <xacro:if value="${controller}">
       <!-- add controllers -->
-      <xacro:right_lwr_arm_gazebo_controller namespace="${prefix}a" port="49940"/>
+        <xacro:if value="${is_right}" >
+          <xacro:right_lwr_arm_gazebo_controller namespace="${prefix}a" port="49940"/>
+        </xacro:if>
+        <xacro:unless value="${is_right}" >
+          <xacro:left_lwr_arm_gazebo_controller namespace="${prefix}a" port="49938"/>
+        </xacro:unless>
     </xacro:if>
     <xacro:if value="${use_prefix}">
       <!-- Effector -->
-      <xacro:call macro="${ee_macro}" prefix="${prefix}h_"/>
+      <xacro:call macro="${ee_macro}" prefix="${prefix}" use_prefix="${use_prefix}"/>
       <!-- Link arm and effector -->
     <joint name="${prefix}a_arm_hand_mount" type="fixed">
@@ -40,5 +45,5 @@
     <xacro:unless value="${use_prefix}">
       <!-- Effector -->
-      <xacro:call macro="${ee_macro}" prefix=""/>
+      <xacro:call macro="${ee_macro}" prefix="" use_prefix="${use_prefix}"/>
     <!-- Link arm and hand -->
     <joint name="${prefix}a_arm_hand_mount" type="fixed">

File: agni_description/robots/left_myrmex_ee.urdf.xacro (robot description, xacro)
@@ -10,8 +10,8 @@
   <xacro:property name="l_ee_base_link" value="myrmex_quick_mount" />
   <xacro:macro name="right_myrmex" params="prefix" >
-    <xacro:myrmex_quick_mount prefix="${prefix}" />
+    <xacro:myrmex_quick_mount prefix="${prefix}h_" />
   </xacro:macro>
   <xacro:macro name="left_myrmex" params="prefix" >
-    <xacro:myrmex_quick_mount prefix="${prefix}" />
+    <xacro:myrmex_quick_mount prefix="${prefix}h_" />
   </xacro:macro>
 </robot>

File: agni_description/robots/left_poking_stick_ee.urdf.xacro (robot description, xacro)
@@ -10,8 +10,8 @@
   <xacro:property name="l_ee_base_link" value="poking_stick" />
   <xacro:macro name="right_poking_stick" params="prefix" >
-    <xacro:poking_stick prefix="${prefix}" />
+    <xacro:poking_stick prefix="${prefix}h_" />
   </xacro:macro>
   <xacro:macro name="left_poking_stick" params="prefix" >
-    <xacro:poking_stick prefix="${prefix}" />
+    <xacro:poking_stick prefix="${prefix}h_" />
   </xacro:macro>
 </robot>

File: agni_description/robots/pa10_anytool.urdf.xacro (robot description, xacro)
@@ -40,5 +40,5 @@
     <xacro:if value="${use_prefix}">
       <!-- Effector -->
-      <xacro:call macro="${ee_macro}" prefix="${prefix}h_"/>
+      <xacro:call macro="${ee_macro}" prefix="${prefix}" use_prefix="${use_prefix}"/>
       <!-- Link arm and effector -->
     <joint name="${prefix}a_arm_hand_mount" type="fixed">
@@ -50,5 +50,5 @@
     <xacro:unless value="${use_prefix}">
       <!-- Effector -->
-      <xacro:call macro="${ee_macro}" prefix=""/>
+      <xacro:call macro="${ee_macro}" prefix="" use_prefix="${use_prefix}"/>
     <!-- Link arm and hand -->
     <joint name="${prefix}a_arm_hand_mount" type="fixed">

File: agni_description/robots/right_myrmex_ee.urdf.xacro (robot description, xacro)
@@ -10,8 +10,8 @@
   <xacro:property name="r_ee_base_link" value="myrmex_quick_mount" />
   <xacro:macro name="right_myrmex" params="prefix" >
-    <xacro:myrmex_quick_mount prefix="${prefix}" />
+    <xacro:myrmex_quick_mount prefix="${prefix}h_" />
   </xacro:macro>
   <xacro:macro name="left_myrmex" params="prefix" >
-    <xacro:myrmex_quick_mount prefix="${prefix}" />
+    <xacro:myrmex_quick_mount prefix="${prefix}h_" />
   </xacro:macro>
 </robot>

File: agni_description/robots/right_poking_stick_ee.urdf.xacro (robot description, xacro)
@@ -10,8 +10,8 @@
   <xacro:property name="r_ee_base_link" value="poking_stick" />
   <xacro:macro name="right_poking_stick" params="prefix" >
-    <xacro:poking_stick prefix="${prefix}" />
+    <xacro:poking_stick prefix="${prefix}h_" />
   </xacro:macro>
   <xacro:macro name="left_poking_stick" params="prefix" >
-    <xacro:poking_stick prefix="${prefix}" />
+    <xacro:poking_stick prefix="${prefix}h_" />
   </xacro:macro>
 </robot>

File: agni_description/robots/shadowhands_ee.urdf.xacro (robot description, xacro)
@@ -4,9 +4,23 @@
   <xacro:include filename="$(find agni_description)/urdf/sr_gazebo.urdf.xacro" />
   <xacro:include filename="$(find sr_description)/hand/xacro/full_hand.urdf.xacro" />
-  <xacro:macro name="right_shadow_motor" params="prefix">
-    <xacro:shadowhand muscletrans="false" muscle="false" bio="false" ubi="$(arg USE_UBI)" eli="false" reflect="1.0" prefix="${prefix}"  />
+  <xacro:macro name="right_shadow_motor" params="prefix use_prefix" >
+    <xacro:if value="${use_prefix}">
+      <xacro:shadowhand muscletrans="false" muscle="false" bio="false" ubi="$(arg USE_UBI)" eli="false" reflect="1.0" prefix="${prefix}h_"  />
+      <xacro:shadow_gazebo_controller_manager namespace="${prefix}h" />
+    </xacro:if>
+    <xacro:unless value="${use_prefix}">
+      <xacro:shadowhand muscletrans="false" muscle="false" bio="false" ubi="$(arg USE_UBI)" eli="false" reflect="1.0" prefix=""  />
+      <xacro:shadow_gazebo_controller_manager namespace="" />
+    </xacro:unless>
   </xacro:macro>
-  <xacro:macro name="left_shadow_motor" params="prefix">
-    <xacro:shadowhand muscletrans="false" muscle="false" bio="false" ubi="$(arg USE_UBI)" eli="false" reflect="-1.0" prefix="${prefix}"  />
+  <xacro:macro name="left_shadow_motor" params="prefix use_prefix" >
+    <xacro:if value="${use_prefix}">
+      <xacro:shadowhand muscletrans="false" muscle="false" bio="false" ubi="$(arg USE_UBI)" eli="false" reflect="-1.0" prefix="${prefix}h_"  />
+      <xacro:shadow_gazebo_controller_manager namespace="${prefix}h" />
+    </xacro:if>
+    <xacro:unless value="${use_prefix}">
+      <xacro:shadowhand muscletrans="false" muscle="false" bio="false" ubi="$(arg USE_UBI)" eli="false" reflect="-1.0" prefix=""  />
+      <xacro:shadow_gazebo_controller_manager namespace="" />
+    </xacro:unless>
   </xacro:macro>
   <xacro:macro name="right_shadow_muscle" params="prefix">

File: agni_description/urdf/pa10_frame.urdf.xacro (robot description, xacro)
@@ -2,4 +2,6 @@
 <root xmlns:xacro="http://www.ros.org/wiki/xacro">
   <xacro:include filename="$(find agni_description)/urdf/frame.urdf.xacro"/>
+  <!-- arm calibration -->
+  <xacro:include filename="$(find agni_description)/calibration/pa10_cal.xml"/>
   <xacro:property name="cal_frame_thick"  value="0.09" />
   <xacro:property name="cal_frame_width"     value="1.92" />
