Commit message: Fixed missing orientation change on shadow_motor_ee

File: agni_description/robots/left_shadow_motor_ee.urdf.xacro (robot description, xacro)
@@ -8,5 +8,5 @@
   <xacro:property name="cal_left_ee_y" value="0.0" />
   <xacro:property name="cal_left_ee_z" value="0.0151" />
-  <xacro:property name="cal_left_ee_yaw" value="0.0" />
+  <xacro:property name="cal_left_ee_yaw" value="1.5707" />
   <xacro:property name="cal_left_ee_pitch" value="0.0" />
   <xacro:property name="cal_left_ee_roll" value="0.0" />

File: agni_description/robots/right_shadow_motor_ee.urdf.xacro (robot description, xacro)
@@ -8,5 +8,5 @@
   <xacro:property name="cal_right_ee_y" value="0.0" />
   <xacro:property name="cal_right_ee_z" value="0.0151" />
-  <xacro:property name="cal_right_ee_yaw" value="0.0" />
+  <xacro:property name="cal_right_ee_yaw" value="1.5707" />
   <xacro:property name="cal_right_ee_pitch" value="0.0" />
   <xacro:property name="cal_right_ee_roll" value="0.0" />
