Commit message: Fixed frame not visible, requires removing of ground plane (due to world frame at tabletop, table poles under ground) Fixed left arm seen even if L:=0

File: agni_description/robots/frame.urdf.xacro (robot description, xacro)
@@ -1,4 +1,4 @@
 <?xml version="1.0"?>
-<robot name="frame"
+<robot name="platform"
 		 xmlns:xacro="http://www.ros.org/wiki/xacro">
   <xacro:arg name="ARM" default="kuka"/>

File: agni_description/urdf/frame-half.urdf.xacro (robot description, xacro)
@@ -23,5 +23,11 @@
 </xacro:macro>
 <xacro:macro name="frame-half" params="prefix thickness width depth height tableHeight">
+  <link name="world"/>
   <link name="${prefix}_frame">
+    <inertial>
+      <mass value="100.0" />
+      <origin xyz="0 1.2 0.3" rpy="0 0 0"/>
+      <inertia ixx="4.0" ixy="0" ixz="0" iyy="4.0" iyz="0" izz="4.0"/>
+    </inertial>
    <!-- horizontal front bar-->
    <xacro:bar thickness="${thickness}" len="${width}">
@@ -138,6 +144,11 @@
   </link>
   <gazebo reference="${prefix}_frame">
-      <material value="kuka-lwr.material"/>
+      <material value="Gazebo/Grey"/>
   </gazebo>
+  <joint name="${prefix}_frame_joint" type="fixed">
+      <origin xyz="0 0 0" rpy="0 0 0"/>
+      <parent link="world"/>
+      <child link="${prefix}_frame"/>
+  </joint>
 </xacro:macro>
 </root>

File: agni_description/urdf/frame.urdf.xacro (robot description, xacro)
@@ -22,5 +22,11 @@
 </xacro:macro>
 <xacro:macro name="frame" params="prefix thickness width depth height tableHeight mountingYpos mountingspacing">
+  <link name="world"/>
   <link name="${prefix}_frame">
+     <inertial>
+      <mass value="100.0" />
+      <origin xyz="0 1.2 0.3" rpy="0 0 0"/>
+      <inertia ixx="4.0" ixy="0" ixz="0" iyy="4.0" iyz="0" izz="4.0"/>
+    </inertial>
 	 <!-- horizontal front bar-->
 	 <xacro:bar thickness="${thickness}" len="${width}">
@@ -140,4 +146,9 @@
     </collision>
   </link>
+  <joint name="${prefix}_frame_joint" type="fixed">
+      <origin xyz="0 0 0" rpy="0 0 0"/>
+      <parent link="world"/>
+      <child link="${prefix}_frame"/>
+  </joint>
 </xacro:macro>
 </root>
