Commit message: Switched arm.launch and dependencies to use new combined urdf description Re-added the ground plane in gazebo at a position lower than zero

File: agni_description/robots/arm_hand_gazebo.urdf.xacro (robot description, xacro)
@@ -4,4 +4,5 @@
   <xacro:arg name="IS_RIGHT" default="1"/>
   <xacro:arg name="USE_PREFIX" default="1"/>
+  <xacro:arg name="SIM" default="1"/>
   <!-- arm with end-effector -->
   <xacro:include filename="$(find agni_description)/robots/$(arg ARM)_anytool.urdf.xacro" />
@@ -10,5 +11,5 @@
   <!-- right end-effector -->
   <xacro:include filename="$(find agni_description)/robots/right_shadow_motor_ee.urdf.xacro" />
-  <!-- left enf-effector -->
+  <!-- left end-effector -->
   <xacro:include filename="$(find agni_description)/robots/left_shadow_motor_ee.urdf.xacro" />
    <!-- must be world to spawn the arm in gazebo and have it fixed at the calibration location -->
@@ -16,5 +17,5 @@
   <!-- arm and hand -->
   <xacro:if value="$(arg IS_RIGHT)" >
-    <xacro:arm_ee parent="world" arm="$(arg ARM)" prefix="r" is_right="1" ee_macro="right_shadow_motor" ee_base_link="forearm" use_prefix="$(arg USE_PREFIX)" controller="true">
+    <xacro:arm_ee parent="world" arm="$(arg ARM)" prefix="r" is_right="1" ee_macro="right_shadow_motor" ee_base_link="forearm" use_prefix="$(arg USE_PREFIX)" controller="$(arg SIM)">
       <origin xyz="${cal_right_arm_x} ${cal_right_arm_y} ${cal_right_arm_z}"
       rpy="${cal_right_arm_roll} ${cal_right_arm_pitch} ${cal_right_arm_yaw}"/>
@@ -24,5 +25,5 @@
   </xacro:if>
   <xacro:unless value="$(arg IS_RIGHT)" >
-    <xacro:arm_ee parent="world" arm="$(arg ARM)" prefix="l" is_right="0" ee_macro="left_shadow_motor" ee_base_link="forearm" use_prefix="$(arg USE_PREFIX)" controller="true">
+    <xacro:arm_ee parent="world" arm="$(arg ARM)" prefix="l" is_right="0" ee_macro="left_shadow_motor" ee_base_link="forearm" use_prefix="$(arg USE_PREFIX)" controller="$(arg SIM)">
       <origin xyz="${cal_left_arm_x} ${cal_left_arm_y} ${cal_left_arm_z}"
           rpy="${cal_left_arm_roll} ${cal_left_arm_pitch} ${cal_left_arm_yaw}"/>

File: agni_description/robots/kuka_gazebo.urdf.xacro (robot description, xacro)
@@ -1,24 +1,28 @@
 <?xml version="1.0"?>
-<robot name="$(arg namespace)_kuka"
+<robot name="$(arg namespace)a_kuka"
 		 xmlns:xacro="http://www.ros.org/wiki/xacro">
-  <xacro:arg name="namespace" default="r"/>
-  <xacro:arg name="is_right" default="1"/>
-  <xacro:arg name="gazebo" default="1"/>
   <xacro:include filename="$(find agni_description)/kuka/kuka.urdf.xacro"/>
   <xacro:include filename="$(find agni_description)/kuka/lwr_controllers.gazebo.xacro"/>
   <!-- KUKA arm -->
-  <xacro:if value="$(arg is_right)" >
-    <xacro:kuka_lwr_arm name="$(arg namespace)a_" reflect="1" tool_name=""/>
-    <xacro:if value="$(arg gazebo)">
+  <xacro:macro name="arm_noee" params="parent arm is_right prefix controller *origin">
+    <xacro:if value="${is_right}" >
+      <xacro:kuka_lwr_arm name="${prefix}a_" reflect="1" tool_name=""/>
+      <xacro:if value="${controller}">
        <!-- add controllers -->
-      <xacro:right_lwr_arm_gazebo_controller namespace="$(arg namespace)a" port="49940"/>
+      <xacro:right_lwr_arm_gazebo_controller namespace="${prefix}a" port="49938"/>
+      </xacro:if>
     </xacro:if>
-  </xacro:if>
-  <xacro:unless value="$(arg is_right)" >
-    <xacro:kuka_lwr_arm name="$(arg namespace)a_" reflect="-1" tool_name=""/>
-    <xacro:if value="$(arg gazebo)">
+    <xacro:unless value="${is_right}" >
+      <xacro:kuka_lwr_arm name="${prefix}a_" reflect="-1" tool_name=""/>
+      <xacro:if value="${controller}">
        <!-- add controllers -->
-      <xacro:left_lwr_arm_gazebo_controller namespace="$(arg namespace)a" port="49938"/>
-    </xacro:if>
-  </xacro:unless>
+      <xacro:left_lwr_arm_gazebo_controller namespace="${prefix}a" port="49940"/>
+      </xacro:if>
+    </xacro:unless>
+    <joint name="${prefix}a_frame_placement" type="fixed">
+      <insert_block name="origin" />
+      <parent link="${parent}"/>
+      <child link="${prefix}a_arm_base_link"/>
+    </joint>
+  </xacro:macro>
 </robot>

File: agni_description/robots/pa10_gazebo.urdf.xacro (robot description, xacro)
@@ -1,29 +1,33 @@
 <?xml version="1.0"?>
-<robot name="$(arg namespace)_pa10"
+<robot name="$(arg namespace)a_pa10"
 		 xmlns:xacro="http://www.ros.org/wiki/xacro">
-  <xacro:arg name="namespace" default="r"/>
-  <xacro:arg name="is_right" default="1"/>
-  <xacro:arg name="gazebo" default="1"/>
   <xacro:include filename="$(find agni_description)/pa10/pa10-a.urdf.xacro"/>
   <xacro:include filename="$(find agni_description)/pa10/pa10-c.urdf.xacro"/>
   <xacro:include filename="$(find agni_description)/pa10/pa10_shadow_controller_manager.xacro"/>
   <!-- PA10 arm -->
-  <xacro:if value="$(arg is_right)" >
-    <xacro:pa10c_arm name="$(arg namespace)a_" />
-    <xacro:if value="$(arg gazebo)">
-      <!-- add controllers -->
-      <!-- pa10 controllers HERE
-      <xacro:pa10_gazebo_controller_manager namespace="$(arg namespace)a"/> ros-hydro-gazebo-ros-control missing-->
-      <xacro:pa10_shadow_gazebo_controller_manager namespace="$(arg namespace)a"/>
+  <xacro:macro name="arm_noee" params="parent arm is_right prefix controller *origin">
+    <xacro:if value="${is_right}" >
+      <xacro:pa10c_arm name="${prefix}a_" />
+      <xacro:if value="${controller}">
+        <!-- add controllers -->
+        <!-- pa10 controllers HERE
+        <xacro:pa10_gazebo_controller_manager namespace="$(arg namespace)a"/> ros-hydro-gazebo-ros-control missing-->
+        <xacro:pa10_shadow_gazebo_controller_manager namespace="${prefix}a"/>
+      </xacro:if>
     </xacro:if>
-  </xacro:if>
-  <xacro:unless value="$(arg is_right)" >
-    <xacro:pa10a_arm name="$(arg namespace)a_" />
-    <xacro:if value="$(arg gazebo)">
-      <!-- add controllers -->
-      <!-- pa10 controllers HERE
-      <xacro:pa10_gazebo_controller_manager namespace="$(arg namespace)a"/> ros-hydro-gazebo-ros-control missing-->
-      <xacro:pa10_shadow_gazebo_controller_manager namespace="$(arg namespace)a"/>
-    </xacro:if>
-  </xacro:unless>
+    <xacro:unless value="${is_right}" >
+      <xacro:pa10a_arm name="${prefix}a_" />
+      <xacro:if value="${controller}">
+        <!-- add controllers -->
+        <!-- pa10 controllers HERE
+        <xacro:pa10_gazebo_controller_manager namespace="$(arg namespace)a"/> ros-hydro-gazebo-ros-control missing-->
+        <xacro:pa10_shadow_gazebo_controller_manager namespace="${prefix}a"/>
+      </xacro:if>
+    </xacro:unless>
+    <joint name="${prefix}a_frame_placement" type="fixed">
+       <insert_block name="origin" />
+      <parent link="${parent}"/>
+      <child link="${prefix}a_arm_base_link"/>
+    </joint>
+  </xacro:macro>
 </robot>
