Commit message: Handle new tip taxels meshes (offset from tip using scale) and fixed blinking taxels Added a poking stick with fingertip

File: agni_description/robots/left_poking_stick_ubi_ee.urdf.xacro (robot description, xacro)
@@ -1,5 +1,5 @@
 <?xml version="1.0"?>
 <robot xmlns:xacro="http://www.ros.org/wiki/xacro">
-  <xacro:include filename="$(find agni_description)/models/poking_stick.urdf.xacro" />
+  <xacro:include filename="$(find agni_description)/models/poking_stick_ubi.urdf.xacro" />
   <xacro:property name="cal_left_ee_x" value="0.0" />
   <xacro:property name="cal_left_ee_y" value="0.0" />
@@ -9,9 +9,9 @@
   <xacro:property name="cal_left_ee_roll" value="0.0" />
   <xacro:property name="l_ee_base_link" value="poking_stick" />
-  <xacro:macro name="right_poking_stick" params="prefix use_prefix" >
-    <xacro:poking_stick prefix="${prefix}h_" />
+  <xacro:macro name="right_poking_stick_ubi" params="prefix use_prefix" >
+    <xacro:poking_stick_ubi prefix="${prefix}h_" />
   </xacro:macro>
-  <xacro:macro name="left_poking_stick" params="prefix use_prefix" >
-    <xacro:poking_stick prefix="${prefix}h_" />
+  <xacro:macro name="left_poking_stick_ubi" params="prefix use_prefix" >
+    <xacro:poking_stick_ubi prefix="${prefix}h_" />
   </xacro:macro>
 </robot>

File: agni_description/robots/right_poking_stick_ubi_ee.urdf.xacro (robot description, xacro)
@@ -1,5 +1,5 @@
 <?xml version="1.0"?>
 <robot xmlns:xacro="http://www.ros.org/wiki/xacro">
-  <xacro:include filename="$(find agni_description)/models/poking_stick.urdf.xacro" />
+  <xacro:include filename="$(find agni_description)/models/poking_stick_ubi.urdf.xacro" />
   <xacro:property name="cal_right_ee_x" value="0.0" />
   <xacro:property name="cal_right_ee_y" value="0.0" />
@@ -9,9 +9,9 @@
   <xacro:property name="cal_right_ee_roll" value="0.0" />
   <xacro:property name="r_ee_base_link" value="poking_stick" />
-  <xacro:macro name="right_poking_stick" params="prefix use_prefix" >
-    <xacro:poking_stick prefix="${prefix}h_" />
+  <xacro:macro name="right_poking_stick_ubi" params="prefix use_prefix" >
+    <xacro:poking_stick_ubi prefix="${prefix}h_" />
   </xacro:macro>
-  <xacro:macro name="left_poking_stick" params="prefix use_prefix" >
-    <xacro:poking_stick prefix="${prefix}h_" />
+  <xacro:macro name="left_poking_stick_ubi" params="prefix use_prefix" >
+    <xacro:poking_stick_ubi prefix="${prefix}h_" />
   </xacro:macro>
 </robot>
