Commit message: Fixed missing use_prefix tag in myrmex ee

File: agni_description/robots/left_myrmex_ee.urdf.xacro (robot description, xacro)
@@ -9,8 +9,8 @@
   <xacro:property name="cal_left_ee_roll" value="0.0" />
   <xacro:property name="l_ee_base_link" value="myrmex_quick_mount" />
-  <xacro:macro name="right_myrmex" params="prefix" >
+  <xacro:macro name="right_myrmex" params="prefix use_prefix" >
     <xacro:myrmex_quick_mount prefix="${prefix}h_" />
   </xacro:macro>
-  <xacro:macro name="left_myrmex" params="prefix" >
+  <xacro:macro name="left_myrmex" params="prefix use_prefix" >
     <xacro:myrmex_quick_mount prefix="${prefix}h_" />
   </xacro:macro>

File: agni_description/robots/right_myrmex_ee.urdf.xacro (robot description, xacro)
@@ -9,8 +9,8 @@
   <xacro:property name="cal_right_ee_roll" value="0.0" />
   <xacro:property name="r_ee_base_link" value="myrmex_quick_mount" />
-  <xacro:macro name="right_myrmex" params="prefix" >
+  <xacro:macro name="right_myrmex" params="prefix use_prefix" >
     <xacro:myrmex_quick_mount prefix="${prefix}h_" />
   </xacro:macro>
-  <xacro:macro name="left_myrmex" params="prefix" >
+  <xacro:macro name="left_myrmex" params="prefix use_prefix" >
     <xacro:myrmex_quick_mount prefix="${prefix}h_" />
   </xacro:macro>
