Commit message: Used new xacro macro calls to generalize end-effector calls created shadow_motor left and right end-effector with internal properties and offsets

File: agni_description/robots/platforms.urdf.xacro (robot description, xacro)
@@ -2,9 +2,13 @@
 <robot name="$(arg ARM)_$(arg R_EE)_flobi"
      xmlns:xacro="http://www.ros.org/wiki/xacro">
-  <xacro:include filename="$(find agni_description)/robots/$(arg ARM)_$(arg R_EE).urdf.xacro" />
-  <xacro:include filename="$(find agni_description)/$(arg ARM)/$(arg ARM)_includes.urdf.xacro" />
-  <xacro:include filename="$(find agni_description)/robots/$(arg R_EE)_includes.urdf.xacro" />
-  <xacro:include filename="$(find agni_description)/robots/$(arg L_EE)_includes.urdf.xacro" />
-  <xacro:include filename="$(find agni_description)/calibration/default_cal.xml"/>
+  <xacro:arg name="ARM" default="kuka"/>
+  <xacro:arg name="R_EE" default="right_shadow_motor"/>
+  <xacro:arg name="L_EE" default="left_shadow_motor"/>
+  <xacro:arg name="FLOBI" default="0"/>
+  <xacro:include filename="$(find agni_description)/robots/$(arg ARM)_anytool.urdf.xacro" />
+  <xacro:include filename="$(find agni_description)/$(arg ARM)/$(arg ARM).urdf.xacro" />
+  <xacro:include filename="$(find agni_description)/robots/$(arg R_EE)_ee.urdf.xacro" />
+  <xacro:include filename="$(find agni_description)/robots/$(arg L_EE)_ee.urdf.xacro" />
+  <xacro:include filename="$(find agni_description)/calibration/$(arg ARM)_cal.xml"/>
   <xacro:include filename="$(find agni_description)/urdf/frame-half.urdf.xacro"/>
   <!--
@@ -13,13 +17,17 @@
   arm and hand -->
   <xacro:if value="$(arg R)">
-    <xacro:arm_ee parent="$(arg ARM)_frame" arm="$(arg ARM)" prefix="r" is_right="1" use_prefix="$(arg USE_PREFIX)" controller="false">
+    <xacro:arm_ee parent="$(arg ARM)_frame" arm="$(arg ARM)" prefix="r" is_right="1" ee_macro="$(arg R_EE)" ee_base_link="${r_ee_base_link}" use_prefix="$(arg USE_PREFIX)" controller="false">
       <origin xyz="${cal_right_arm_x} ${cal_right_arm_y} ${cal_right_arm_z}"
       rpy="${cal_right_arm_roll} ${cal_right_arm_pitch} ${cal_right_arm_yaw}"/>
+      <origin xyz="${cal_right_ee_x} ${cal_right_ee_y} ${cal_right_ee_z}"
+      rpy="${cal_right_ee_roll} ${cal_right_ee_pitch} ${cal_right_ee_yaw}"/>
     </xacro:arm_ee>
   </xacro:if>
   <xacro:if value="$(arg L)">
-    <xacro:arm_ee parent="$(arg ARM)_frame" arm="$(arg ARM)" prefix="l" is_right="0" use_prefix="$(arg USE_PREFIX)" controller="false">
+    <xacro:arm_ee parent="$(arg ARM)_frame" arm="$(arg ARM)" prefix="l" is_right="0" ee_macro="$(arg L_EE)" ee_base_link="${l_ee_base_link}" use_prefix="$(arg USE_PREFIX)" controller="false">
       <origin xyz="${cal_left_arm_x} ${cal_left_arm_y} ${cal_left_arm_z}"
           rpy="${cal_left_arm_roll} ${cal_left_arm_pitch} ${cal_left_arm_yaw}"/>
+      <origin xyz="${cal_left_ee_x} ${cal_left_ee_y} ${cal_left_ee_z}"
+      rpy="${cal_left_ee_roll} ${cal_left_ee_pitch} ${cal_left_ee_yaw}"/>
     </xacro:arm_ee>
   </xacro:if>

Commit message: Added dual arm robot_description Fixed platform and launch files to handle no R_EE_TYPE='-' Fixed arm_and_hand launch to pass all the args Updated documentation

File: agni_description/robots/platforms.urdf.xacro (robot description, xacro)
@@ -56,4 +56,7 @@
   <!-- frame generation -->
   <xacro:call macro="$(arg ARM)_frame" prefix="$(arg ARM)" />
+  <xacro:property name="r" value="$(arg R)"/>
+  <xacro:property name="r_ee_type" value="$(arg R_EE_TYPE)"/>
+  <xacro:property name="l_ee_type" value="$(arg L_EE_TYPE)"/>
   <xacro:if value="$(arg R)">
     <!-- Arm -->
@@ -63,13 +66,12 @@
       rpy="${cal_arm_roll.get('right',0.0)} ${cal_arm_pitch.get('right',0.0)} ${cal_arm_yaw.get('right',0.0)}"/>
     </xacro:call>
-    <xacro:property name="r_ee_type" value="$(arg R_EE_TYPE)"/>
     <xacro:property name="r_ee_side" value="$(arg R_EE_SIDE)"/>
     <xacro:property name="r_ee_model" value="$(arg R_EE_MODEL)"/>
     <xacro:property name="r_ee_prefix" value="${'rh' if r_ee_side=='right' else 'lh'}"/>
     <xacro:property name="r_ee_tactile" value="$(arg R_EE_TACTILE)"/>
-    <xacro:if value="${r_ee_type!='-'}">
+    <xacro:if value="${1 if r_ee_type!='-' else 0}">
      <!-- right end-effector -->
-      <xacro:include filename="$(find agni_description)/robots/$(arg R_EE_TYPE)_ee.urdf.xacro" />
-      <xacro:include filename="$(find agni_description)/calibration/$(arg R_EE_TYPE)_$(arg R_EE_MODEL)_cal.xml"/>
+      <xacro:include filename="$(find agni_description)/robots/${r_ee_type}_ee.urdf.xacro" />
+      <xacro:include filename="$(find agni_description)/calibration/${r_ee_type}_${r_ee_model}_cal.xml"/>
       <xacro:call macro="${r_ee_type}" model="$(arg R_EE_MODEL)" tactile="${r_ee_tactile if r_ee_tactile!='-' else ''}" side="${r_ee_side}" prefix="${r_ee_prefix}"/>
      <!-- Link arm and effector -->
@@ -83,5 +85,5 @@
   </xacro:if>
   <xacro:if value="$(arg L)">
-    <!-- Arm -->
+    <!-- Arm  -->
     <xacro:property name="arm"  value="$(arg ARM)" />
     <xacro:call macro="${arm}_arm" parent="world" side="left" controller="$(arg SIM)">
@@ -89,17 +91,16 @@
       rpy="${cal_arm_roll.get('left',0.0)} ${cal_arm_pitch.get('left',0.0)} ${cal_arm_yaw.get('left',0.0)}"/>
     </xacro:call>
-    <xacro:property name="l_ee_type" value="$(arg L_EE_TYPE)"/>
     <xacro:property name="l_ee_side" value="$(arg L_EE_SIDE)"/>
     <xacro:property name="l_ee_model" value="$(arg L_EE_MODEL)"/>
     <xacro:property name="l_ee_prefix" value="${'rh' if l_ee_side=='right' else 'lh'}"/>
     <xacro:property name="l_ee_tactile" value="$(arg L_EE_TACTILE)"/>
-    <xacro:if value="${l_ee_type!='-'}">
+    <xacro:if value="${1 if l_ee_type!='-' else 0}">
       <!-- left end-effector -->
-      <xacro:if value="${r_ee_type!=l_ee_type}">
-        <xacro:include filename="$(find agni_description)/robots/$(arg L_EE_TYPE)_ee.urdf.xacro" />
-        <xacro:include filename="$(find agni_description)/calibration/$(arg L_EE_TYPE)_$(arg L_EE_MODEL)_cal.xml"/>
+      <xacro:if value="${1 if (r_ee_type!=l_ee_type or r=='0') else 0}">
+        <xacro:include filename="$(find agni_description)/robots/${l_ee_type}_ee.urdf.xacro" />
+        <xacro:include filename="$(find agni_description)/calibration/${l_ee_type}_${l_ee_model}_cal.xml"/>
       </xacro:if>
       <xacro:call macro="${l_ee_type}" model="$(arg L_EE_MODEL)" tactile="${l_ee_tactile if l_ee_tactile!='-' else ''}" side="${l_ee_side}" prefix="${l_ee_prefix}"/>
-     <!-- Link arm and effector -->
+      <!-- Link arm and effector -->
       <joint name="la_arm_hand_mount" type="fixed">
         <parent link="la_${arm_mount[arm]}"/>
