Commit message: Added cmake xacro generation of sfb urdf files Fixed left_arm_and_hand typo Added agni_path replacement with a single find Updated sfb.launch to reduce includes Added famula setup

File: agni_description/robots/famula.urdf.xacro (robot description, xacro)
@@ -2,19 +2,20 @@
 <robot name="arm_hand_shadow" xmlns:xacro="http://www.ros.org/wiki/xacro">
   <xacro:arg name="SIM" default="1"/>
-  <xacro:include filename="$(find agni_description)/urdf/pa10_frame.urdf.xacro"/>
-  <!-- arm with end-effector
-  <xacro:include filename="$(find agni_description)/robots/pa10_arm.urdf.xacro" /> -->
+  <xacro:include filename="$(find agni_description)/urdf/kuka_frame.urdf.xacro"/>
+  <!-- arm with -->
+  <xacro:include filename="$(find agni_description)/robots/kuka_arm.urdf.xacro" />
   <!-- arm calibration -->
-  <xacro:include filename="$(find agni_description)/calibration/pa10_cal.xml"/>
+  <xacro:include filename="$(find agni_description)/calibration/kuka_cal.xml"/>
   <!-- end-effector -->
   <xacro:include filename="$(find agni_description)/robots/shadow_hand_ee.urdf.xacro" />
-  <!-- must be world to spawn the arm in gazebo and have it fixed at the calibration location -->
-  <link name="world" />
-  <xacro:call macro="pa10_frame" prefix="pa10" />
+  <!-- arm and hand mount calibration (should always be last) -->
+  <xacro:include filename="$(find agni_description)/calibration/famula_cal.xml"/>
+  <!-- Frame -->
+  <xacro:call macro="kuka_frame" prefix="kuka" />
   <!-- Right -->
     <!-- Arm -->
-    <xacro:call macro="kuka_arm" parent="world" side="right" controller="$(arg CTRL)">
-      <origin xyz="${cal_right_arm_x} ${cal_right_arm_y} ${cal_right_arm_z}"
-        rpy="${cal_right_arm_roll} ${cal_right_arm_pitch} ${cal_right_arm_yaw}"/>
+    <xacro:call macro="kuka_arm" parent="world" side="right" controller="$(arg SIM)">
+      <origin xyz="${cal_arm_x['right']} ${cal_arm_y['right']} ${cal_arm_z['right']}"
+      rpy="${cal_arm_roll['right']} ${cal_arm_pitch['right']} ${cal_arm_yaw['right']}"/>
     </xacro:call>
     <!-- Effector -->
@@ -22,14 +23,14 @@
     <!-- Link arm and effector -->
     <joint name="ra_arm_hand_mount" type="fixed">
-      <parent link="ra_arm_hand_mount"/>
-      <child link="rh_forearm}"/>
-      <origin xyz="${cal_right_ee_x} ${cal_right_ee_y} ${cal_right_ee_z}"
-    rpy="${cal_right_ee_roll} ${cal_right_ee_pitch} ${cal_right_ee_yaw}"/>
+      <parent link="ra_${arm_mount['kuka']}"/>
+      <child link="rh_${ee_mount['shadow_hand']}"/>
+      <origin xyz="${cal_ee_x['shadow_hand']['right']} ${cal_ee_y['shadow_hand']['right']} ${cal_ee_z['shadow_hand']['right']}"
+  rpy="${cal_ee_roll['shadow_hand']['right']} ${cal_ee_pitch['shadow_hand']['right']} ${cal_ee_yaw['shadow_hand']['right']}"/>
     </joint>
   <!-- Left -->
     <!-- Arm -->
-    <xacro:call macro="kuka_arm" parent="world" side="right" controller="$(arg CTRL)">
-      <origin xyz="${cal_left_arm_x} ${cal_left_arm_y} ${cal_left_arm_z}"
-          rpy="${cal_left_arm_roll} ${cal_left_arm_pitch} ${cal_left_arm_yaw}"/>
+    <xacro:call macro="kuka_arm" parent="world" side="right" controller="$(arg SIM)">
+     <origin xyz="${cal_arm_x['left']} ${cal_arm_y['left']} ${cal_arm_z['left']}"
+      rpy="${cal_arm_roll['left']} ${cal_arm_pitch['left']} ${cal_arm_yaw['left']}"/>
     </xacro:call>
     <!-- Effector -->
@@ -37,8 +38,13 @@
     <!-- Link arm and effector -->
     <joint name="la_arm_hand_mount" type="fixed">
-      <parent link="la_arm_hand_mount"/>
-      <child link="lh_forearm}"/>
-      <origin xyz="${cal_left_ee_x} ${cal_left_ee_y} ${cal_left_ee_z}"
-      rpy="${cal_left_ee_roll} ${cal_left_ee_pitch} ${cal_left_ee_yaw}"/>
+      <parent link="la_${arm_mount['kuka']}"/>
+      <child link="lh_${ee_mount['shadow_hand']}"/>
+      <origin xyz="${cal_ee_x['shadow_hand']['left']} ${cal_ee_y['shadow_hand']['left']} ${cal_ee_z['shadow_hand']['left']}"
+  rpy="${cal_ee_roll['shadow_hand']['left']} ${cal_ee_pitch['shadow_hand']['left']} ${cal_ee_yaw['shadow_hand']['left']}"/>
     </joint>
+    <!-- flobi -->
+    <xacro:include filename="$(find flobi_sim)/defs/xacro/flobiv3.urdf.xacro" />
+    <xacro:flobi prefix="" neutral="1" gender="0" parent="kuka_frame" >
+      <origin xyz="0 ${cal_arm_y['right']} ${cal_arm_z['right']+mount_triangle_length/2*sin(60/180.0*pi)+0.01}" rpy="0 0 ${-pi/2.0}"/>
+    </xacro:flobi>
 </robot>

File: agni_description/robots/platforms.urdf.xacro (robot description, xacro)
@@ -47,11 +47,13 @@
           of the mounting part of this effector when attached on the arm
           -->
+  <!-- speeding up -->
+  <xacro:property name="agni_description_path" value="$(find agni_description)"/>
   <xacro:include filename="$(find sr_description)/materials.urdf.xacro" />
   <!-- arm -->
-  <xacro:include filename="$(find agni_description)/robots/$(arg ARM)_arm.urdf.xacro" />
+  <xacro:include filename="${agni_description_path}/robots/$(arg ARM)_arm.urdf.xacro" />
   <!-- frame -->
-  <xacro:include filename="$(find agni_description)/urdf/$(arg ARM)_frame.urdf.xacro"/>
+  <xacro:include filename="${agni_description_path}/urdf/$(arg ARM)_frame.urdf.xacro"/>
   <!-- arm calibration -->
-  <xacro:include filename="$(find agni_description)/calibration/$(arg ARM)_cal.xml"/>
+  <xacro:include filename="${agni_description_path}/calibration/$(arg ARM)_cal.xml"/>
   <!-- frame generation -->
   <xacro:call macro="$(arg ARM)_frame" prefix="$(arg ARM)" />
@@ -72,6 +74,6 @@
     <xacro:if value="${1 if r_ee_type!='-' else 0}">
      <!-- right end-effector -->
-      <xacro:include filename="$(find agni_description)/robots/${r_ee_type}_ee.urdf.xacro" />
-      <xacro:include filename="$(find agni_description)/calibration/${r_ee_type}_${r_ee_model}_cal.xml"/>
+      <xacro:include filename="${agni_description_path}/robots/${r_ee_type}_ee.urdf.xacro" />
+      <xacro:include filename="${agni_description_path}/calibration/${r_ee_type}_${r_ee_model}_cal.xml"/>
       <xacro:call macro="${r_ee_type}" model="$(arg R_EE_MODEL)" tactile="${r_ee_tactile if r_ee_tactile!='-' else ''}" side="${r_ee_side}" prefix="${r_ee_prefix}"/>
      <!-- Link arm and effector -->
@@ -97,7 +99,7 @@
     <xacro:if value="${1 if l_ee_type!='-' else 0}">
       <!-- left end-effector -->
-      <xacro:if value="${1 if (r_ee_type!=l_ee_type or r=='0') else 0}">
-        <xacro:include filename="$(find agni_description)/robots/${l_ee_type}_ee.urdf.xacro" />
-        <xacro:include filename="$(find agni_description)/calibration/${l_ee_type}_${l_ee_model}_cal.xml"/>
+      <xacro:if value="${1 if (r_ee_type!=l_ee_type or r==0) else 0}">
+        <xacro:include filename="${agni_description_path}/robots/${l_ee_type}_ee.urdf.xacro" />
+        <xacro:include filename="${agni_description_path}/calibration/${l_ee_type}_${l_ee_model}_cal.xml"/>
       </xacro:if>
       <xacro:call macro="${l_ee_type}" model="$(arg L_EE_MODEL)" tactile="${l_ee_tactile if l_ee_tactile!='-' else ''}" side="${l_ee_side}" prefix="${l_ee_prefix}"/>

Commit message: reworked frame.urdf, separated calibration files

File: agni_description/robots/famula.urdf.xacro (robot description, xacro)
@@ -1,50 +1,52 @@
 <?xml version="1.0"?>
 <robot name="arm_hand_shadow" xmlns:xacro="http://www.ros.org/wiki/xacro">
-  <xacro:arg name="SIM" default="1"/>
-  <xacro:include filename="../urdf/kuka_frame.urdf.xacro"/>
-  <!-- arm with -->
-  <xacro:include filename="../robots/kuka_arm.urdf.xacro" />
-  <!-- arm calibration -->
-  <xacro:include filename="../calibration/kuka_cal.xml"/>
-  <!-- end-effector -->
-  <xacro:include filename="../robots/shadow_hand_ee.urdf.xacro" />
-  <!-- arm and hand mount calibration (should always be last) -->
-  <xacro:include filename="../calibration/famula_cal.xml"/>
-  <!-- Frame -->
-  <xacro:call macro="kuka_frame" prefix="kuka" />
-  <!-- Right -->
-    <!-- Arm -->
-    <xacro:call macro="kuka_arm" parent="world" side="right" controller="$(arg SIM)">
-      <origin xyz="${cal_arm_x['right']} ${cal_arm_y['right']} ${cal_arm_z['right']}"
-      rpy="${cal_arm_roll['right']} ${cal_arm_pitch['right']} ${cal_arm_yaw['right']}"/>
-    </xacro:call>
-    <!-- Effector -->
-    <xacro:call macro="shadow_hand" model="motor" side="right" tactile="ubi" prefix="rh" />
-    <!-- Link arm and effector -->
-    <joint name="ra_arm_hand_mount" type="fixed">
-      <parent link="ra_${arm_mount['kuka']}"/>
-      <child link="rh_${ee_mount['shadow_hand']}"/>
-      <origin xyz="${cal_ee_x['shadow_hand']['right']} ${cal_ee_y['shadow_hand']['right']} ${cal_ee_z['shadow_hand']['right']}"
-  rpy="${cal_ee_roll['shadow_hand']['right']} ${cal_ee_pitch['shadow_hand']['right']} ${cal_ee_yaw['shadow_hand']['right']}"/>
-    </joint>
-  <!-- Left -->
-    <!-- Arm -->
-    <xacro:call macro="kuka_arm" parent="world" side="left" controller="$(arg SIM)">
-     <origin xyz="${cal_arm_x['left']} ${cal_arm_y['left']} ${cal_arm_z['left']}"
-      rpy="${cal_arm_roll['left']} ${cal_arm_pitch['left']} ${cal_arm_yaw['left']}"/>
-    </xacro:call>
-    <!-- Effector -->
-    <xacro:call macro="shadow_hand" model="motor" side="left" tactile="ubi" prefix="lh" />
-    <!-- Link arm and effector -->
-    <joint name="la_arm_hand_mount" type="fixed">
-      <parent link="la_${arm_mount['kuka']}"/>
-      <child link="lh_${ee_mount['shadow_hand']}"/>
-      <origin xyz="${cal_ee_x['shadow_hand']['left']} ${cal_ee_y['shadow_hand']['left']} ${cal_ee_z['shadow_hand']['left']}"
-  rpy="${cal_ee_roll['shadow_hand']['left']} ${cal_ee_pitch['shadow_hand']['left']} ${cal_ee_yaw['shadow_hand']['left']}"/>
-    </joint>
-    <!-- flobi -->
-    <xacro:include filename="$(find flobi_sim)/defs/xacro/flobiv3.urdf.xacro" />
-    <xacro:flobi prefix="" neutral="1" gender="0" parent="kuka_frame" >
-      <origin xyz="0 ${cal_arm_y['right']} ${cal_arm_z['right']+mount_triangle_length/2*sin(60/180.0*pi)+0.01}" rpy="0 0 ${-pi/2.0}"/>
-    </xacro:flobi>
+	<xacro:arg name="SIM" default="1"/>
+	<!-- Frame -->
+	<xacro:include filename="../urdf/frame-half.urdf.xacro"/>
+	<xacro:include filename="../calibration/kuka_frame_cal.xml"/>
+	<xacro:frame prefix="kuka"/>
+	<!-- arm with -->
+	<xacro:include filename="../robots/kuka_arm.urdf.xacro" />
+	<!-- end-effector -->
+	<xacro:include filename="../robots/shadow_hand_ee.urdf.xacro" />
+	<!-- Right -->
+	<!-- Arm -->
+	<xacro:include filename="../calibration/famula_kuka_right_cal.xml"/>
+	<xacro:call macro="kuka_arm" parent="world" side="right" controller="$(arg SIM)">
+		<origin xyz="${cal_arm_x} ${cal_arm_y} ${cal_arm_z}"
+		        rpy="${cal_arm_roll} ${cal_arm_pitch} ${cal_arm_yaw}"/>
+	</xacro:call>
+	<!-- Effector -->
+	<xacro:call macro="shadow_hand" model="motor" side="right" tactile="ubi" prefix="rh" />
+	<!-- Link arm and effector -->
+	<xacro:include filename="../calibration/famula_shadow_hand_motor_right_cal.xml"/>
+	<joint name="ra_arm_hand_mount" type="fixed">
+		<parent link="ra_${arm_mount['kuka']}"/>
+		<child link="rh_${ee_mount['shadow_hand']}"/>
+		<origin xyz="${cal_ee_x} ${cal_ee_y} ${cal_ee_z}"
+		        rpy="${cal_ee_roll} ${cal_ee_pitch} ${cal_ee_yaw}"/>
+	</joint>
+	<!-- Left -->
+	<!-- Arm -->
+	<xacro:include filename="../calibration/famula_kuka_left_cal.xml"/>
+	<xacro:call macro="kuka_arm" parent="world" side="left" controller="$(arg SIM)">
+		<origin xyz="${cal_arm_x} ${cal_arm_y} ${cal_arm_z}"
+		        rpy="${cal_arm_roll} ${cal_arm_pitch} ${cal_arm_yaw}"/>
+	</xacro:call>
+	<!-- Effector -->
+	<xacro:call macro="shadow_hand" model="motor" side="left" tactile="ubi" prefix="lh" />
+	<!-- Link arm and effector -->
+	<xacro:include filename="../calibration/famula_shadow_hand_motor_left_cal.xml"/>
+	<joint name="la_arm_hand_mount" type="fixed">
+		<parent link="la_${arm_mount['kuka']}"/>
+		<child link="lh_${ee_mount['shadow_hand']}"/>
+		<origin xyz="${cal_ee_x} ${cal_ee_y} ${cal_ee_z}"
+		        rpy="${cal_ee_roll} ${cal_ee_pitch} ${cal_ee_yaw}"/>
+	</joint>
+	<!-- flobi -->
+	<xacro:include filename="$(find flobi_sim)/defs/xacro/flobiv3.urdf.xacro" />
+	<xacro:flobi prefix="" neutral="1" gender="0" parent="kuka_frame" >
+		<origin xyz="0 ${cal_mount_triangle_offset[1]} ${cal_mount_triangle_offset[2]+mount_triangle_length/2*sin(60/180.0*pi)+0.01}"
+		        rpy="0 0 ${-pi/2.0}"/>
+	</xacro:flobi>
 </robot>

File: agni_description/robots/frame.urdf.xacro (robot description, xacro)
@@ -1,7 +1,13 @@
 <?xml version="1.0"?>
-<robot name="platform"
-		 xmlns:xacro="http://www.ros.org/wiki/xacro">
-  <xacro:arg name="FRAME" default="kuka"/>
-  <xacro:include filename="../urdf/$(arg FRAME)_frame.urdf.xacro"/>
-  <xacro:call macro="$(arg FRAME)_frame" prefix="$(arg FRAME)" />
+<robot name="platform" xmlns:xacro="http://www.ros.org/wiki/xacro">
+	<!-- create the frame description, arguments: FRAME:=kuka|pa10 -->
+	<xacro:property name="FRAME" value="$(arg FRAME)"/>
+	<xacro:if value="${FRAME == 'kuka'}">
+		<xacro:include filename="../urdf/frame-half.urdf.xacro"/>
+	</xacro:if>
+	<xacro:if value="${FRAME == 'pa10'}">
+		<xacro:include filename="../urdf/frame.urdf.xacro"/>
+	</xacro:if>
+	<xacro:include filename="../calibration/${FRAME}_frame_cal.xml"/>
+	<xacro:frame prefix="${FRAME}"/>
 </robot>

File: agni_description/robots/sfb.urdf.xacro (robot description, xacro)
@@ -1,43 +1,42 @@
 <?xml version="1.0"?>
 <robot name="arm_hand_shadow" xmlns:xacro="http://www.ros.org/wiki/xacro">
-  <xacro:arg name="SIM" default="1"/>
-  <xacro:include filename="../urdf/pa10_frame.urdf.xacro"/>
-  <!-- arm  -->
-  <xacro:include filename="../robots/pa10_arm.urdf.xacro" />
-  <!-- end-effector -->
-  <xacro:include filename="../robots/shadow_hand_ee.urdf.xacro" />
-  <!-- arm and hand mount calibration (should always be last) -->
-  <xacro:include filename="../calibration/sfb_cal.xml"/>
-  <!-- Frame -->
-  <xacro:call macro="pa10_frame" prefix="pa10" />
-  <!-- Right -->
-    <!-- Arm -->
-    <xacro:call macro="pa10_arm" parent="world" side="right" controller="$(arg SIM)">
-      <origin xyz="${cal_arm_x['right']} ${cal_arm_y['right']} ${cal_arm_z['right']}"
-      rpy="${cal_arm_roll['right']} ${cal_arm_pitch['right']} ${cal_arm_yaw['right']}"/>
-    </xacro:call>
-    <!-- Effector -->
-    <xacro:call macro="shadow_hand" model="motor" side="right" tactile="ubi" prefix="rh" />
-    <!-- Link arm and effector -->
-    <joint name="ra_arm_hand_mount" type="fixed">
-      <parent link="ra_${arm_mount['pa10']}"/>
-      <child link="rh_${ee_mount['shadow_hand']}"/>
-  <origin xyz="${cal_ee_x['shadow_hand']['right']} ${cal_ee_y['shadow_hand']['right']} ${cal_ee_z['shadow_hand']['right']}"
-  rpy="${cal_ee_roll['shadow_hand']['right']} ${cal_ee_pitch['shadow_hand']['right']} ${cal_ee_yaw['shadow_hand']['right']}"/>
-    </joint>
-  <!-- Left -->
-    <!-- Arm -->
-    <xacro:call macro="pa10_arm" parent="world" side="left" controller="$(arg SIM)">
-      <origin xyz="${cal_arm_x['left']} ${cal_arm_y['left']} ${cal_arm_z['left']}"
-      rpy="${cal_arm_roll['left']} ${cal_arm_pitch['left']} ${cal_arm_yaw['left']}"/>
-    </xacro:call>
-    <!-- Effector -->
-    <xacro:call macro="shadow_hand" model="motor" side="left" tactile="ubi" prefix="lh" />
-    <!-- Link arm and effector -->
-    <joint name="la_arm_hand_mount" type="fixed">
-      <parent link="la_${arm_mount['pa10']}"/>
-      <child link="lh_${ee_mount['shadow_hand']}"/>
-        <origin xyz="${cal_ee_x['shadow_hand']['left']} ${cal_ee_y['shadow_hand']['left']} ${cal_ee_z['shadow_hand']['left']}"
-  rpy="${cal_ee_roll['shadow_hand']['left']} ${cal_ee_pitch['shadow_hand']['left']} ${cal_ee_yaw['shadow_hand']['left']}"/>
-    </joint>
+	<xacro:arg name="SIM" default="1"/>
+	<!-- Frame -->
+	<xacro:include filename="../urdf/frame.urdf.xacro"/>
+	<xacro:include filename="../calibration/pa10_frame_cal.xml"/>
+	<xacro:frame prefix="pa10"/>
+	<!-- arm  -->
+	<xacro:include filename="../robots/pa10_arm.urdf.xacro" />
+	<!-- end-effector -->
+	<xacro:include filename="../robots/shadow_hand_ee.urdf.xacro" />
+	<!-- Right -->
+	<!-- Arm -->
+	<xacro:include filename="../calibration/sfb_pa10_right_cal.xml"/>
+	<xacro:call macro="pa10_arm" parent="world" side="right" controller="$(arg SIM)">
+		<origin xyz="${cal_arm_x} ${cal_arm_y} ${cal_arm_z}" rpy="${cal_arm_roll} ${cal_arm_pitch} ${cal_arm_yaw}"/>
+	</xacro:call>
+	<!-- Effector -->
+	<xacro:call macro="shadow_hand" model="motor" side="right" tactile="ubi" prefix="rh" />
+	<!-- Link arm and effector -->
+	<xacro:include filename="../calibration/sfb_shadow_hand_motor_right_cal.xml"/>
+	<joint name="ra_arm_hand_mount" type="fixed">
+		<parent link="ra_${arm_mount['pa10']}"/>
+		<child link="rh_${ee_mount['shadow_hand']}"/>
+		<origin xyz="${cal_ee_x} ${cal_ee_y} ${cal_ee_z}" rpy="${cal_ee_roll} ${cal_ee_pitch} ${cal_ee_yaw}"/>
+	</joint>
+	<!-- Left -->
+	<!-- Arm -->
+	<xacro:include filename="../calibration/sfb_pa10_left_cal.xml"/>
+	<xacro:call macro="pa10_arm" parent="world" side="left" controller="$(arg SIM)">
+		<origin xyz="${cal_arm_x} ${cal_arm_y} ${cal_arm_z}" rpy="${cal_arm_roll} ${cal_arm_pitch} ${cal_arm_yaw}"/>
+	</xacro:call>
+	<!-- Effector -->
+	<xacro:call macro="shadow_hand" model="motor" side="left" tactile="ubi" prefix="lh" />
+	<!-- Link arm and effector -->
+	<xacro:include filename="../calibration/sfb_shadow_hand_motor_left_cal.xml"/>
+	<joint name="la_arm_hand_mount" type="fixed">
+		<parent link="la_${arm_mount['pa10']}"/>
+		<child link="lh_${ee_mount['shadow_hand']}"/>
+		<origin xyz="${cal_ee_x} ${cal_ee_y} ${cal_ee_z}" rpy="${cal_ee_roll} ${cal_ee_pitch} ${cal_ee_yaw}"/>
+	</joint>
 </robot>
