Commit message: reworked frame.urdf, separated calibration files

File: agni_description/urdf/frame-half.urdf.xacro (robot description, xacro)
@@ -4,148 +4,157 @@
       xmlns:controller="http://playerstage.sourceforge.net/gazebo/xmlschema/#controller"
       xmlns:interface="http://playerstage.sourceforge.net/gazebo/xmlschema/#interface">
-<xacro:include filename="../urdf/util.urdf.xacro"/>
-<xacro:include filename="../urdf/materials.urdf.xacro"/>
-<xacro:include filename="../calibration/kuka_cal.xml"/>
-  <xacro:property name="mount_triangle_length"     value="0.26" />
-<xacro:macro name="bar" params="thickness len *origin">
-   <visual>
-    <xacro:insert_block name="origin"/>
-    <geometry><box size="${thickness} ${thickness} ${len}"/></geometry>
-    <material name="Silver"/>
-   </visual>
-   <collision>
-    <xacro:insert_block name="origin"/>
-    <geometry><box size="${thickness} ${thickness} ${len}"/></geometry>
-   </collision>
-</xacro:macro>
-<xacro:macro name="frame-half" params="prefix thickness width depth height tableHeight">
-  <link name="world"/>
-  <link name="${prefix}_frame">
-    <inertial>
-      <mass value="100.0" />
-      <origin xyz="0 1.2 0.3" rpy="0 0 0"/>
-      <inertia ixx="4.0" ixy="0" ixz="0" iyy="4.0" iyz="0" izz="4.0"/>
-    </inertial>
-   <!-- horizontal front bar-->
-   <xacro:bar thickness="${thickness}" len="${width}">
-    <origin xyz="0 ${thickness/2} ${-thickness/2}" rpy="0 ${-pi/2} 0"/>
-   </xacro:bar>
-   <!-- horizontal rear bar -->
-   <xacro:bar thickness="${thickness}" len="${width}">
-    <origin xyz="0 ${depth+thickness/2} ${-thickness/2}" rpy="0 ${-pi/2} 0"/>
-   </xacro:bar>
-   <!-- horizontal rear bar top -->
-   <xacro:bar thickness="${thickness}" len="${width}">
-    <origin xyz="0 ${depth+thickness/2} ${height+thickness/2}" rpy="0 ${-pi/2} 0"/>
-   </xacro:bar>
-   <!-- left front pole -->
-   <xacro:bar thickness="${thickness}" len="${thickness+tableHeight}">
-    <origin xyz="${-(width+thickness)/2} ${thickness/2} ${-(thickness+tableHeight)/2}"/>
-   </xacro:bar>
-   <!-- right front pole -->
-   <xacro:bar thickness="${thickness}" len="${thickness+tableHeight}">
-    <origin xyz="${+(width+thickness)/2} ${thickness/2} ${-(thickness+tableHeight)/2}"/>
-   </xacro:bar>
-   <!-- left rear pole -->
-   <xacro:bar thickness="${thickness}" len="${height+2*thickness+tableHeight}">
-    <origin xyz="${-(width+thickness)/2} ${depth+thickness/2} ${(height-tableHeight)/2}"/>
-   </xacro:bar>
-   <!-- right rear pole -->
-   <xacro:bar thickness="${thickness}" len="${height+2*thickness+tableHeight}">
-    <origin xyz="${+(width+thickness)/2} ${depth+thickness/2} ${(height-tableHeight)/2}"/>
-   </xacro:bar>
-   <!-- left side bottom -->
-   <xacro:bar thickness="${thickness}" len="${depth}">
-    <origin xyz="${-(width+thickness)/2} ${depth/2} ${-thickness/2}"
-          rpy="${-pi/2} 0 0"/>
-   </xacro:bar>
-   <!-- right side bottom -->
-   <xacro:bar thickness="${thickness}" len="${depth}">
-    <origin xyz="${+(width+thickness)/2} ${depth/2} ${-thickness/2}"
-          rpy="${-pi/2} 0 0"/>
-   </xacro:bar>
-   <!-- left central pole -->
-   <xacro:bar thickness="${thickness}" len="${thickness+tableHeight+(height)/2}">
-    <origin xyz="${-thickness} ${(depth)/2+2*thickness} ${-(2*tableHeight-height)/4-thickness/2}"/>
-   </xacro:bar>
-   <!-- right central pole -->
-   <xacro:bar thickness="${thickness}" len="${thickness+tableHeight+(height)/2}">
-    <origin xyz="${thickness} ${(depth)/2+2*thickness} ${-(2*tableHeight-height)/4-thickness/2}"/>
-   </xacro:bar>
-   <!-- virtual protection plane for the screens -->
-    <!-- right screen -->
-   <visual>
-    <origin xyz="${-width/2+0.3} ${depth-thickness} ${height}"
-          rpy="0 0 0"/>
-    <geometry><box size="${0.6} ${0.1} ${0.4}"/></geometry>
-    <material name="Silver"/>
-   </visual>
-    <!-- left screen -->
-   <visual>
-     <origin xyz="${width/2-0.3} ${depth-thickness} ${height}"
-          rpy="0 0 0"/>
-    <geometry><box size="${0.6} ${0.1} ${0.4}"/></geometry>
-    <material name="Silver"/>
-   </visual>
-   <collision>
-      <origin xyz="0 ${depth-2*thickness} ${height/2}"
-          rpy="0 0 0"/>
-      <geometry><box size="${width+2*thickness} ${0.01} ${height+0.4+2*thickness}"/></geometry>
-    </collision>
-  <!-- kuka mount triangle -->
-   <visual>
-     <origin xyz="${cal_arm_x['left']-cos(30/180.0*pi)*0.01} ${cal_arm_y['left']} ${cal_arm_z['left']-sin(30/180.0*pi)*0.01}"
-        rpy="0 ${pi/3} 0"/>
-    <geometry><box size="${mount_triangle_length} ${mount_triangle_length} ${0.02}"/></geometry>
-    <material name="Silver"/>
-   </visual>
-   <collision>
-     <origin xyz="${cal_arm_x['left']-cos(30/180.0*pi)*0.01} ${cal_arm_y['left']} ${cal_arm_z['left']-sin(30/180.0*pi)*0.01}"
-        rpy="0 ${pi/3} 0"/>
-    <geometry><box size="${mount_triangle_length} ${mount_triangle_length} ${0.015}"/></geometry>
-   </collision>
-   <visual>
-     <origin xyz="${cal_arm_x['right']+cos(30/180.0*pi)*0.01} ${cal_arm_y['right']} ${cal_arm_z['right']-sin(30/180.0*pi)*0.01}"
-        rpy="0 ${-pi/3} 0"/>
-    <geometry><box size="${mount_triangle_length} ${mount_triangle_length} ${0.02}"/></geometry>
-    <material name="Silver"/>
-   </visual>
-    <collision>
-       <origin xyz="${cal_arm_x['right']+cos(30/180.0*pi)*0.01} ${cal_arm_y['right']} ${cal_arm_z['right']-sin(30/180.0*pi)*0.01}"
-        rpy="0 ${-pi/3} 0"/>
-    <geometry><box size="${mount_triangle_length} ${mount_triangle_length} ${0.015}"/></geometry>
-   </collision>
-   <visual>
-     <origin xyz="0 ${cal_arm_y['right']} ${cal_arm_z['right']-sin(30/180.0*pi)*0.02-mount_triangle_length/2*sin(60/180.0*pi)-0.01}"
-        rpy="0 0 0"/>
-    <geometry><box size="${mount_triangle_length} ${mount_triangle_length} ${0.02}"/></geometry>
-    <material name="Silver"/>
-   </visual>
-   <collision>
-      <origin xyz="0 ${cal_arm_y['right']} ${cal_arm_z['right']-sin(30/180.0*pi)*0.02-mount_triangle_length/2*sin(60/180.0*pi)-0.01}"
-        rpy="0 0 0"/>
-    <geometry><box size="${mount_triangle_length} ${mount_triangle_length} ${0.015}"/></geometry>
-   </collision>
-  <!-- table plane -->
-   <visual>
-    <origin xyz="0 ${depth/2} -0.01"
-          rpy="0 0 0"/>
-    <geometry><box size="${width} ${depth} ${0.02}"/></geometry>
-    <material name="Silver"/>
-   </visual>
-   <collision>
-      <origin xyz="0 ${depth/2} -0.01"
-          rpy="0 0 0"/>
-      <geometry><box size="${width} ${depth} ${0.02}"/></geometry>
-    </collision>
-  </link>
-  <gazebo reference="${prefix}_frame">
-      <material value="Gazebo/Grey"/>
-  </gazebo>
-  <joint name="${prefix}_frame_joint" type="fixed">
-      <origin xyz="0 0 0" rpy="0 0 0"/>
-      <parent link="world"/>
-      <child link="${prefix}_frame"/>
-  </joint>
-</xacro:macro>
+	<xacro:property name="mount_triangle_length" value="0.26" />
+	<xacro:include filename="../urdf/materials.urdf.xacro"/>
+	<xacro:macro name="bar" params="thickness len *origin">
+		<visual>
+			<xacro:insert_block name="origin"/>
+			<geometry><box size="${thickness} ${thickness} ${len}"/></geometry>
+			<material name="Silver"/>
+		</visual>
+		<collision>
+			<xacro:insert_block name="origin"/>
+			<geometry><box size="${thickness} ${thickness} ${len}"/></geometry>
+		</collision>
+	</xacro:macro>
+	<xacro:macro name="frame" params="prefix thickness:=${cal_frame_thick}
+	   width:=${cal_frame_width} depth:=${cal_frame_depth} height:=${cal_frame_height}
+	   tableHeight:=${cal_frame_table_height}
+	   triangle_offset:=${cal_mount_triangle_offset}">
+		<link name="world"/>
+		<link name="${prefix}_frame">
+			<inertial>
+				<mass value="100.0" />
+				<origin xyz="0 1.2 0.3" rpy="0 0 0"/>
+				<inertia ixx="4.0" ixy="0" ixz="0" iyy="4.0" iyz="0" izz="4.0"/>
+			</inertial>
+			<!-- horizontal front bar-->
+			<xacro:bar thickness="${thickness}" len="${width}">
+				<origin xyz="0 ${thickness/2} ${-thickness/2}" rpy="0 ${-pi/2} 0"/>
+			</xacro:bar>
+			<!-- horizontal rear bar -->
+			<xacro:bar thickness="${thickness}" len="${width}">
+				<origin xyz="0 ${depth+thickness/2} ${-thickness/2}" rpy="0 ${-pi/2} 0"/>
+			</xacro:bar>
+			<!-- horizontal rear bar top -->
+			<xacro:bar thickness="${thickness}" len="${width}">
+				<origin xyz="0 ${depth+thickness/2} ${height+thickness/2}" rpy="0 ${-pi/2} 0"/>
+			</xacro:bar>
+			<!-- left front pole -->
+			<xacro:bar thickness="${thickness}" len="${thickness+tableHeight}">
+				<origin xyz="${-(width+thickness)/2} ${thickness/2} ${-(thickness+tableHeight)/2}"/>
+			</xacro:bar>
+			<!-- right front pole -->
+			<xacro:bar thickness="${thickness}" len="${thickness+tableHeight}">
+				<origin xyz="${+(width+thickness)/2} ${thickness/2} ${-(thickness+tableHeight)/2}"/>
+			</xacro:bar>
+			<!-- left rear pole -->
+			<xacro:bar thickness="${thickness}" len="${height+2*thickness+tableHeight}">
+				<origin xyz="${-(width+thickness)/2} ${depth+thickness/2} ${(height-tableHeight)/2}"/>
+			</xacro:bar>
+			<!-- right rear pole -->
+			<xacro:bar thickness="${thickness}" len="${height+2*thickness+tableHeight}">
+				<origin xyz="${+(width+thickness)/2} ${depth+thickness/2} ${(height-tableHeight)/2}"/>
+			</xacro:bar>
+			<!-- left side bottom -->
+			<xacro:bar thickness="${thickness}" len="${depth}">
+				<origin xyz="${-(width+thickness)/2} ${depth/2} ${-thickness/2}"
+				        rpy="${-pi/2} 0 0"/>
+			</xacro:bar>
+			<!-- right side bottom -->
+			<xacro:bar thickness="${thickness}" len="${depth}">
+				<origin xyz="${+(width+thickness)/2} ${depth/2} ${-thickness/2}"
+				        rpy="${-pi/2} 0 0"/>
+			</xacro:bar>
+			<!-- left central pole -->
+			<xacro:bar thickness="${thickness}" len="${thickness+tableHeight+(height)/2}">
+				<origin xyz="${-thickness} ${(depth)/2+2*thickness} ${-(2*tableHeight-height)/4-thickness/2}"/>
+			</xacro:bar>
+			<!-- right central pole -->
+			<xacro:bar thickness="${thickness}" len="${thickness+tableHeight+(height)/2}">
+				<origin xyz="${thickness} ${(depth)/2+2*thickness} ${-(2*tableHeight-height)/4-thickness/2}"/>
+			</xacro:bar>
+			<!-- virtual protection plane for the screens -->
+			<!-- right screen -->
+			<visual>
+				<origin xyz="${-width/2+0.3} ${depth-thickness} ${height}"
+				        rpy="0 0 0"/>
+				<geometry><box size="${0.6} ${0.1} ${0.4}"/></geometry>
+				<material name="Silver"/>
+			</visual>
+			<!-- left screen -->
+			<visual>
+				<origin xyz="${width/2-0.3} ${depth-thickness} ${height}"
+				        rpy="0 0 0"/>
+				<geometry><box size="${0.6} ${0.1} ${0.4}"/></geometry>
+				<material name="Silver"/>
+			</visual>
+			<collision>
+				<origin xyz="0 ${depth-2*thickness} ${height/2}"
+				        rpy="0 0 0"/>
+				<geometry><box size="${width+2*thickness} ${0.01} ${height+0.4+2*thickness}"/></geometry>
+			</collision>
+			<!-- kuka mount triangle -->
+			<visual>
+				<origin xyz="${triangle_offset[0]-0.01*cos(30/180.0*pi)}
+				             ${triangle_offset[1]}
+				             ${triangle_offset[2]-0.01*sin(30/180.0*pi)}"
+				        rpy="0 ${pi/3} 0"/>
+				<geometry><box size="${mount_triangle_length} ${mount_triangle_length} ${0.02}"/></geometry>
+				<material name="Silver"/>
+			</visual>
+			<collision>
+				<origin xyz="${triangle_offset[0]-0.01*cos(30/180.0*pi)}
+				             ${triangle_offset[1]}
+				             ${triangle_offset[2]-0.01*sin(30/180.0*pi)}"
+				        rpy="0 ${pi/3} 0"/>
+				<geometry><box size="${mount_triangle_length} ${mount_triangle_length} ${0.015}"/></geometry>
+			</collision>
+			<visual>
+				<origin xyz="-${triangle_offset[0]+0.01*cos(30/180.0*pi)}
+				             ${triangle_offset[1]}
+				             ${triangle_offset[2]-0.01*sin(30/180.0*pi)}"
+				        rpy="0 ${-pi/3} 0"/>
+				<geometry><box size="${mount_triangle_length} ${mount_triangle_length} ${0.02}"/></geometry>
+				<material name="Silver"/>
+			</visual>
+			<collision>
+				<origin xyz="-${triangle_offset[0]+0.01*cos(30/180.0*pi)}
+				             ${triangle_offset[1]}
+				             ${triangle_offset[2]-0.01*sin(30/180.0*pi)}"
+				        rpy="0 ${-pi/3} 0"/>
+				<geometry><box size="${mount_triangle_length} ${mount_triangle_length} ${0.015}"/></geometry>
+			</collision>
+			<visual>
+				<origin xyz="0 ${triangle_offset[1]} ${triangle_offset[2]-sin(30/180.0*pi)*0.02-mount_triangle_length/2*sin(60/180.0*pi)-0.01}"
+				        rpy="0 0 0"/>
+				<geometry><box size="${mount_triangle_length} ${mount_triangle_length} ${0.02}"/></geometry>
+				<material name="Silver"/>
+			</visual>
+			<collision>
+				<origin xyz="0 ${triangle_offset[1]} ${triangle_offset[2]-sin(30/180.0*pi)*0.02-mount_triangle_length/2*sin(60/180.0*pi)-0.01}"
+				        rpy="0 0 0"/>
+				<geometry><box size="${mount_triangle_length} ${mount_triangle_length} ${0.015}"/></geometry>
+			</collision>
+			<!-- table plane -->
+			<visual>
+				<origin xyz="0 ${depth/2} -0.01"
+				        rpy="0 0 0"/>
+				<geometry><box size="${width} ${depth} ${0.02}"/></geometry>
+				<material name="Silver"/>
+			</visual>
+			<collision>
+				<origin xyz="0 ${depth/2} -0.01"
+				        rpy="0 0 0"/>
+				<geometry><box size="${width} ${depth} ${0.02}"/></geometry>
+			</collision>
+		</link>
+		<gazebo reference="${prefix}_frame">
+			<material value="Gazebo/Grey"/>
+		</gazebo>
+		<joint name="${prefix}_frame_joint" type="fixed">
+			<origin xyz="0 0 0" rpy="0 0 0"/>
+			<parent link="world"/>
+			<child link="${prefix}_frame"/>
+		</joint>
+	</xacro:macro>
 </root>
