Commit message: reworked frame.urdf, separated calibration files

File: agni_description/urdf/frame.urdf.xacro (robot description, xacro)
@@ -1,154 +1,157 @@
 <?xml version="1.0"?>
 <root xmlns:xacro="http://www.ros.org/wiki/xacro">
-<xacro:include filename="../urdf/util.urdf.xacro"/>
-<xacro:include filename="../urdf/materials.urdf.xacro"/>
-<xacro:macro name="barcollision" params="thickness len *origin">
-   <visual>
-    <xacro:insert_block name="origin"/>
-    <geometry><box size="${thickness} ${thickness} ${len}"/></geometry>
-    <material name="Silver"/>
-   </visual>
-   <collision>
-    <xacro:insert_block name="origin"/>
-    <geometry><box size="${thickness} ${thickness} ${len}"/></geometry>
-   </collision>
-</xacro:macro>
-<xacro:macro name="bar" params="thickness len *origin">
-   <visual>
-    <xacro:insert_block name="origin"/>
-    <geometry><box size="${thickness} ${thickness} ${len}"/></geometry>
-    <material name="Silver"/>
-   </visual>
-</xacro:macro>
-<xacro:macro name="frame" params="prefix thickness width depth height tableHeight mountingYpos mountingspacing">
-  <link name="world"/>
-  <link name="${prefix}_frame">
-     <inertial>
-      <mass value="100.0" />
-      <origin xyz="0 1.2 0.3" rpy="0 0 0"/>
-      <inertia ixx="4.0" ixy="0" ixz="0" iyy="4.0" iyz="0" izz="4.0"/>
-    </inertial>
-	 <!-- horizontal front bar-->
-	 <xacro:bar thickness="${thickness}" len="${width}">
-		<origin xyz="0 ${-thickness/2} ${-thickness/2}" rpy="0 ${-pi/2} 0"/>
-	 </xacro:bar>
-	 <!-- horizontal rear bar -->
-	 <xacro:bar thickness="${thickness}" len="${width}">
-		<origin xyz="0 ${depth+thickness/2} ${-thickness/2}" rpy="0 ${-pi/2} 0"/>
-	 </xacro:bar>
-    <!-- robot mounting bars -->
-	 <!-- horizontal front bar top -->
-	 <xacro:bar thickness="${thickness}" len="${width}">
-		<origin xyz="0 ${mountingYpos-mountingspacing/2 + thickness/2} ${height+thickness/2}" rpy="0 ${-pi/2} 0"/>
-	 </xacro:bar>
-	 <!-- horizontal rear bar top -->
-	 <xacro:bar thickness="${thickness}" len="${width}">
-		<origin xyz="0 ${mountingYpos+mountingspacing/2 - thickness/2} ${height+thickness/2}" rpy="0 ${-pi/2} 0"/>
-	 </xacro:bar>
-    <!-- additional collision box inbetzeen the mounting bars at the top -->
-     <collision>
-      <origin xyz="0 ${mountingYpos} ${height+thickness/2}"
-          rpy="0 0 0"/>
-      <geometry><box size="${width} ${mountingspacing-thickness} ${thickness}"/></geometry>
-    </collision>
-	 <!-- left front pole -->
-	 <xacro:bar thickness="${thickness}" len="${height+2*thickness+tableHeight}">
-		<origin xyz="${-(width+thickness)/2} ${-thickness/2} ${(height-tableHeight)/2}"/>
-	 </xacro:bar>
-	 <!-- right front pole -->
-	 <xacro:bar thickness="${thickness}" len="${height+2*thickness+tableHeight}">
-		<origin xyz="${+(width+thickness)/2} ${-thickness/2} ${(height-tableHeight)/2}"/>
-	 </xacro:bar>
-	 <!-- left rear pole -->
-	 <xacro:bar thickness="${thickness}" len="${height+2*thickness+tableHeight}">
-		<origin xyz="${-(width+thickness)/2} ${depth+thickness/2} ${(height-tableHeight)/2}"/>
-	 </xacro:bar>
-	 <!-- right rear pole -->
-	 <xacro:bar thickness="${thickness}" len="${height+2*thickness+tableHeight}">
-		<origin xyz="${+(width+thickness)/2} ${depth+thickness/2} ${(height-tableHeight)/2}"/>
-	 </xacro:bar>
-	 <!-- left side bottom -->
-	 <xacro:bar thickness="${thickness}" len="${depth}">
-		<origin xyz="${-(width+thickness)/2} ${depth/2} ${-thickness/2}"
-				  rpy="${-pi/2} 0 0"/>
-	 </xacro:bar>
-	 <!-- right side bottom -->
-	 <xacro:bar thickness="${thickness}" len="${depth}">
-		<origin xyz="${+(width+thickness)/2} ${depth/2} ${-thickness/2}"
-				  rpy="${-pi/2} 0 0"/>
-	 </xacro:bar>
-	 <!-- left side top -->
-	 <xacro:bar thickness="${thickness}" len="${depth}">
-		<origin xyz="${-(width+thickness)/2} ${depth/2} ${height+thickness/2}"
-				  rpy="${-pi/2} 0 0"/>
-	 </xacro:bar>
-	 <!-- right side top -->
-	 <xacro:bar thickness="${thickness}" len="${depth}">
-		<origin xyz="${+(width+thickness)/2} ${depth/2} ${height+thickness/2}"
-				  rpy="${-pi/2} 0 0"/>
-	 </xacro:bar>
-   <!-- table plane -->
-   <visual>
-    <origin xyz="0 ${depth/2} -0.01"
-          rpy="0 0 0"/>
-    <geometry><box size="${width} ${depth} ${0.02}"/></geometry>
-    <material name="Silver"/>
-   </visual>
-   <collision>
-      <origin xyz="0 ${depth/2} -0.01"
-          rpy="0 0 0"/>
-      <geometry><box size="${width} ${depth} ${0.02}"/></geometry>
-    </collision>
-   <!-- virtual fence -->
-   <!-- left pane -->
-   <collision>
-      <origin xyz="${-(width+thickness)/2} ${depth/2} ${height/2}"
-          rpy="0 0 0"/>
-      <geometry><box size="${thickness} ${depth} ${height}"/></geometry>
-   </collision>
-   <!-- right pane -->
-   <collision>
-      <origin xyz="${+(width+thickness)/2} ${depth/2} ${height/2}"
-          rpy="0 0 0"/>
-      <geometry><box size="${thickness} ${depth} ${height}"/></geometry>
-   </collision>
-   <!-- front pane -->
-   <collision>
-      <origin xyz="0 ${-thickness/2} ${height/2}"
-          rpy="0 0 0"/>
-      <geometry><box size="${width} ${thickness} ${height}"/></geometry>
-   </collision>
-   <!-- back pane -->
-   <collision>
-      <origin xyz="0 ${depth + thickness/2} ${height/2}"
-          rpy="0 0 0"/>
-      <geometry><box size="${width} ${thickness} ${height}"/></geometry>
-   </collision>
-  <!-- virtual protection box for the screens -->
-    <!-- right screen -->
-   <visual>
-    <origin xyz="${+0.575/2} ${mountingYpos-mountingspacing/2 -thickness} ${height+thickness/2}"
-          rpy="0.32 0 0"/>
-    <geometry><box size="${0.550} ${0.07} ${0.35}"/></geometry>
-    <material name="Silver"/>
-   </visual>
-    <!-- left screen -->
-   <visual>
-    <origin xyz="${-0.575/2} ${mountingYpos-mountingspacing/2 -thickness} ${height+thickness/2}"
-          rpy="0.32 0 0"/>
-    <geometry><box size="${0.550} ${0.07} ${0.35}"/></geometry>
-    <material name="Silver"/>
-   </visual>
-   <collision>
-      <origin xyz="0 ${mountingYpos-mountingspacing/2 -thickness} ${height+thickness/2}"
-          rpy="0 0 0"/>
-      <geometry><box size="${0.575*2} ${0.250} ${0.350}"/></geometry>
-    </collision>
-  </link>
-  <joint name="${prefix}_frame_joint" type="fixed">
-      <origin xyz="0 0 0" rpy="0 0 0"/>
-      <parent link="world"/>
-      <child link="${prefix}_frame"/>
-  </joint>
-</xacro:macro>
+	<xacro:include filename="../urdf/materials.urdf.xacro"/>
+	<xacro:macro name="barcollision" params="thickness len *origin">
+		<visual>
+			<xacro:insert_block name="origin"/>
+			<geometry><box size="${thickness} ${thickness} ${len}"/></geometry>
+			<material name="Silver"/>
+		</visual>
+		<collision>
+			<xacro:insert_block name="origin"/>
+			<geometry><box size="${thickness} ${thickness} ${len}"/></geometry>
+		</collision>
+	</xacro:macro>
+	<xacro:macro name="bar" params="thickness len *origin">
+		<visual>
+			<xacro:insert_block name="origin"/>
+			<geometry><box size="${thickness} ${thickness} ${len}"/></geometry>
+			<material name="Silver"/>
+		</visual>
+	</xacro:macro>
+	<xacro:macro name="frame" params="prefix thickness:=${cal_frame_thick}
+	   width:=${cal_frame_width} depth:=${cal_frame_depth} height:=${cal_frame_height}
+	   tableHeight:=${cal_frame_table_height}
+	   mountingYpos:=${cal_frame_mounting_ypos}
+	   mountingspacing:=${cal_frame_mounting_spacing}">
+		<link name="world"/>
+		<link name="${prefix}_frame">
+			<inertial>
+				<mass value="100.0" />
+				<origin xyz="0 1.2 0.3" rpy="0 0 0"/>
+				<inertia ixx="4.0" ixy="0" ixz="0" iyy="4.0" iyz="0" izz="4.0"/>
+			</inertial>
+			<!-- horizontal front bar-->
+			<xacro:bar thickness="${thickness}" len="${width}">
+				<origin xyz="0 ${-thickness/2} ${-thickness/2}" rpy="0 ${-pi/2} 0"/>
+			</xacro:bar>
+			<!-- horizontal rear bar -->
+			<xacro:bar thickness="${thickness}" len="${width}">
+				<origin xyz="0 ${depth+thickness/2} ${-thickness/2}" rpy="0 ${-pi/2} 0"/>
+			</xacro:bar>
+			<!-- robot mounting bars -->
+			<!-- horizontal front bar top -->
+			<xacro:bar thickness="${thickness}" len="${width}">
+				<origin xyz="0 ${mountingYpos-mountingspacing/2 + thickness/2} ${height+thickness/2}" rpy="0 ${-pi/2} 0"/>
+			</xacro:bar>
+			<!-- horizontal rear bar top -->
+			<xacro:bar thickness="${thickness}" len="${width}">
+				<origin xyz="0 ${mountingYpos+mountingspacing/2 - thickness/2} ${height+thickness/2}" rpy="0 ${-pi/2} 0"/>
+			</xacro:bar>
+			<!-- additional collision box inbetween the mounting bars at the top -->
+			<collision>
+				<origin xyz="0 ${mountingYpos} ${height+thickness/2}"
+				        rpy="0 0 0"/>
+				<geometry><box size="${width} ${mountingspacing-thickness} ${thickness}"/></geometry>
+			</collision>
+			<!-- left front pole -->
+			<xacro:bar thickness="${thickness}" len="${height+2*thickness+tableHeight}">
+				<origin xyz="${-(width+thickness)/2} ${-thickness/2} ${(height-tableHeight)/2}"/>
+			</xacro:bar>
+			<!-- right front pole -->
+			<xacro:bar thickness="${thickness}" len="${height+2*thickness+tableHeight}">
+				<origin xyz="${+(width+thickness)/2} ${-thickness/2} ${(height-tableHeight)/2}"/>
+			</xacro:bar>
+			<!-- left rear pole -->
+			<xacro:bar thickness="${thickness}" len="${height+2*thickness+tableHeight}">
+				<origin xyz="${-(width+thickness)/2} ${depth+thickness/2} ${(height-tableHeight)/2}"/>
+			</xacro:bar>
+			<!-- right rear pole -->
+			<xacro:bar thickness="${thickness}" len="${height+2*thickness+tableHeight}">
+				<origin xyz="${+(width+thickness)/2} ${depth+thickness/2} ${(height-tableHeight)/2}"/>
+			</xacro:bar>
+			<!-- left side bottom -->
+			<xacro:bar thickness="${thickness}" len="${depth}">
+				<origin xyz="${-(width+thickness)/2} ${depth/2} ${-thickness/2}"
+				        rpy="${-pi/2} 0 0"/>
+			</xacro:bar>
+			<!-- right side bottom -->
+			<xacro:bar thickness="${thickness}" len="${depth}">
+				<origin xyz="${+(width+thickness)/2} ${depth/2} ${-thickness/2}"
+				        rpy="${-pi/2} 0 0"/>
+			</xacro:bar>
+			<!-- left side top -->
+			<xacro:bar thickness="${thickness}" len="${depth}">
+				<origin xyz="${-(width+thickness)/2} ${depth/2} ${height+thickness/2}"
+				        rpy="${-pi/2} 0 0"/>
+			</xacro:bar>
+			<!-- right side top -->
+			<xacro:bar thickness="${thickness}" len="${depth}">
+				<origin xyz="${+(width+thickness)/2} ${depth/2} ${height+thickness/2}"
+				        rpy="${-pi/2} 0 0"/>
+			</xacro:bar>
+			<!-- table plane -->
+			<visual>
+				<origin xyz="0 ${depth/2} -0.01"
+				        rpy="0 0 0"/>
+				<geometry><box size="${width} ${depth} ${0.02}"/></geometry>
+				<material name="Silver"/>
+			</visual>
+			<collision>
+				<origin xyz="0 ${depth/2} -0.01"
+				        rpy="0 0 0"/>
+				<geometry><box size="${width} ${depth} ${0.02}"/></geometry>
+			</collision>
+			<!-- virtual fence -->
+			<!-- left pane -->
+			<collision>
+				<origin xyz="${-(width+thickness)/2} ${depth/2} ${height/2}"
+				        rpy="0 0 0"/>
+				<geometry><box size="${thickness} ${depth} ${height}"/></geometry>
+			</collision>
+			<!-- right pane -->
+			<collision>
+				<origin xyz="${+(width+thickness)/2} ${depth/2} ${height/2}"
+				        rpy="0 0 0"/>
+				<geometry><box size="${thickness} ${depth} ${height}"/></geometry>
+			</collision>
+			<!-- front pane -->
+			<collision>
+				<origin xyz="0 ${-thickness/2} ${height/2}"
+				        rpy="0 0 0"/>
+				<geometry><box size="${width} ${thickness} ${height}"/></geometry>
+			</collision>
+			<!-- back pane -->
+			<collision>
+				<origin xyz="0 ${depth + thickness/2} ${height/2}"
+				        rpy="0 0 0"/>
+				<geometry><box size="${width} ${thickness} ${height}"/></geometry>
+			</collision>
+			<!-- virtual protection box for the screens -->
+			<!-- right screen -->
+			<visual>
+				<origin xyz="${+0.575/2} ${mountingYpos-mountingspacing/2 -thickness} ${height+thickness/2}"
+				        rpy="0.32 0 0"/>
+				<geometry><box size="${0.550} ${0.07} ${0.35}"/></geometry>
+				<material name="Silver"/>
+			</visual>
+			<!-- left screen -->
+			<visual>
+				<origin xyz="${-0.575/2} ${mountingYpos-mountingspacing/2 -thickness} ${height+thickness/2}"
+				        rpy="0.32 0 0"/>
+				<geometry><box size="${0.550} ${0.07} ${0.35}"/></geometry>
+				<material name="Silver"/>
+			</visual>
+			<collision>
+				<origin xyz="0 ${mountingYpos-mountingspacing/2 -thickness} ${height+thickness/2}"
+				        rpy="0 0 0"/>
+				<geometry><box size="${0.575*2} ${0.250} ${0.350}"/></geometry>
+			</collision>
+		</link>
+		<joint name="${prefix}_frame_joint" type="fixed">
+			<origin xyz="0 0 0" rpy="0 0 0"/>
+			<parent link="world"/>
+			<child link="${prefix}_frame"/>
+		</joint>
+	</xacro:macro>
 </root>

File: agni_description/urdf/materials.urdf.xacro (robot description, xacro)
@@ -2,5 +2,5 @@
 <robot xmlns:xacro="http://www.ros.org/wiki/xacro">
   <material name="Silver">
-	 <color rgba="0.5 0.5 0.5 1.0"/>
+    <color rgba="0.5 0.5 0.5 1.0"/>
   </material>
   <material name="DarkGrey">
