Commit message: fixed cmake xacro generation

File: agni_description/robots/single.urdf.xacro (robot description, xacro)
@@ -2,9 +2,10 @@
 <robot name="single" xmlns:xacro="http://www.ros.org/wiki/xacro">
 	<xacro:property name="settings" value="${load_yaml('robots.yaml')}" />
-	<xacro:arg name="SIM" default="1"/>
-	<xacro:arg name="CALIB" default="$(arg FRAME)"/>
 	<xacro:arg name="FRAME" default="-"/>
 	<xacro:arg name="ARM" default="-"/>
 	<xacro:arg name="TOOL" default="-"/>
+	<xacro:arg name="PREFIX" default="-"/>
+	<xacro:arg name="SIM" default="1"/>
+	<xacro:arg name="CALIB" default="default"/>
 	<xacro:property name="parent" value="world"/>
 	<!-- FRAME -->
@@ -26,4 +27,6 @@
 	<xacro:include filename="../urdf/helpers.urdf.xacro" />
 	<!-- SINGLE ARM with TOOL -->
-	<xacro:arm_with_tool parent="${parent}" arm_type="$(arg ARM)" tool_type="$(arg TOOL)"/>
+	<xacro:property name="PREFIX" value="$(arg PREFIX)"/>
+	<xacro:arm_with_tool parent="${parent}" arm_type="$(arg ARM)" tool_type="$(arg TOOL)"
+	                     prefix="${PREFIX if PREFIX != '-' else ''}"/>
 </robot>

Commit message: Added the possibility to not connect single robot_description to world link (parent:='-')

File: agni_description/robots/single.urdf.xacro (robot description, xacro)
@@ -8,6 +8,9 @@
 	<xacro:arg name="ARM" default="-"/>
 	<xacro:arg name="TOOL" default="-"/>
-	<xacro:property name="parent" value="world"/>
-	<link name="${parent}"/>
+	<xacro:arg name="PARENT" default="world"/>
+	<xacro:property name="parent" value="$(arg PARENT)"/>
+	<xacro:if value="${parent != '-'}">
+		<link name="${parent}"/>
+	</xacro:if>
 	<!-- FRAME -->
 	<xacro:property name="FRAME" value="$(arg FRAME)"/>

File: agni_description/urdf/helpers.urdf.xacro (robot description, xacro)
@@ -9,9 +9,11 @@
                 prefix="${prefix}" controller="${controller}"/>
     <!-- attach arm to parent link -->
-    <joint name="${prefix_}arm_mount" type="fixed">
-      <parent link="${parent}"/>
-      <child link="${prefix_}arm_base_link"/>
-      <xacro:insert_block name="origin" />
-    </joint>
+    <xacro:if value="${parent != '-'}">
+      <joint name="${prefix_}arm_mount" type="fixed">
+        <parent link="${parent}"/>
+        <child link="${prefix_}arm_base_link"/>
+        <xacro:insert_block name="origin" />
+      </joint>
+    </xacro:if>
   </xacro:macro>
   <xacro:macro name="tool" params="type prefix:='' parent:='world' *origin">
@@ -23,9 +25,11 @@
                 prefix="${prefix}" />
     <!-- attach tool to parent link -->
-    <joint name="${prefix_}tool_mount" type="fixed">
-      <parent link="${parent}"/>
-      <child link="${prefix_}${settings['tools'][type]['mount']}"/>
-      <xacro:insert_block name="origin" />
-    </joint>
+    <xacro:if value="${parent != '-'}">
+      <joint name="${prefix_}tool_mount" type="fixed">
+        <parent link="${parent}"/>
+        <child link="${prefix_}${settings['tools'][type]['mount']}"/>
+        <xacro:insert_block name="origin" />
+      </joint>
+    </xacro:if>
   </xacro:macro>
   <!-- create arm + tool
@@ -43,5 +47,5 @@
     <xacro:property name="arm_prefix_" value="${arm_prefix + '_' if arm_prefix else ''}"/>
     <xacro:property name="tool_prefix_" value="${tool_prefix + '_' if tool_prefix else ''}"/>
-    <xacro:property name="tool_parent" value="world"/>
+    <xacro:property name="tool_parent" value="${parent}"/>
     <xacro:if value="${arm_type not in ['','-']}">
       <!-- load arm calibration and instantiate arm -->
