Commit message: moved world-link definition to top-level files (single, bimanual, sfb, famula)

File: agni_description/robots/bimanual.urdf.xacro (robot description, xacro)
@@ -3,5 +3,5 @@
 	<xacro:property name="settings" value="${load_yaml('robots.yaml')}" />
 	<xacro:arg name="SIM" default="1"/>
-	<xacro:arg name="CALIB" default="$(arg FRAME)"/>
+	<xacro:arg name="CALIB" default="default"/>
 	<xacro:arg name="FRAME" default="-"/>
 	<xacro:arg name="ARM_L" default="-"/>
@@ -10,4 +10,5 @@
 	<xacro:arg name="TOOL_R" default="-"/>
 	<xacro:property name="parent" value="world"/>
+	<link name="${parent}"/>
 	<!-- FRAME -->
 	<xacro:property name="FRAME" value="$(arg FRAME)"/>
@@ -21,10 +22,6 @@
 		</xacro:if>
 		<xacro:include filename="../calibration/${FRAME}_frame_cal.xml"/>
-		<xacro:frame/>
-		<xacro:property name="parent" value="frame"/>
+		<xacro:frame parent="${parent}"/>
 	</xacro:if>
-	<xacro:unless value="${FRAME not in ['', '-']}">
-		<link name="world"/>
-	</xacro:unless>
 	<xacro:include filename="../urdf/helpers.urdf.xacro" />
 	<!-- LEFT ARM with TOOL -->

File: agni_description/robots/famula.urdf.xacro (robot description, xacro)
@@ -4,8 +4,10 @@
 	<xacro:arg name="SIM" default="1"/>
 	<xacro:arg name="CALIB" default="famula"/>
+	<xacro:property name="parent" value="world"/>
+	<link name="${parent}"/>
 	<!-- frame -->
 	<xacro:include filename="../urdf/frame-half.urdf.xacro"/>
 	<xacro:include filename="../calibration/famula_frame_cal.xml"/>
-	<xacro:frame/>
+	<xacro:frame parent="${parent}"/>
 	<xacro:include filename="../urdf/helpers.urdf.xacro" />
 	<xacro:arm_with_tool parent="frame" prefix="r"

File: agni_description/robots/sfb.urdf.xacro (robot description, xacro)
@@ -4,8 +4,10 @@
 	<xacro:arg name="SIM" default="1"/>
 	<xacro:arg name="CALIB" default="sfb"/>
-	<!-- Frame -->
+	<xacro:property name="parent" value="world"/>
+	<link name="${parent}"/>
+	<!-- frame -->
 	<xacro:include filename="../urdf/frame.urdf.xacro"/>
 	<xacro:include filename="../calibration/sfb_frame_cal.xml"/>
-	<xacro:frame/>
+	<xacro:frame parent="${parent}"/>
 	<xacro:include filename="../urdf/helpers.urdf.xacro" />
 	<xacro:arm_with_tool parent="frame" prefix="r"

File: agni_description/robots/single.urdf.xacro (robot description, xacro)
@@ -2,11 +2,12 @@
 <robot name="single" xmlns:xacro="http://www.ros.org/wiki/xacro">
 	<xacro:property name="settings" value="${load_yaml('robots.yaml')}" />
+	<xacro:arg name="PREFIX" default="-"/>
+	<xacro:arg name="SIM" default="1"/>
+	<xacro:arg name="CALIB" default="default"/>
 	<xacro:arg name="FRAME" default="-"/>
 	<xacro:arg name="ARM" default="-"/>
 	<xacro:arg name="TOOL" default="-"/>
-	<xacro:arg name="PREFIX" default="-"/>
-	<xacro:arg name="SIM" default="1"/>
-	<xacro:arg name="CALIB" default="default"/>
 	<xacro:property name="parent" value="world"/>
+	<link name="${parent}"/>
 	<!-- FRAME -->
 	<xacro:property name="FRAME" value="$(arg FRAME)"/>
@@ -19,10 +20,6 @@
 		</xacro:if>
 		<xacro:include filename="../calibration/${FRAME}_frame_cal.xml"/>
-		<xacro:frame/>
-		<xacro:property name="parent" value="frame"/>
+		<xacro:frame parent="${parent}"/>
 	</xacro:if>
-	<xacro:unless value="${FRAME not in ['', '-']}">
-		<link name="world"/>
-	</xacro:unless>
 	<xacro:include filename="../urdf/helpers.urdf.xacro" />
 	<!-- SINGLE ARM with TOOL -->

File: agni_description/urdf/frame-half.urdf.xacro (robot description, xacro)
@@ -16,10 +16,10 @@
 		</collision>
 	</xacro:macro>
-	<xacro:macro name="frame" params="prefix:='' thickness:=${cal_frame_thick}
+	<xacro:macro name="frame" params="prefix:='' parent:=''
+	   thickness:=${cal_frame_thick}
 	   width:=${cal_frame_width} depth:=${cal_frame_depth} height:=${cal_frame_height}
 	   tableHeight:=${cal_frame_table_height} triangle_pos:=${cal_triangle_pos}">
 		<xacro:property name="mount_triangle_length" value="0.26" />
 		<xacro:property name="mount_triangle_thickness" value="0.02"/>
-		<link name="world"/>
 		<link name="${prefix}frame">
 			<inertial>
@@ -145,9 +145,11 @@
 			<material value="Gazebo/Grey"/>
 		</gazebo>
-		<joint name="${prefix}frame_joint" type="fixed">
-			<origin xyz="0 0 0" rpy="0 0 0"/>
-			<parent link="world"/>
-			<child link="${prefix}frame"/>
-		</joint>
+		<xacro:if value="${parent != ''}">
+			<joint name="${prefix}frame_joint" type="fixed">
+				<origin xyz="0 0 0" rpy="0 0 0"/>
+				<parent link="${parent}"/>
+				<child link="${prefix}frame"/>
+			</joint>
+		</xacro:if>
 	</xacro:macro>
 </root>

File: agni_description/urdf/frame.urdf.xacro (robot description, xacro)
@@ -20,10 +20,10 @@
 		</visual>
 	</xacro:macro>
-	<xacro:macro name="frame" params="prefix:='' thickness:=${cal_frame_thick}
+	<xacro:macro name="frame" params="prefix:='' parent:=''
+	   thickness:=${cal_frame_thick}
 	   width:=${cal_frame_width} depth:=${cal_frame_depth} height:=${cal_frame_height}
 	   tableHeight:=${cal_frame_table_height}
 	   mountingYpos:=${cal_frame_mounting_ypos}
 	   mountingspacing:=${cal_frame_mounting_spacing}">
-		<link name="world"/>
 		<link name="${prefix}frame">
 			<inertial>
@@ -149,9 +149,11 @@
 			</collision>
 		</link>
-		<joint name="${prefix}frame_joint" type="fixed">
-			<origin xyz="0 0 0" rpy="0 0 0"/>
-			<parent link="world"/>
-			<child link="${prefix}frame"/>
-		</joint>
+		<xacro:if value="${parent != ''}">
+			<joint name="${prefix}frame_joint" type="fixed">
+				<origin xyz="0 0 0" rpy="0 0 0"/>
+				<parent link="${parent}"/>
+				<child link="${prefix}frame"/>
+			</joint>
+		</xacro:if>
 	</xacro:macro>
 </root>

Commit message: determine CALIB from FRAME

File: agni_description/robots/bimanual.urdf.xacro (robot description, xacro)
@@ -2,6 +2,4 @@
 <robot name="bimanual" xmlns:xacro="http://www.ros.org/wiki/xacro">
 	<xacro:property name="settings" value="${load_yaml('robots.yaml')}" />
-	<xacro:arg name="SIM" default="1"/>
-	<xacro:arg name="CALIB" default="default"/>
 	<xacro:arg name="FRAME" default="-"/>
 	<xacro:arg name="ARM_L" default="-"/>
@@ -9,8 +7,12 @@
 	<xacro:arg name="TOOL_L" default="-"/>
 	<xacro:arg name="TOOL_R" default="-"/>
-	<xacro:property name="parent" value="world"/>
-	<link name="${parent}"/>
+	<xacro:arg name="PARENT" default="world"/>
+	<xacro:arg name="SIM" default="1"/>
+	<xacro:include filename="../urdf/CALIB.from.FRAME.xacro"/>
+	<xacro:property name="parent" value="$(arg PARENT)"/>
+	<xacro:if value="${parent not in ['', '-' ]}">
+		<link name="${parent}"/>
+	</xacro:if>
 	<!-- FRAME -->
-	<xacro:property name="FRAME" value="$(arg FRAME)"/>
 	<xacro:if value="${FRAME not in ['', '-']}">
 		<xacro:property name="FRAME" value="$(arg FRAME)"/>

File: agni_description/robots/single.urdf.xacro (robot description, xacro)
@@ -2,17 +2,16 @@
 <robot name="single" xmlns:xacro="http://www.ros.org/wiki/xacro">
 	<xacro:property name="settings" value="${load_yaml('robots.yaml')}" />
-	<xacro:arg name="PREFIX" default="-"/>
-	<xacro:arg name="SIM" default="1"/>
-	<xacro:arg name="CALIB" default="default"/>
 	<xacro:arg name="FRAME" default="-"/>
 	<xacro:arg name="ARM" default="-"/>
 	<xacro:arg name="TOOL" default="-"/>
 	<xacro:arg name="PARENT" default="world"/>
+	<xacro:arg name="PREFIX" default="-"/>
+	<xacro:arg name="SIM" default="1"/>
+	<xacro:include filename="../urdf/CALIB.from.FRAME.xacro"/>
 	<xacro:property name="parent" value="$(arg PARENT)"/>
-	<xacro:if value="${parent != '-'}">
+	<xacro:if value="${parent not in ['', '-' ]}">
 		<link name="${parent}"/>
 	</xacro:if>
 	<!-- FRAME -->
-	<xacro:property name="FRAME" value="$(arg FRAME)"/>
 	<xacro:if value="${FRAME not in ['', '-']}">
 		<xacro:if value="${FRAME == 'famula'}">
@@ -29,4 +28,4 @@
 	<xacro:property name="PREFIX" value="$(arg PREFIX)"/>
 	<xacro:arm_with_tool parent="${parent}" arm_type="$(arg ARM)" tool_type="$(arg TOOL)"
-	                     prefix="${PREFIX if PREFIX != '-' else ''}"/>
+	                     prefix="${PREFIX if PREFIX not in ['', '-'] else ''}"/>
 </robot>
