Commit message: Adapted poking stick after distal.tactile.xacro update

File: agni_description/robots/poking_stick.urdf.xacro (robot description, xacro)
@@ -7,10 +7,10 @@
     <xacro:poking_stick_generic prefix="${prefix_}" tactile="${props['tactile']}"/>
     <xacro:if value="${props['tactile'] in ['bio', 'ubi', 'eli']}">
-      <xacro:include filename="$(find sr_description)/hand/xacro/finger/distal/distal.tactile.xacro" />
+      <xacro:include filename="$(find sr_description)/hand/xacro/tactile.${props['tactile']}.xacro" />
       <!-- tactile marker mapping description -->
-      <xacro:distal_tactile bio="${props['tactile'] == 'bio'}"
-                            ubi="${props['tactile'] == 'ubi'}"
-                            eli="${props['tactile'] == 'eli'}"
-                            prefix="${prefix_}" link_prefix="ff" finger_number="0"/>
+      <xacro:property name="ns" value="${prefix_}"/>
+      <xacro:property name="xs" value="1023 0"/>
+      <xacro:property name="taxel_dir" value="$(find sr_description)/hand/xacro/finger"/>
+      <xacro:distal_tactile finger="ff" taxel_data="${load_yaml(taxel_dir + '/distal/distal.taxels.ubi.yaml')}"/>
     </xacro:if>
   </xacro:macro>

Commit message: Poking stick shoud use prefix not ns for tactile to work nice

File: agni_description/robots/poking_stick.urdf.xacro (robot description, xacro)
@@ -9,5 +9,5 @@
       <xacro:include filename="$(find sr_description)/hand/xacro/tactile.${props['tactile']}.xacro" />
       <!-- tactile marker mapping description -->
-      <xacro:property name="ns" value="${prefix_}"/>
+      <xacro:property name="prefix" value="${prefix_}"/>
       <xacro:property name="xs" value="1023 0"/>
       <xacro:property name="taxel_dir" value="$(find sr_description)/hand/xacro/finger"/>
