Commit message: Fixed lf parameter missing in shadow hand instantiation with ati

File: agni_description/robots/shadow_hand_ati.urdf.xacro (robot description, xacro)
@@ -7,5 +7,8 @@
                                           tactile:=${props.get('tactile','ubi')}
                                           side:=${props.get('side','right')}
-                                          prefix:=''">
+                                          prefix:=''
+                                          lf:=${props.get('lf','True')} ">
+    <xacro:property name="ns" value="${prefix}"/>
+    <xacro:property name="prefix_" value="${'' if prefix=='' else prefix+'_'}"/>
     <xacro:shadowhand muscletrans="${'trans' in model}"
                       muscle="${'muscle' in model}"
@@ -15,7 +18,7 @@
                       eli="${'eli' in tactile}"
                       reflect="${1 if side=='right' else -1}"
-                      prefix="${'' if prefix=='' else prefix+'_'}"  />
+                      prefix="${prefix_}"
+                      lf="${lf}" />
     <!-- add tool frame -->
-    <xacro:property name="prefix_" value="${'' if prefix=='' else prefix+'_'}"/>
     <joint name="${prefix_}tool_frame" type="fixed">
       <parent link="${prefix_}forearm"/>
@@ -26,5 +29,6 @@
     <!-- add tactile markers -->
     <xacro:shadowhand_tactile reflect="${1 if side=='right' else -1}"
-                              prefix="${'' if prefix=='' else prefix+'_'}" />
+                              prefix="${'' if prefix=='' else prefix+'_'}"
+                              lf="${lf}" />
     <!-- add ati sensor -->
     <xacro:include filename="../models/ati_sensor.urdf.xacro" />
