Commit message: Added a virtual fence that is deactivable for gazebo

File: agni_description/robots/moveable_famula.urdf.xacro (robot description, xacro)
@@ -9,5 +9,5 @@
 	<xacro:include filename="../urdf/frame-moveable.urdf.xacro"/>
 	<xacro:include filename="../calibration/moveable_famula_frame_cal.xml"/>
-	<xacro:frame parent="${parent}"/>
+	<xacro:frame parent="${parent}" use_virtual_fence="1" />
 	<xacro:include filename="../urdf/helpers.urdf.xacro" />
 	<xacro:arm_with_tool parent="frame" prefix="r"

File: agni_description/urdf/frame-moveable.urdf.xacro (robot description, xacro)
@@ -19,5 +19,5 @@
 	   thickness:=${cal_frame_thick} pole_front_dist:=${cal_frame_pole_front_dist}
 	   width:=${cal_frame_width} depth:=${cal_frame_depth} height:=${cal_frame_height}
-	   tableHeight:=${cal_frame_table_height} triangle_pos:=${cal_triangle_pos}">
+	   tableHeight:=${cal_frame_table_height} triangle_pos:=${cal_triangle_pos} use_virtual_fence:=0">
 		<xacro:property name="mount_triangle_length" value="0.26" />
 		<xacro:property name="mount_triangle_thickness" value="0.02"/>
@@ -83,4 +83,30 @@
 				<geometry><box size="${width} ${depth} ${0.02}"/></geometry>
 			</collision>
+			<xacro:if value="${use_virtual_fence}">
+				<!-- virtual fence -->
+				<!-- side plane -->
+				<collision>
+					<origin xyz="${-width/2} ${depth/2} ${height/2}"
+						rpy="0 0 0"/>
+					<geometry><box size="${0.02} ${depth} ${height}"/></geometry>
+				</collision>
+				<collision>
+					<origin xyz="${++width/2} ${depth/2} ${height/2}"
+						rpy="0 0 0"/>
+					<geometry><box size="${0.02} ${depth} ${height}"/></geometry>
+				</collision>
+				<!-- back plane -->
+				<collision>
+					<origin xyz="0 ${triangle_pos['Y'] + 0.2} ${height/2}"
+						rpy="0 0 0"/>
+					<geometry><box size="${width} ${0.02} ${height}"/></geometry>
+				</collision>
+				<!-- front plane -->
+				<collision>
+					<origin xyz="0 ${0-0.01} ${height/2}"
+						rpy="0 0 0"/>
+					<geometry><box size="${width} ${0.02} ${height}"/></geometry>
+				</collision>
+			</xacro:if>
 		</link>
 		<gazebo reference="${prefix}frame">
