Commit message: Fixed sdh mount (cable adapter and FCS were missing)

File: agni_description/robots/schunk_hand.urdf.xacro (robot description, xacro)
@@ -5,5 +5,33 @@
     <xacro:property name="prefix_" value="${'' if prefix=='' else prefix+'_'}"/>
     <link name="${prefix_}sdh_mount" />
-    <xacro:call macro="schunk_sdh" parent="${prefix_}sdh_mount" name="${prefix_}sdh" >
+     <!-- add cable adapter + female FCS part + red ring to schunk base frame -->
+    <xacro:property name="cable_fcs_adapter_thickness" value="0.02" />
+    <xacro:property name="cable_fcs_adapter_mass" value="0.030" />
+    <joint name="${prefix_}cable_adapter_joint" type="fixed">
+      <parent link="${prefix_}sdh_mount"/>
+      <child link="${prefix_}cable_adapter_frame"/>
+      <origin rpy="0 0 0" xyz="0.0 0.0 ${cable_fcs_adapter_thickness}"/>
+    </joint>
+    <link name="${prefix_}cable_adapter_frame" >
+      <inertial>
+        <mass value="${cable_fcs_adapter_mass}"/> <!-- estimated not measured -->
+        <origin xyz="0 0 ${-cable_fcs_adapter_thickness/2.0}"/>
+        <xacro:cylinder_inertia_def length="${cable_fcs_adapter_thickness}" radius="0.038" mass="${cable_fcs_adapter_mass}"/>
+      </inertial>
+      <visual>
+        <origin xyz="0 0 ${-cable_fcs_adapter_thickness/2.0}" rpy="0 0 0"/>
+        <geometry>
+           <cylinder radius="0.038" length="${cable_fcs_adapter_thickness}" />
+        </geometry>
+        <material name="Black"/>
+      </visual>
+      <collision>
+        <origin xyz="0 0 ${-cable_fcs_adapter_thickness/2.0}" rpy="0 0 0"/>
+        <geometry>
+          <cylinder radius="0.038" length="${cable_fcs_adapter_thickness}" />
+        </geometry>
+      </collision>
+    </link>
+    <xacro:call macro="schunk_sdh" parent="${prefix_}cable_adapter_frame" name="${prefix_}sdh" >
       <origin xyz="0 0 0" rpy="0 0 0"/>
     </xacro:call>

Commit message: Fixed schunk description (but controllers pid param loading still failing)

File: agni_description/robots/schunk_hand.urdf.xacro (robot description, xacro)
@@ -14,9 +14,8 @@
     </joint>
     <link name="${prefix_}cable_adapter_frame" >
-      <inertial>
-        <mass value="${cable_fcs_adapter_mass}"/> <!-- estimated not measured -->
+      <!-- mass estimated not measured -->
+      <xacro:cylinder_inertial length="${cable_fcs_adapter_thickness}" radius="0.038" mass="${cable_fcs_adapter_mass}">
         <origin xyz="0 0 ${-cable_fcs_adapter_thickness/2.0}"/>
-        <xacro:cylinder_inertia_def length="${cable_fcs_adapter_thickness}" radius="0.038" mass="${cable_fcs_adapter_mass}"/>
-      </inertial>
+      </xacro:cylinder_inertial>
       <visual>
         <origin xyz="0 0 ${-cable_fcs_adapter_thickness/2.0}" rpy="0 0 0"/>
