Commit message: cleanup srdf
- use chains and subgroups to compose groups
- added [rh|lh]_tool_frame to shadow hand (relative to arm's tool mount) to mimic Vortex' kinematics
- renamed groups *_armpalm to *_arm_palm
- added group [left|right]_arm_hand: includes both, arm and hand
- renamed group upper_body to both_arms_hand, added group both_arms_palm
- use *_fingers instead of *_hand as end-effector group and for parent group of *_fingers

File: agni_description/robots/shadow_hand.urdf.xacro (robot description, xacro)
@@ -15,4 +15,13 @@
                       reflect="${1 if side=='right' else -1}"
                       prefix="${'' if prefix=='' else prefix+'_'}"  />
+    <!-- add tool frame -->
+    <xacro:property name="prefix_" value="${'' if prefix=='' else prefix+'_'}"/>
+    <joint name="${prefix_}tool_frame" type="fixed">
+      <parent link="${prefix_.replace('h_', 'a_')}tool_mount"/>
+      <child link="${prefix_}tool_frame"/>
+      <!-- Hm. For some reason, the me files use an offset of 1cm -->
+      <origin rpy="${pi/2} 0 ${pi/2}" xyz="0.0 -0.01 0.327"/>
+    </joint>
+    <link name="${prefix_}tool_frame"/>
     <!-- add tactile markers -->
     <xacro:shadowhand_tactile reflect="${1 if side=='right' else -1}"

Commit message: fixed tool_frame for shadow hand
link to forearm instead of arm's tool mount

File: agni_description/robots/shadow_hand.urdf.xacro (robot description, xacro)
@@ -18,8 +18,7 @@
     <xacro:property name="prefix_" value="${'' if prefix=='' else prefix+'_'}"/>
     <joint name="${prefix_}tool_frame" type="fixed">
-      <parent link="${prefix_.replace('h_', 'a_')}tool_mount"/>
+      <parent link="${prefix_}forearm"/>
       <child link="${prefix_}tool_frame"/>
-      <!-- Hm. For some reason, the me files use an offset of 1cm -->
-      <origin rpy="${pi/2} 0 ${pi/2}" xyz="0.0 -0.01 0.327"/>
+      <origin rpy="${pi/2} 0 0" xyz="0.0 -0.01 0.327"/>
     </joint>
     <link name="${prefix_}tool_frame"/>

Commit message: Adapted agni_description to latest shadow code, before split (new gazebo_sim, new biotact)

File: agni_description/robots/shadow_hand.urdf.xacro (robot description, xacro)
@@ -11,4 +11,5 @@
                       muscle="${'muscle' in model}"
                       bio="${'bio' in tactile}"
+                      bt_sp="${'bt_stp' in tactile}"
                       ubi="${'ubi' in tactile}"
                       eli="${'eli' in tactile}"

File: agni_description/urdf/sr_gazebo.urdf.xacro (robot description, xacro)
@@ -2,9 +2,8 @@
 <robot xmlns:xacro="http://www.ros.org/wiki/xacro">
 	<!-- namespace must be set up according to launch file namespace -->
-  <xacro:macro name="shadow_gazebo_controller_manager" params="namespace">
+	<xacro:macro name="shadow_gazebo_controller_manager" params="namespace">
 		<gazebo>
-			<plugin name="sr_gazebo_ros_controller_manager" filename="libsr_gazebo_ros_controller_manager.so">
-				<alwaysOn>true</alwaysOn>
-				<updateRate>1000.0</updateRate>
+			<plugin name="gazebo_ros_control" filename="libgazebo_ros_control.so">
+				<robotSimType>sr_gazebo_sim/SrGazeboHWSim</robotSimType>
 				<robotNamespace>${namespace}</robotNamespace>
 			</plugin>

Commit message: Support namespace for tactile plugin in distal urdf

File: agni_description/robots/shadow_hand.urdf.xacro (robot description, xacro)
@@ -8,5 +8,7 @@
                                           side:=${props.get('side','right')}
                                           prefix:=''
-                                          lf:=${props.get('lf','True')}">
+                                          lf:=${props.get('lf','True')} ">
+    <xacro:property name="ns" value="${prefix}"/>
+    <xacro:property name="prefix_" value="${'' if prefix=='' else prefix+'_'}"/>
     <xacro:shadowhand muscletrans="${'trans' in model}"
                       muscle="${'muscle' in model}"
@@ -16,8 +18,7 @@
                       eli="${'eli' in tactile}"
                       reflect="${1 if side=='right' else -1}"
-                      prefix="${'' if prefix=='' else prefix+'_'}"
-                      lf="${lf}"  />
+                      prefix="${prefix_}"
+                      lf="${lf}" />
     <!-- add tool frame -->
-    <xacro:property name="prefix_" value="${'' if prefix=='' else prefix+'_'}"/>
     <joint name="${prefix_}tool_frame" type="fixed">
       <parent link="${prefix_}forearm"/>
@@ -28,5 +29,5 @@
     <!-- add tactile markers -->
     <xacro:shadowhand_tactile reflect="${1 if side=='right' else -1}"
-                              prefix="${'' if prefix=='' else prefix+'_'}"
+                              prefix="${prefix_}"
                               lf="${lf}" />
     <xacro:shadow_gazebo_controller_manager namespace="${prefix}" />

Commit message: Adapted sensor selection to newer sr_description

File: agni_description/robots/shadow_hand.urdf.xacro (robot description, xacro)
@@ -5,18 +5,17 @@
   <xacro:include filename="$(find sr_description)/hand/xacro/full_hand.tactile.xacro" />
   <xacro:macro name="shadow_hand" params="model:=${props.get('model','motor')}
-                                          tip_sensor:=${props.get('tip_sensor','ubi')}
-                                          mid_sensor:=${props.get('mid_sensor','ubi')}
-                                          prox_sensor:=${props.get('prox_sensor','ubi')}
+                                          tip_sensors:=${props.get('tip_sensor',['ubi','ubi','ubi','ubi','ubi'])}
+                                          mid_sensors:=${props.get('mid_sensor',['ubi','ubi','ubi','ubi','ubi'])}
+                                          prox_sensors:=${props.get('prox_sensor',['ubi','ubi','ubi','ubi','ubi'])}
                                           palm_sensor:=${props.get('palm_sensor','ubi_fabric')}
                                           side:=${props.get('side','right')}
-                                          prefix:=''
-                                          lf:=${props.get('lf','True')} ">
+                                          prefix:='' ">
     <xacro:property name="ns" value="${prefix}"/>
     <xacro:property name="prefix_" value="${'' if prefix=='' else prefix+'_'}"/>
-    <xacro:shadowhand muscletrans="${'trans' in model}"
-                      muscle="${'muscle' in model}"
-                      tip_sensor="${tip_sensor}"
-                      mid_sensor="${mid_sensor}"
-                      prox_sensor="${prox_sensor}"
+    <xacro:property name="hand_type" value="${'hand_e' if model=='motor' else 'hand_m' if model=='muscle' else model}"/>
+    <xacro:shadowhand hand_type="${hand_type}"
+                      tip_sensors="${tip_sensors}"
+                      mid_sensors="${mid_sensors}"
+                      prox_sensors="${prox_sensors}"
                       palm_sensor="${palm_sensor}"
                       reflect="${1 if side=='right' else -1}"
@@ -31,6 +30,5 @@
     <!-- add tactile markers -->
     <xacro:shadowhand_tactile reflect="${1 if side=='right' else -1}"
-                              prefix="${prefix_}"
-                              lf="${lf}" />
+                              prefix="${prefix_}"/>
     <xacro:shadow_gazebo_controller_manager namespace="${prefix}" />
   </xacro:macro>

File: agni_description/robots/shadow_hand_ati.urdf.xacro (robot description, xacro)
@@ -5,22 +5,20 @@
   <xacro:include filename="$(find sr_description)/hand/xacro/full_hand.tactile.xacro" />
   <xacro:macro name="shadow_hand" params="model:=${props.get('model','motor')}
-                                          tip_sensor:=${props.get('tip_sensor','ubi')}
-                                          mid_sensor:=${props.get('mid_sensor','ubi')}
-                                          prox_sensor:=${props.get('prox_sensor','ubi')}
+                                          tip_sensors:=${props.get('tip_sensor',['ubi','ubi','ubi','ubi','ubi'])}
+                                          mid_sensors:=${props.get('mid_sensor',['ubi','ubi','ubi','ubi','ubi'])}
+                                          prox_sensors:=${props.get('prox_sensor',['ubi','ubi','ubi','ubi','ubi'])}
                                           palm_sensor:=${props.get('palm_sensor','ubi_fabric')}
                                           side:=${props.get('side','right')}
-                                          prefix:=''
-                                          lf:=${props.get('lf','True')} ">
+                                          prefix:='' ">
     <xacro:property name="ns" value="${prefix}"/>
     <xacro:property name="prefix_" value="${'' if prefix=='' else prefix+'_'}"/>
-    <xacro:shadowhand muscletrans="${'trans' in model}"
-                      muscle="${'muscle' in model}"
-                      tip_sensor="${tip_sensor}"
-                      mid_sensor="${mid_sensor}"
-                      prox_sensor="${prox_sensor}"
+    <xacro:property name="hand_type" value="${'hand_e' if model=='motor' else 'hand_m' if model=='muscle' else model}"/>
+    <xacro:shadowhand hand_type="${hand_type}"
+                      tip_sensors="${tip_sensors}"
+                      mid_sensors="${mid_sensors}"
+                      prox_sensors="${prox_sensors}"
                       palm_sensor="${palm_sensor}"
                       reflect="${1 if side=='right' else -1}"
-                      prefix="${prefix_}"
-                      lf="${lf}" />
+                      prefix="${prefix_}" />
     <!-- add tool frame -->
     <joint name="${prefix_}tool_frame" type="fixed">
@@ -32,6 +30,5 @@
     <!-- add tactile markers -->
     <xacro:shadowhand_tactile reflect="${1 if side=='right' else -1}"
-                              prefix="${'' if prefix=='' else prefix+'_'}"
-                              lf="${lf}" />
+                              prefix="${'' if prefix=='' else prefix+'_'}" />
     <!-- add ati sensor with our special mount adaptor for kuka 0.0094 m thick -->
     <xacro:include filename="$(find ati_sensor_description)/urdf/ati_sensor.urdf.xacro" />
