Commit message: Fusion of real and sim arm done and checked Clean-up of unused files (replaced by others) Fixed kuka_lwr urdf (material unused) Fixed static transform publisher launch

File: agni_description/kuka/lwr.urdf.xacro (robot description, xacro)
@@ -38,5 +38,5 @@
     </link>
     <gazebo reference="${name}arm_base_link">
-      <material value="kuka-lwr.material"/>
+      <!--<material value="kuka-lwr.material"/>-->
     </gazebo>
     <joint name="${name}arm_0_joint" type="revolute">
@@ -80,5 +80,5 @@
     </link>
     <gazebo reference="${name}arm_1_link">
-      <material value="kuka-lwr.material"/>
+      <!--<material value="kuka-lwr.material"/>-->
     </gazebo>
     <joint name="${name}arm_1_joint" type="revolute">
@@ -123,5 +123,5 @@
     </link>
     <gazebo reference="${name}arm_2_link">
-      <material value="kuka-lwr.material"/>
+      <!--<material value="kuka-lwr.material"/>-->
     </gazebo>
     <joint name="${name}arm_2_joint" type="revolute">
@@ -166,5 +166,5 @@
     </link>
     <gazebo reference="${name}arm_3_link">
-      <material value="kuka-lwr.material"/>
+      <!--<material value="kuka-lwr.material"/>-->
     </gazebo>
     <joint name="${name}arm_3_joint" type="revolute">
@@ -209,5 +209,5 @@
     </link>
     <gazebo reference="${name}arm_4_link">
-      <material value="kuka-lwr.material"/>
+      <!--<material value="kuka-lwr.material"/>-->
     </gazebo>
     <joint name="${name}arm_4_joint" type="revolute">
@@ -252,5 +252,5 @@
     </link>
     <gazebo reference="${name}arm_5_link">
-      <material value="kuka-lwr.material"/>
+      <!--<material value="kuka-lwr.material"/>-->
     </gazebo>
     <joint name="${name}arm_5_joint" type="revolute">
@@ -295,5 +295,5 @@
     </link>
     <gazebo reference="${name}arm_6_link">
-      <material value="kuka-lwr.material"/>
+      <!--<material value="kuka-lwr.material"/>-->
     </gazebo>
     <joint name="${name}arm_6_joint" type="revolute">
@@ -338,5 +338,5 @@
     </link>
     <gazebo reference="${name}arm_7_link">
-      <material value="kuka-lwr.material"/>
+      <!--<material value="kuka-lwr.material"/>-->
     </gazebo>
     <joint name="${name}arm_hand_fixed_joint" type="fixed">

Commit message: Tried to unify all the robots and all the possible end-effectors, but problems remain on origin passing and ee selection

File: agni_description/kuka/lwr.urdf.xacro (robot description, xacro)
@@ -14,5 +14,5 @@
   <property name="arm_velocity_scale_factor" value="1"/>
   <!-- reflect is either 1 (for right arm) or -1 (for left arm) -->
-  <macro name="kuka_lwr_arm" params="name reflect tool_name">
+  <macro name="kuka_lwr_arm" params="name reflect tool_name:=''">
     <link name="${name}arm_base_link">
       <inertial>

File: agni_description/robots/right_kuka_shadow.urdf.xacro (robot description, xacro)
@@ -11,5 +11,5 @@
   <!-- parent is the frame the robot is fixed to -->
   <!-- origin is the position of the robot in this frame -->
-  <xacro:macro name="rightkukashadow" params="parent *origin prefix controller">
+  <xacro:macro name="rightkukashadow" params="parent *origin prefix muscle:=false controller">
     <!-- KUKA arm -->
     <xacro:kuka_lwr_arm name="ra_" reflect="1" tool_name=""/>
@@ -26,5 +26,5 @@
     <xacro:if value="${prefix}">
       <!-- Shadow Hands -->
-      <xacro:shadowhand muscletrans="false" muscle="false" bio="false" ubi="true" eli="false" reflect="1.0" prefix="rh_"  />
+      <xacro:shadowhand muscletrans="false" muscle="${muscle}" bio="false" ubi="true" eli="false" reflect="1.0" prefix="rh_"  />
       <!-- Link arm and hand -->
       <joint name="ra_arm_hand_mount" type="fixed">
@@ -35,5 +35,5 @@
     </xacro:if>
     <xacro:unless value="${prefix}">
-      <xacro:shadowhand muscletrans="false" muscle="false" bio="false" ubi="true" eli="false" reflect="1.0" prefix=""  />
+      <xacro:shadowhand muscletrans="false" muscle="${muscle}" bio="false" ubi="true" eli="false" reflect="1.0" prefix=""  />
       <!-- Shadow Hands -->
       <!-- Link arm and hand -->
