Commit message: Simplified xacros using more complex properties with python and dictionaries for nesting Adapted launch files to use them

File: agni_description/kuka/lwr_controllers.gazebo.xacro (robot description, xacro)
@@ -1,11 +1,15 @@
 <?xml version="1.0"?>
 <robot xmlns:xacro="http://www.ros.org/wiki/xacro">
+  <!-- default port value. do not modify here.
+       If not correct, redefine your own property and pass the values through macro param -->
+  <xacro:property name="port" value="${dict( right=49938, left=49940)}"/>
   <!-- namespace must be set up according to launch file namespace -->
   <!-- port is the port number for the FRI UDP connection (be aware that port+1 is also used) -->
-  <macro name="left_lwr_arm_gazebo_controller" params="namespace port">
+  <xacro:macro name="left_lwr_arm_gazebo_controller" params="namespace port:=$port['left']">
+    <xacro:property name="prefix"  value="${'' if namespace=='' else namespace+'_'}" />
 		<gazebo>
 			<plugin name="left_lwr_arm_controller" filename="liblwr_controller.so">
 				<alwaysOn>true</alwaysOn>
-				<robotPrefix>la</robotPrefix>
+				<robotPrefix>${prefix}</robotPrefix>
 				<robotNamespace>${namespace}</robotNamespace>
 				<remotePort>${port}</remotePort>
@@ -21,8 +25,8 @@
 			</plugin>
 		</gazebo>
-	</macro>
+	</xacro:macro>
 	<!-- namespace must be set up according to launch file namespace -->
   <!-- port is the port number for the FRI UDP connection (be aware that port+1 is also used) -->
-  <macro name="right_lwr_arm_gazebo_controller" params="namespace port">
+  <xacro:macro name="right_lwr_arm_gazebo_controller" params="namespace port:=$port['right']">
 		<gazebo>
 			<plugin name="right_lwr_arm_controller" filename="liblwr_controller.so">
@@ -42,4 +46,4 @@
 			</plugin>
 		</gazebo>
-	</macro>
+	</xacro:macro>
 </robot>

File: agni_description/models/myrmex_quick_mount.urdf.xacro (robot description, xacro)
@@ -1,5 +1,5 @@
 <?xml version="1.0"?>
 <robot name="myrmex_quick_mount" xmlns:xacro="http://www.ros.org/wiki/xacro">
-  <xacro:macro name="myrmex_quick_mount" params="prefix">
+  <xacro:macro name="myrmex_quick_mount" params="prefix tactile">
   <link name="${prefix}myrmex_quick_mount">
     <visual>

File: agni_description/models/poking_stick.urdf.xacro (robot description, xacro)
@@ -1,5 +1,5 @@
 <?xml version="1.0"?>
 <robot name="poking_stick" xmlns:xacro="http://www.ros.org/wiki/xacro">
-  <xacro:macro name="poking_stick" params="prefix">
+  <xacro:macro name="poking_stick" params="prefix tactile">
   <link name="${prefix}poking_stick">
     <visual>
@@ -7,6 +7,12 @@
           rpy="0 0 0"/>
       <geometry>
+        <xacro:if value="${'ubi' in tactile}">
+        <mesh scale="0.001 0.001 0.001"
+					 filename="package://agni_description/models/meshes/poking_stick_for_ubi.dae"/>
+        </xacro:if>
+        <xacro:unless value="${'ubi' in tactile}">
         <mesh scale="0.001 0.001 0.001"
 					 filename="package://agni_description/models/meshes/poking_stick.dae"/>
+        </xacro:unless>
       </geometry>
     </visual>
@@ -18,19 +24,55 @@
       </geometry>
     </collision>
-    <collision>
-      <origin xyz="0 0 0.08875"
-          rpy="0 0 0"/>
-      <geometry>
-        <cylinder radius="0.0075" length="0.1475"/>
-      </geometry>
-    </collision>
-    <collision>
-      <origin xyz="0 0 0.1625"
-          rpy="0 0 0"/>
-      <geometry>
-        <sphere radius="0.0075"/>
-      </geometry>
-    </collision>
+    <xacro:if value="${'ubi' in tactile}">
+      <collision>
+        <origin xyz="0 0 0.07375"
+            rpy="0 0 0"/>
+        <geometry>
+          <cylinder radius="0.0075" length="0.1445"/>
+        </geometry>
+      </collision>
+    </xacro:if>
+    <xacro:unless value="${'ubi' in tactile}">
+      <collision>
+        <origin xyz="0 0 0.08875"
+            rpy="0 0 0"/>
+        <geometry>
+          <cylinder radius="0.0075" length="0.1475"/>
+        </geometry>
+      </collision>
+      <collision>
+        <origin xyz="0 0 0.1625"
+            rpy="0 0 0"/>
+        <geometry>
+          <sphere radius="0.0075"/>
+        </geometry>
+      </collision>
+    </xacro:unless>
   </link>
+  <xacro:if value="${'ubi' in tactile}">
+    <joint name="${prefix}stick_to_ubi" type="fixed">
+      <origin xyz="0 0 0.13605" rpy="0 0 0"/>
+      <parent link="${prefix}poking_stick"/>
+      <child link="${prefix}ffdistal"/>
+    </joint>
+    <link name="${prefix}ffdistal">
+      <visual>
+        <origin xyz="0 0 0"
+            rpy="0 0 0"/>
+        <geometry>
+          <mesh scale="0.001 0.001 0.001"
+             filename="package://sr_description/hand/model/ubi_tactiles/ubi_tip_visual.dae"/>
+        </geometry>
+      </visual>
+      <collision>
+        <origin xyz="0 0 0"
+            rpy="0 0 0"/>
+        <geometry>
+          <mesh scale="0.001 0.001 0.001"
+             filename="package://sr_description/hand/model/ubi_tactiles/ubi_tip_collision.dae"/>
+        </geometry>
+      </collision>
+    </link>
+  </xacro:if>
   <gazebo reference="${prefix}poking_stick">
   </gazebo>

File: agni_description/robots/frame.urdf.xacro (robot description, xacro)
@@ -2,6 +2,6 @@
 <robot name="platform"
 		 xmlns:xacro="http://www.ros.org/wiki/xacro">
-  <xacro:arg name="ARM" default="kuka"/>
-  <xacro:include filename="$(find agni_description)/urdf/$(arg ARM)_frame.urdf.xacro"/>
-  <xacro:call macro="$(arg ARM)_frame" prefix="$(arg ARM)" />
+  <xacro:arg name="FRAME" default="kuka"/>
+  <xacro:include filename="$(find agni_description)/urdf/$(arg FRAME)_frame.urdf.xacro"/>
+  <xacro:call macro="$(arg FRAME)_frame" prefix="$(arg FRAME)" />
 </robot>

File: agni_description/robots/platforms.urdf.xacro (robot description, xacro)
@@ -3,11 +3,15 @@
   <xacro:arg name="ARM" default="kuka"/>
   <xacro:arg name="R" default="1"/>
-  <xacro:arg name="L" default="1"/>
-  <xacro:arg name="R_EE_TYPE" default="shadow_motor"/>
-  <xacro:arg name="L_EE_TYPE" default="shadow_motor"/>
+  <xacro:arg name="L" default="0"/>
+  <xacro:arg name="R_EE_TYPE" default="-"/>
+  <xacro:arg name="R_EE_MODEL" default="-"/>
   <xacro:arg name="R_EE_SIDE" default="right"/>
+  <xacro:arg name="R_EE_TACTILE" default="-"/>
+  <xacro:arg name="L_EE_TYPE" default="-"/>
+  <xacro:arg name="L_EE_MODEL" default=""/>
   <xacro:arg name="L_EE_SIDE" default="left"/>
+  <xacro:arg name="L_EE_TACTILE" default="-"/>
   <xacro:arg name="FLOBI" default="0"/>
-  <xacro:arg name="USE_PREFIX" default="true"/>
+  <xacro:arg name="SIM" default="1"/>
   <!-- USE_PREFIX [true|false] to tell to use prefix for the end-effector or not.
        Is mandatory if using two hands -->
@@ -30,52 +34,85 @@
   <!-- R_EE_TYPE and L_EE_TYPE are the names of the end-effectors
        mounted on right and left arms respectively -->
+  <!-- R_EE_MODEL and L_EE_MODEL are the model of the end-effectors
+       mounted on right and left arms respectively -->
   <!-- R_EE_SIDE and L_EE_SIDE are the variants of the end-effectors
        for right and left arms respectively
        Note a left hand can be mounted on the right arm
        with R_EE_SIDE:=left -->
-  <!-- file called right_<R_EE_TYPE>_ee.urdf.xacro should exist and provide
-        - a macro called <R_EE_SIDE>_<R_EE_TYPE>
-        - a property r_ee_base_link with the name of the attachement link
+  <!-- R_EE_TACTILE and L_EE_TACTILE define the type of tactile system of the end-effectors
+       mounted on right and left arms respectively -->
+  <!-- file called right_<R_EE_TYPE>.urdf.xacro should exist and provide
+        - a macro called <R_EE_TYPE> taking parameters model, tactile, side and prefix
+        - a property as a dictionary ee_mount['<R_EE_TYPE>'] with the name of the attachement link
           for this end-effector type
-        - offset properties cal_right_ee_x|y|z|yaw|pitch|roll of the mounting
-          part of this effector when attached at the right arm
-       The same for left
+        - offset properties as a dictionary cal_ee_x|y|z|yaw|pitch|roll['<R_EE_TYPE>']['left|right']
+          of the mounting part of this effector when attached on the arm
           -->
-  <!-- arm with end-effector -->
-  <xacro:include filename="$(find agni_description)/robots/$(arg ARM)_anytool.urdf.xacro" />
+  <xacro:include filename="$(find sr_description)/materials.urdf.xacro" />
+  <!-- arm -->
+  <xacro:include filename="$(find agni_description)/robots/$(arg ARM)_arm.urdf.xacro" />
+  <!-- frame -->
+  <xacro:include filename="$(find agni_description)/urdf/$(arg ARM)_frame.urdf.xacro"/>
   <!-- arm calibration -->
   <xacro:include filename="$(find agni_description)/calibration/$(arg ARM)_cal.xml"/>
-  <!-- right end-effector -->
-  <xacro:include filename="$(find agni_description)/robots/right_$(arg R_EE_TYPE)_ee.urdf.xacro" />
-  <!-- left enf-effector -->
-  <xacro:include filename="$(find agni_description)/robots/left_$(arg L_EE_TYPE)_ee.urdf.xacro" />
-  <!-- frame -->
-  <xacro:include filename="$(find agni_description)/urdf/$(arg ARM)_frame.urdf.xacro"/>
-  <!-- flobi -->
-  <xacro:include filename="$(find flobi_sim)/defs/xacro/flobiv3.urdf.xacro" />
   <!-- frame generation -->
   <xacro:call macro="$(arg ARM)_frame" prefix="$(arg ARM)" />
   <xacro:if value="$(arg R)">
-    <!-- right arm with a right end-effector (can be of type left if needed, but must profide r_ee_base_link and cal_right_ee_x|y|z|yaw|pitch|roll) -->
-    <xacro:arm_ee parent="$(arg ARM)_frame" arm="$(arg ARM)" prefix="r" is_right="1" ee_macro="$(arg R_EE_SIDE)_$(arg R_EE_TYPE)" ee_base_link="${r_ee_base_link}" use_prefix="$(arg USE_PREFIX)" controller="false">
-      <origin xyz="${cal_right_arm_x} ${cal_right_arm_y} ${cal_right_arm_z}"
-      rpy="${cal_right_arm_roll} ${cal_right_arm_pitch} ${cal_right_arm_yaw}"/>
-      <origin xyz="${cal_right_ee_x} ${cal_right_ee_y} ${cal_right_ee_z}"
-      rpy="${cal_right_ee_roll} ${cal_right_ee_pitch} ${cal_right_ee_yaw}"/>
-    </xacro:arm_ee>
+    <!-- Arm -->
+    <xacro:property name="arm"  value="$(arg ARM)" />
+    <xacro:call macro="${arm}_arm" parent="world" side="right" controller="$(arg SIM)">
+    <origin xyz="${cal_arm_x.get('right',0.0)} ${cal_arm_y.get('right',0.0)} ${cal_arm_z.get('right',0.0)}"
+      rpy="${cal_arm_roll.get('right',0.0)} ${cal_arm_pitch.get('right',0.0)} ${cal_arm_yaw.get('right',0.0)}"/>
+    </xacro:call>
+    <xacro:property name="r_ee_type" value="$(arg R_EE_TYPE)"/>
+    <xacro:property name="r_ee_side" value="$(arg R_EE_SIDE)"/>
+    <xacro:property name="r_ee_model" value="$(arg R_EE_MODEL)"/>
+    <xacro:property name="r_ee_prefix" value="${'rh' if r_ee_side=='right' else 'lh'}"/>
+    <xacro:property name="r_ee_tactile" value="$(arg R_EE_TACTILE)"/>
+    <xacro:if value="${r_ee_type!='-'}">
+     <!-- right end-effector -->
+      <xacro:include filename="$(find agni_description)/robots/${r_ee_type}_ee.urdf.xacro" />
+      <xacro:include filename="$(find agni_description)/calibration/${r_ee_type}${'_'+r_ee_model if r_ee_model!='-' else ''}_cal.xml"/>
+      <xacro:call macro="${r_ee_type}" model="$(arg R_EE_MODEL)" tactile="${r_ee_tactile if r_ee_tactile!='-' else ''}" side="${r_ee_side}" prefix="${r_ee_prefix}"/>
+     <!-- Link arm and effector -->
+      <joint name="ra_arm_hand_mount" type="fixed">
+        <parent link="ra_${arm_mount[arm]}"/>
+        <child link="${r_ee_prefix}_${ee_mount[r_ee_type]}"/>
+          <origin xyz="${cal_ee_x[r_ee_type].get(r_ee_side,0.0)} ${cal_ee_y[r_ee_type].get(r_ee_side,0.0)} ${cal_ee_z[r_ee_type].get(r_ee_side,0.0)}"
+        rpy="${cal_ee_roll[r_ee_type].get(r_ee_side,0.0)} ${cal_ee_pitch[r_ee_type].get(r_ee_side,0.0)} ${cal_ee_yaw[r_ee_type].get(r_ee_side,0.0)}"/>
+      </joint>
+    </xacro:if>
   </xacro:if>
   <xacro:if value="$(arg L)">
-    <!--left arm with a left end-effector (can be of type right if needed, but must profide l_ee_base_link and cal_left_ee_x|y|z|yaw|pitch|roll) -->
-    <xacro:arm_ee parent="$(arg ARM)_frame" arm="$(arg ARM)" prefix="l" is_right="0" ee_macro="$(arg L_EE_SIDE)_$(arg L_EE_TYPE)" ee_base_link="${l_ee_base_link}" use_prefix="$(arg USE_PREFIX)" controller="false">
-      <origin xyz="${cal_left_arm_x} ${cal_left_arm_y} ${cal_left_arm_z}"
-          rpy="${cal_left_arm_roll} ${cal_left_arm_pitch} ${cal_left_arm_yaw}"/>
-      <origin xyz="${cal_left_ee_x} ${cal_left_ee_y} ${cal_left_ee_z}"
-      rpy="${cal_left_ee_roll} ${cal_left_ee_pitch} ${cal_left_ee_yaw}"/>
-    </xacro:arm_ee>
+    <!-- Arm -->
+    <xacro:property name="arm"  value="$(arg ARM)" />
+    <xacro:call macro="${arm}_arm" parent="world" side="left" controller="$(arg SIM)">
+      <origin xyz="${cal_arm_x.get('left',0.0)} ${cal_arm_y.get('left',0.0)} ${cal_arm_z.get('left',0.0)}"
+      rpy="${cal_arm_roll.get('left',0.0)} ${cal_arm_pitch.get('left',0.0)} ${cal_arm_yaw.get('left',0.0)}"/>
+    </xacro:call>
+    <xacro:property name="l_ee_type" value="$(arg L_EE_TYPE)"/>
+    <xacro:property name="l_ee_side" value="$(arg L_EE_SIDE)"/>
+    <xacro:property name="l_ee_model" value="$(arg L_EE_MODEL)"/>
+    <xacro:property name="l_ee_prefix" value="${'rh' if l_ee_side=='right' else 'lh'}"/>
+    <xacro:property name="l_ee_tactile" value="$(arg L_EE_TACTILE)"/>
+    <xacro:if value="${l_ee_type!='-'}">
+     <!-- left end-effector -->
+      <xacro:include filename="$(find agni_description)/robots/${l_ee_type}_ee.urdf.xacro" />
+      <xacro:include filename="$(find agni_description)/calibration/${l_ee_type}${'_'+l_ee_model if l_ee_model!='-' else ''}_cal.xml"/>
+      <xacro:call macro="${l_ee_type}" model="$(arg L_EE_MODEL)" tactile="${l_ee_tactile if l_ee_tactile!='-' else ''}" side="${l_ee_side}" prefix="${l_ee_prefix}"/>
+     <!-- Link arm and effector -->
+      <joint name="la_arm_hand_mount" type="fixed">
+        <parent link="la_${arm_mount[arm]}"/>
+        <child link="${l_ee_prefix}_${ee_mount[l_ee_type]}"/>
+          <origin xyz="${cal_ee_x[l_ee_type].get(l_ee_side,0.0)} ${cal_ee_y[l_ee_type].get(l_ee_side,0.0)} ${cal_ee_z[l_ee_type].get(l_ee_side,0.0)}"
+      rpy="${cal_ee_roll[l_ee_type].get(l_ee_side,0.0)} ${cal_ee_pitch[l_ee_type].get(l_ee_side,0.0)} ${cal_ee_yaw[l_ee_type].get(l_ee_side,0.0)}"/>
+      </joint>
+    </xacro:if>
   </xacro:if>
   <xacro:if value="$(arg FLOBI)">
     <!-- flobi -->
+    <xacro:include filename="$(find flobi_sim)/defs/xacro/flobiv3.urdf.xacro" />
     <xacro:flobi prefix="" neutral="1" gender="0" parent="$(arg ARM)_frame" >
-      <origin xyz="0 ${cal_right_arm_y} ${cal_right_arm_z+mount_triangle_length/2*sin60+0.01}" rpy="0 0 ${-M_PI/2}"/>
+      <origin xyz="0 ${cal_arm_y['right']} ${cal_arm_z['right']+mount_triangle_length/2*sin(60/180.0*pi)+0.01}" rpy="0 0 ${-pi/2.0}"/>
     </xacro:flobi>
  </xacro:if>

File: agni_description/robots/sfb.urdf.xacro (robot description, xacro)
@@ -2,33 +2,42 @@
 <robot name="arm_hand_shadow" xmlns:xacro="http://www.ros.org/wiki/xacro">
   <xacro:arg name="SIM" default="1"/>
-  <!-- arm with end-effector
-  <xacro:include filename="$(find agni_description)/robots/$(arg ARM)_anytool.urdf.xacro" /> -->
-  <!-- arm calibration -->
-  <xacro:include filename="$(find agni_description)/calibration/$(arg ARM)_cal.xml"/>-->
+  <xacro:include filename="$(find agni_description)/urdf/pa10_frame.urdf.xacro"/>
+  <!-- arm  -->
+  <xacro:include filename="$(find agni_description)/robots/pa10_arm.urdf.xacro" />
   <!-- end-effector -->
-  <xacro:include filename="$(find agni_description)/robots/shadow_hand.urdf.xacro" />
-  <!-- must be world to spawn the arm in gazebo and have it fixed at the calibration location -->
-  <link name="world" />
-  <!-- arm and hand
-  <xacro:if value="$(arg IS_RIGHT)" >
-    <xacro:arm_ee parent="world" arm="$(arg ARM)" prefix="r" is_right="1" ee_macro="right_shadow_motor" ee_base_link="forearm" use_prefix="$(arg USE_PREFIX)" controller="$(arg SIM)">
-      <origin xyz="${cal_right_arm_x} ${cal_right_arm_y} ${cal_right_arm_z}"
-      rpy="${cal_right_arm_roll} ${cal_right_arm_pitch} ${cal_right_arm_yaw}"/>
-      <origin xyz="${cal_right_ee_x} ${cal_right_ee_y} ${cal_right_ee_z}"
-      rpy="${cal_right_ee_roll} ${cal_right_ee_pitch} ${cal_right_ee_yaw}"/>
-    </xacro:arm_ee>
-  </xacro:if>
-  <xacro:unless value="$(arg IS_RIGHT)" >
-    <xacro:arm_ee parent="world" arm="$(arg ARM)" prefix="l" is_right="0" ee_macro="left_shadow_motor" ee_base_link="forearm" use_prefix="$(arg USE_PREFIX)" controller="$(arg SIM)">
-      <origin xyz="${cal_left_arm_x} ${cal_left_arm_y} ${cal_left_arm_z}"
-          rpy="${cal_left_arm_roll} ${cal_left_arm_pitch} ${cal_left_arm_yaw}"/>
-      <origin xyz="${cal_left_ee_x} ${cal_left_ee_y} ${cal_left_ee_z}"
-      rpy="${cal_left_ee_roll} ${cal_left_ee_pitch} ${cal_left_ee_yaw}"/>
-    </xacro:arm_ee>
-  </xacro:unless>-->
-  <xacro:call macro="shadow_hand" model="motor" side="right" tactile="bio" prefix="lh">
-  </xacro:call>
-   <!--
-  <xacro:call macro="shadow_hand" model="motor" side="left" tactile="bio" prefix="lh">
-  </xacro:call>-->
+  <xacro:include filename="$(find agni_description)/robots/shadow_hand_ee.urdf.xacro" />
+  <!-- arm and hand mount calibration (should always be last) -->
+  <xacro:include filename="$(find agni_description)/calibration/sfb_cal.xml"/>
+  <!-- Frame -->
+  <xacro:call macro="pa10_frame" prefix="pa10" />
+  <!-- Right -->
+    <!-- Arm -->
+    <xacro:call macro="pa10_arm" parent="world" side="right" controller="$(arg SIM)">
+      <origin xyz="${cal_arm_x['right']} ${cal_arm_y['right']} ${cal_arm_z['right']}"
+      rpy="${cal_arm_roll['right']} ${cal_arm_pitch['right']} ${cal_arm_yaw['right']}"/>
+    </xacro:call>
+    <!-- Effector -->
+    <xacro:call macro="shadow_hand" model="motor" side="right" tactile="ubi" prefix="rh" />
+    <!-- Link arm and effector -->
+    <joint name="ra_arm_hand_mount" type="fixed">
+      <parent link="ra_${arm_mount['pa10']}"/>
+      <child link="rh_${ee_mount['shadow_hand']}"/>
+  <origin xyz="${cal_ee_x['shadow_hand']['right']} ${cal_ee_y['shadow_hand']['right']} ${cal_ee_z['shadow_hand']['right']}"
+  rpy="${cal_ee_roll['shadow_hand']['right']} ${cal_ee_pitch['shadow_hand']['right']} ${cal_ee_yaw['shadow_hand']['right']}"/>
+    </joint>
+  <!-- Left -->
+    <!-- Arm -->
+    <xacro:call macro="pa10_arm" parent="world" side="left" controller="$(arg SIM)">
+      <origin xyz="${cal_arm_x['left']} ${cal_arm_y['left']} ${cal_arm_z['left']}"
+      rpy="${cal_arm_roll['left']} ${cal_arm_pitch['left']} ${cal_arm_yaw['left']}"/>
+    </xacro:call>
+    <!-- Effector -->
+    <xacro:call macro="shadow_hand" model="motor" side="left" tactile="ubi" prefix="lh" />
+    <!-- Link arm and effector -->
+    <joint name="la_arm_hand_mount" type="fixed">
+      <parent link="la_${arm_mount['pa10']}"/>
+      <child link="lh_${ee_mount['shadow_hand']}"/>
+        <origin xyz="${cal_ee_x['shadow_hand']['left']} ${cal_ee_y['shadow_hand']['left']} ${cal_ee_z['shadow_hand']['left']}"
+  rpy="${cal_ee_roll['shadow_hand']['left']} ${cal_ee_pitch['shadow_hand']['left']} ${cal_ee_yaw['shadow_hand']['left']}"/>
+    </joint>
 </robot>

File: agni_description/urdf/frame-half.urdf.xacro (robot description, xacro)
@@ -7,7 +7,4 @@
 <xacro:include filename="$(find agni_description)/urdf/materials.urdf.xacro"/>
 <xacro:include filename="$(find agni_description)/calibration/kuka_cal.xml"/>
-  <property name="cos30"     value="0.866025404" />
-  <property name="sin30"     value="0.5" />
-  <property name="sin60"     value="0.866025404" />
   <property name="mount_triangle_length"     value="0.26" />
 <xacro:macro name="bar" params="thickness len *origin">
@@ -98,5 +95,5 @@
   <!-- kuka mount triangle -->
    <visual>
-     <origin xyz="${cal_left_arm_x-cos30*0.01} ${cal_left_arm_y} ${cal_left_arm_z-sin30*0.01}"
+     <origin xyz="${cal_arm_x['left']-cos(30/180.0*pi)*0.01} ${cal_arm_y['left']} ${cal_arm_z['left']-sin(30/180.0*pi)*0.01}"
         rpy="0 ${M_PI/3} 0"/>
     <geometry><box size="${mount_triangle_length} ${mount_triangle_length} ${0.02}"/></geometry>
@@ -104,10 +101,10 @@
    </visual>
    <collision>
-     <origin xyz="${cal_left_arm_x-cos30*0.01} ${cal_left_arm_y} ${cal_left_arm_z-sin30*0.01}"
+     <origin xyz="${cal_arm_x['left']-cos(30/180.0*pi)*0.01} ${cal_arm_y['left']} ${cal_arm_z['left']-sin(30/180.0*pi)*0.01}"
         rpy="0 ${M_PI/3} 0"/>
     <geometry><box size="${mount_triangle_length} ${mount_triangle_length} ${0.015}"/></geometry>
    </collision>
    <visual>
-     <origin xyz="${cal_right_arm_x+cos30*0.01} ${cal_right_arm_y} ${cal_right_arm_z-sin30*0.01}"
+     <origin xyz="${cal_arm_x['right']+cos(30/180.0*pi)*0.01} ${cal_arm_y['right']} ${cal_arm_z['right']-sin(30/180.0*pi)*0.01}"
         rpy="0 ${-M_PI/3} 0"/>
     <geometry><box size="${mount_triangle_length} ${mount_triangle_length} ${0.02}"/></geometry>
@@ -115,10 +112,10 @@
    </visual>
     <collision>
-       <origin xyz="${cal_right_arm_x+cos30*0.01} ${cal_right_arm_y} ${cal_right_arm_z-sin30*0.01}"
+       <origin xyz="${cal_arm_x['right']+cos(30/180.0*pi)*0.01} ${cal_arm_y['right']} ${cal_arm_z['right']-sin(30/180.0*pi)*0.01}"
         rpy="0 ${-M_PI/3} 0"/>
     <geometry><box size="${mount_triangle_length} ${mount_triangle_length} ${0.015}"/></geometry>
    </collision>
    <visual>
-     <origin xyz="0 ${cal_right_arm_y} ${cal_right_arm_z-sin30*0.02-mount_triangle_length/2*sin60-0.01}"
+     <origin xyz="0 ${cal_arm_y['right']} ${cal_arm_z['right']-sin(30/180.0*pi)*0.02-mount_triangle_length/2*sin(60/180.0*pi)-0.01}"
         rpy="0 0 0"/>
     <geometry><box size="${mount_triangle_length} ${mount_triangle_length} ${0.02}"/></geometry>
@@ -126,5 +123,5 @@
    </visual>
    <collision>
-      <origin xyz="0 ${cal_right_arm_y} ${cal_right_arm_z-sin30*0.02-mount_triangle_length/2*sin60-0.01}"
+      <origin xyz="0 ${cal_arm_y['right']} ${cal_arm_z['right']-sin(30/180.0*pi)*0.02-mount_triangle_length/2*sin(60/180.0*pi)-0.01}"
         rpy="0 0 0"/>
     <geometry><box size="${mount_triangle_length} ${mount_triangle_length} ${0.015}"/></geometry>

File: agni_description/urdf/kuka_frame.urdf.xacro (robot description, xacro)
@@ -8,4 +8,6 @@
     <xacro:property name="cal_frame_table_height"  value="1.00" />
   <xacro:macro name="kuka_frame" params="prefix">
+    <!-- arm calibration (local) -->
+    <xacro:include filename="$(find agni_description)/calibration/kuka_cal.xml"/>
     <xacro:frame-half prefix="${prefix}" thickness="${cal_frame_thick}" width="${cal_frame_width}" depth="${cal_frame_depth}"
               height="${cal_frame_height}" tableHeight="${cal_frame_table_height}"/>
