Commit message: Simplified xacros using more complex properties with python and dictionaries for nesting Adapted launch files to use them

File: agni_description/urdf/materials.urdf.xacro (robot description, xacro)
@@ -3,22 +3,4 @@
   <material name="Silver">
 	 <color rgba="0.5 0.5 0.5 1.0"/>
-  </material>
-  <material name="Red">
-    <color rgba="0.8 0.0 0.0 1.0"/>
-  </material>
-  <material name="Green">
-    <color rgba="0.0 0.8 0.0 1.0"/>
-  </material>
-  <material name="Blue">
-    <color rgba="0.0 0.0 0.8 1.0"/>
-  </material>
-  <material name="White">
-    <color rgba="1.0 1.0 1.0 1.0"/>
-  </material>
-  <material name="LightGrey">
-    <color rgba="0.6 0.6 0.6 1.0"/>
-  </material>
-  <material name="Grey">
-    <color rgba="0.2 0.2 0.2 1.0"/>
   </material>
   <material name="DarkGrey">

File: agni_description/urdf/pa10_frame.urdf.xacro (robot description, xacro)
@@ -2,6 +2,4 @@
 <root xmlns:xacro="http://www.ros.org/wiki/xacro">
   <xacro:include filename="$(find agni_description)/urdf/frame.urdf.xacro"/>
-  <!-- arm calibration -->
-  <xacro:include filename="$(find agni_description)/calibration/pa10_cal.xml"/>
   <xacro:property name="cal_frame_thick"  value="0.09" />
   <xacro:property name="cal_frame_width"     value="1.92" />
@@ -11,6 +9,8 @@
   <xacro:property name="cal_frame_mounting_spacing" value="0.513" />
   <xacro:macro name="pa10_frame" params="prefix">
+    <!-- arm calibration (local) -->
+    <xacro:include filename="$(find agni_description)/calibration/pa10_cal.xml"/>
     <xacro:frame prefix="${prefix}"  thickness="${cal_frame_thick}" width="${cal_frame_width}" depth="${cal_frame_depth}"
-              height="${cal_frame_height}" tableHeight="${cal_frame_table_height}" mountingYpos="${cal_right_arm_y}" mountingspacing="${cal_frame_mounting_spacing}" />
+              height="${cal_frame_height}" tableHeight="${cal_frame_table_height}" mountingYpos="${cal_arm_y.get('right',0.0)}" mountingspacing="${cal_frame_mounting_spacing}" />
   </xacro:macro>
 </root>

Commit message: Removed left|right|both files when possible and simplified arm|hand|arm_and_hand launch files Fixed FRAME arg Added conditional RTT motion_manager deploy Removed USE_PREFIX (use prefix everytime now) Only re-include xacro if effector type is different for left and right Added xacro pre-generation Fixed lwr_controller dictionary usage

File: agni_description/kuka/lwr_controllers.gazebo.xacro (robot description, xacro)
@@ -3,9 +3,9 @@
   <!-- default port value. do not modify here.
        If not correct, redefine your own property and pass the values through macro param -->
-  <xacro:property name="port" value="${dict( right=49938, left=49940)}"/>
+  <xacro:property name="portlist" value="${dict(right=49938, left=49940)}"/>
   <!-- namespace must be set up according to launch file namespace -->
   <!-- port is the port number for the FRI UDP connection (be aware that port+1 is also used) -->
-  <xacro:macro name="left_lwr_arm_gazebo_controller" params="namespace port:=$port['left']">
-    <xacro:property name="prefix"  value="${'' if namespace=='' else namespace+'_'}" />
+  <xacro:macro name="left_lwr_arm_gazebo_controller" params="namespace port:=${portlist['left']}">
+    <xacro:property name="prefix"  value="${'' if namespace=='' else namespace}" />
 		<gazebo>
 			<plugin name="left_lwr_arm_controller" filename="liblwr_controller.so">
@@ -28,5 +28,5 @@
 	<!-- namespace must be set up according to launch file namespace -->
   <!-- port is the port number for the FRI UDP connection (be aware that port+1 is also used) -->
-  <xacro:macro name="right_lwr_arm_gazebo_controller" params="namespace port:=$port['right']">
+  <xacro:macro name="right_lwr_arm_gazebo_controller" params="namespace port:=${portlist['right']}">
 		<gazebo>
 			<plugin name="right_lwr_arm_controller" filename="liblwr_controller.so">

File: agni_description/robots/arms.urdf.xacro (robot description, xacro)
@@ -7,4 +7,5 @@
   <xacro:include filename="$(find agni_description)/robots/$(arg ARM)_arm.urdf.xacro"/>
   <xacro:property name="side" value="$(arg SIDE)"/>
+  <xacro:include filename="$(find agni_description)/calibration/$(arg ARM)_cal.xml"/>
   <!-- must be world to spawn the arm in gazebo and have it fixed at the calibration location -->
   <link name="world" />

File: agni_description/robots/kuka_arm.urdf.xacro (robot description, xacro)
@@ -28,5 +28,5 @@
     <xacro:if value="${controller}">
       <!-- add controllers -->
-      <xacro:call macro="${side}_lwr_arm_gazebo_controller" namespace="${prefix}" port="$port['side']"/>
+      <xacro:call macro="${side}_lwr_arm_gazebo_controller" namespace="${prefix}" port="${portlist[side]}"/>
     </xacro:if>
   </xacro:macro>

File: agni_description/robots/platforms.urdf.xacro (robot description, xacro)
@@ -14,6 +14,4 @@
   <xacro:arg name="FLOBI" default="0"/>
   <xacro:arg name="SIM" default="1"/>
-  <!-- USE_PREFIX [true|false] to tell to use prefix for the end-effector or not.
-       Is mandatory if using two hands -->
   <!-- ARM to select the arm type.
        files called <ARM>.urdf.xacro and <ARM>_cal.xml should exist and provide
@@ -72,6 +70,6 @@
     <xacro:if value="${r_ee_type!='-'}">
      <!-- right end-effector -->
-      <xacro:include filename="$(find agni_description)/robots/${r_ee_type}_ee.urdf.xacro" />
-      <xacro:include filename="$(find agni_description)/calibration/${r_ee_type}${'_'+r_ee_model if r_ee_model!='-' else ''}_cal.xml"/>
+      <xacro:include filename="$(find agni_description)/robots/$(arg R_EE_TYPE)_ee.urdf.xacro" />
+      <xacro:include filename="$(find agni_description)/calibration/$(arg R_EE_TYPE)_$(arg R_EE_MODEL)_cal.xml"/>
       <xacro:call macro="${r_ee_type}" model="$(arg R_EE_MODEL)" tactile="${r_ee_tactile if r_ee_tactile!='-' else ''}" side="${r_ee_side}" prefix="${r_ee_prefix}"/>
      <!-- Link arm and effector -->
@@ -97,7 +95,9 @@
     <xacro:property name="l_ee_tactile" value="$(arg L_EE_TACTILE)"/>
     <xacro:if value="${l_ee_type!='-'}">
-     <!-- left end-effector -->
-      <xacro:include filename="$(find agni_description)/robots/${l_ee_type}_ee.urdf.xacro" />
-      <xacro:include filename="$(find agni_description)/calibration/${l_ee_type}${'_'+l_ee_model if l_ee_model!='-' else ''}_cal.xml"/>
+      <!-- left end-effector -->
+      <xacro:if value="${r_ee_type!=l_ee_type}">
+        <xacro:include filename="$(find agni_description)/robots/$(arg L_EE_TYPE)_ee.urdf.xacro" />
+        <xacro:include filename="$(find agni_description)/calibration/$(arg L_EE_TYPE)_$(arg L_EE_MODEL)_cal.xml"/>
+      </xacro:if>
       <xacro:call macro="${l_ee_type}" model="$(arg L_EE_MODEL)" tactile="${l_ee_tactile if l_ee_tactile!='-' else ''}" side="${l_ee_side}" prefix="${l_ee_prefix}"/>
      <!-- Link arm and effector -->

File: agni_description/robots/shadow_hand_ee.urdf.xacro (robot description, xacro)
@@ -13,5 +13,5 @@
   <xacro:property name="cal_ee_pitch" value="${dict(shadow_hand=dict(default=0.0))}" />
   <xacro:property name="cal_ee_roll" value="${dict(shadow_hand=dict(default=0.0))}" />
-  <xacro:macro name="shadow_hand" params="model:='motor' tactile:='ubi' side:='right' prefix:='rh'">
+  <xacro:macro name="shadow_hand" params="model:=motor tactile:=ubi side:=right prefix:=rh">
     <xacro:shadow_gazebo_controller_manager namespace="${prefix}" />
     <xacro:shadowhand muscletrans="${'trans' in model}"
