Commit message: Added intrinsic damping to kuka and pa10 urdf and fixed kuka inertia Exchanged kuka controller port to reflect real world Added shutdown timeout on pa10 controllers

File: agni_description/kuka/kuka.urdf.xacro (robot description, xacro)
@@ -53,4 +53,8 @@
       <child link="${name}arm_1_link"/>
     </joint>
+    <gazebo reference="${name}arm_0_joint">
+      <provideFeedback>1</provideFeedback>
+      <implicitSpringDamper>1</implicitSpringDamper>
+    </gazebo>
     <transmission name="${name}arm_0_trans" type="pr2_mechanism_model/SimpleTransmission">
       <actuator name="${name}arm_0_motor"/>
@@ -62,5 +66,5 @@
         <mass value="${arm_elem_link_mass}"/>
         <origin rpy="0 0 0" xyz="0 0 0.130"/>
-        <cuboid_inertia_def length="0.12" width="0.06" height="0.260"
+        <cuboid_inertia_def length="0.260" width="0.06" height="0.12"
                             mass="${arm_elem_link_mass}"/>
       </inertial>
@@ -95,4 +99,8 @@
       <child link="${name}arm_2_link"/>
     </joint>
+    <gazebo reference="${name}arm_1_joint">
+      <provideFeedback>1</provideFeedback>
+      <implicitSpringDamper>1</implicitSpringDamper>
+    </gazebo>
     <transmission name="${name}arm_1_trans" type="pr2_mechanism_model/SimpleTransmission">
       <actuator name="${name}arm_1_motor"/>
@@ -103,6 +111,6 @@
       <inertial>
         <mass value="${arm_elem_link_mass}"/>
-        <origin rpy="0 0 0" xyz="0 0.06 ${0.130 - 0.06}"/>
-        <cuboid_inertia_def length="0.12" width="0.06" height="0.260"
+        <origin rpy="0 0 0" xyz="0 -0.06 ${0.130 - 0.06}"/>
+        <cuboid_inertia_def length="0.260" width="0.06" height="0.12"
                             mass="${arm_elem_link_mass}"/>
       </inertial>
@@ -138,4 +146,8 @@
       <child link="${name}arm_3_link"/>
     </joint>
+    <gazebo reference="${name}arm_2_joint">
+      <provideFeedback>1</provideFeedback>
+      <implicitSpringDamper>1</implicitSpringDamper>
+    </gazebo>
     <transmission name="${name}arm_2_trans" type="pr2_mechanism_model/SimpleTransmission">
       <actuator name="${name}arm_2_motor"/>
@@ -146,6 +158,6 @@
       <inertial>
         <mass value="${arm_elem_link_mass}"/>
-        <origin rpy="0 0 0" xyz="0 0.06 0.130"/>
-        <cuboid_inertia_def length="0.12" width="0.06" height="0.260"
+        <origin rpy="0 0 0" xyz="0 -0.06 0.130"/>
+        <cuboid_inertia_def length="0.260" width="0.06" height="0.12"
                             mass="${arm_elem_link_mass}"/>
       </inertial>
@@ -181,4 +193,8 @@
       <child link="${name}arm_4_link"/>
     </joint>
+    <gazebo reference="${name}arm_3_joint">
+      <provideFeedback>1</provideFeedback>
+      <implicitSpringDamper>1</implicitSpringDamper>
+    </gazebo>
     <transmission name="${name}arm_3_trans" type="pr2_mechanism_model/SimpleTransmission">
       <actuator name="${name}arm_3_motor"/>
@@ -189,6 +205,6 @@
       <inertial>
         <mass value="${arm_elem_link_mass}"/>
-        <origin rpy="0 0 0" xyz="0 -0.06 ${0.130 - 0.06}"/>
-        <cuboid_inertia_def length="0.12" width="0.06" height="0.2600"
+        <origin rpy="0 0 0" xyz="0 0.06 ${0.130 - 0.06}"/>
+        <cuboid_inertia_def length="0.260" width="0.06" height="0.12"
                             mass="${arm_elem_link_mass}"/>
       </inertial>
@@ -224,4 +240,8 @@
       <child link="${name}arm_5_link"/>
     </joint>
+    <gazebo reference="${name}arm_4_joint">
+      <provideFeedback>1</provideFeedback>
+      <implicitSpringDamper>1</implicitSpringDamper>
+    </gazebo>
     <transmission name="${name}arm_4_trans" type="pr2_mechanism_model/SimpleTransmission">
       <actuator name="${name}arm_4_motor"/>
@@ -233,5 +253,5 @@
         <mass value="${arm_elem_link_mass}"/>
         <origin rpy="0 0 0" xyz="0 0 0.124"/>
-        <cuboid_inertia_def length="0.12" width="0.06" height="0.248"
+        <cuboid_inertia_def length="0.248" width="0.06" height="0.12"
                             mass="${arm_elem_link_mass}"/>
       </inertial>
@@ -267,4 +287,8 @@
       <child link="${name}arm_6_link"/>
     </joint>
+    <gazebo reference="${name}arm_5_joint">
+      <provideFeedback>1</provideFeedback>
+      <implicitSpringDamper>1</implicitSpringDamper>
+    </gazebo>
     <transmission name="${name}arm_5_trans" type="pr2_mechanism_model/SimpleTransmission">
       <actuator name="${name}arm_5_motor"/>
@@ -275,5 +299,5 @@
       <inertial>
         <mass value="${arm_elem_ball_link_mass}"/>
-        <origin rpy="0 0 0" xyz="0 0 0.0625"/>
+        <origin rpy="0 0 0" xyz="0 0 0.0"/>
         <cuboid_inertia_def length="0.125" width="0.125" height="0.125"
                             mass="${arm_elem_ball_link_mass}"/>
@@ -310,4 +334,8 @@
       <child link="${name}arm_7_link"/>
     </joint>
+    <gazebo reference="${name}arm_6_joint">
+      <provideFeedback>1</provideFeedback>
+      <implicitSpringDamper>1</implicitSpringDamper>
+    </gazebo>
     <transmission name="${name}arm_6_trans" type="pr2_mechanism_model/SimpleTransmission">
       <actuator name="${name}arm_6_motor"/>
@@ -319,5 +347,5 @@
         <mass value="${arm_elem_end_link_mass}"/>
         <origin xyz="0 0 0"/>
-        <cuboid_inertia_def length="1" width="1" height="1"
+        <cuboid_inertia_def length="0.02" width="0.06" height="0.06"
                             mass="${arm_elem_end_link_mass}"/>
       </inertial>

Commit message: Switched to larger damping and implicit damping in kuka Fixed collision at base Added gazeboAttach component and deployed it Fixed kuka port numbers to reflect real world

File: agni_description/kuka/kuka.urdf.xacro (robot description, xacro)
@@ -7,9 +7,9 @@
   <property name="arm_elem_base_mass" value="2.0"/>
   <property name="arm_elem_link_mass" value="2.0"/>
-  <property name="arm_elem_ball_link_mass" value="2.0"/>
-  <property name="arm_elem_end_link_mass" value="2.0"/>
+  <property name="arm_elem_ball_link_mass" value="1.0"/>
+  <property name="arm_elem_end_link_mass" value="0.2"/>
   <property name="safety_controller_k_pos" value="100" />
   <property name="safety_controller_k_vel" value="2" />
-  <property name="joint_damping" value="0.1" />
+  <property name="joint_damping" value="1.0" />
   <property name="arm_velocity_scale_factor" value="1"/>
   <!-- reflect is either 1 (for right arm) or -1 (for left arm) -->
@@ -31,7 +31,7 @@
       </visual>
       <collision>
-        <origin xyz="0 0 0" rpy="0 0 0"/>
-        <geometry>
-          <mesh filename="package://agni_description/kuka/meshes/convex/arm_base_convex.stl"/>
+        <origin xyz="0 0 0.01" rpy="0 0 0"/>
+        <geometry>
+          <mesh filename="package://agni_description/kuka/meshes/convex/arm_base_convex.stl" scale="0.9 0.9 0.9"/>
         </geometry>
       </collision>
@@ -79,5 +79,5 @@
         <origin xyz="0 0 0" rpy="0 0 ${M_PI}"/>
         <geometry>
-          <mesh filename="package://agni_description/kuka/meshes/convex/arm_segment_a_convex.stl"/>
+          <mesh filename="package://agni_description/kuka/meshes/convex/arm_segment_a_convex.stl" scale="1.0 1.0 1.0"/>
         </geometry>
       </collision>
@@ -126,5 +126,5 @@
         <origin xyz="0 0 0.2" rpy="${M_PI} 0 ${M_PI}"/>
         <geometry>
-          <mesh filename="package://agni_description/kuka/meshes/convex/arm_segment_b_convex.stl"/>
+          <mesh filename="package://agni_description/kuka/meshes/convex/arm_segment_b_convex.stl" scale="1.0 1.0 1.0"/>
         </geometry>
       </collision>
@@ -173,5 +173,5 @@
         <origin xyz="0 0 0" rpy="0 0 0"/>
         <geometry>
-          <mesh filename="package://agni_description/kuka/meshes/convex/arm_segment_a_convex.stl"/>
+          <mesh filename="package://agni_description/kuka/meshes/convex/arm_segment_a_convex.stl" scale="1.0 1.0 1.0"/>
         </geometry>
       </collision>
@@ -220,5 +220,5 @@
         <origin xyz="0 0 0.2" rpy="0 ${M_PI} ${M_PI}"/>
         <geometry>
-          <mesh filename="package://agni_description/kuka/meshes/convex/arm_segment_b_convex.stl"/>
+          <mesh filename="package://agni_description/kuka/meshes/convex/arm_segment_b_convex.stl" scale="1.0 1.0 1.0"/>
         </geometry>
       </collision>
@@ -267,5 +267,5 @@
         <origin xyz="0 0 0" rpy="0 0 ${M_PI}"/>
         <geometry>
-          <mesh filename="package://agni_description/kuka/meshes/convex/arm_segment_last_convex.stl"/>
+          <mesh filename="package://agni_description/kuka/meshes/convex/arm_segment_last_convex.stl" scale="1.0 1.0 1.0"/>
         </geometry>
       </collision>
@@ -314,5 +314,5 @@
         <origin xyz="0 0 0" rpy="0 0 ${M_PI}"/>
         <geometry>
-          <mesh filename="package://agni_description/kuka/meshes/convex/arm_wrist_convex.stl"/>
+          <mesh filename="package://agni_description/kuka/meshes/convex/arm_wrist_convex.stl" scale="1.0 1.0 1.0"/>
         </geometry>
       </collision>
@@ -361,5 +361,5 @@
         <origin xyz="0 0 0" rpy="0 0 ${reflect * -1/4 * M_PI  +  M_PI}"/>
         <geometry>
-          <mesh filename="package://agni_description/kuka/meshes/convex/arm_flanche${tool_name}_convex.stl"/>
+          <mesh filename="package://agni_description/kuka/meshes/convex/arm_flanche${tool_name}_convex.stl" scale="1.0 1.0 1.0"/>
         </geometry>
       </collision>

File: agni_description/robots/kuka_anytool.urdf.xacro (robot description, xacro)
@@ -27,8 +27,8 @@
       <!-- add controllers -->
         <xacro:if value="${is_right}" >
-          <xacro:right_lwr_arm_gazebo_controller namespace="${prefix}a" port="49940"/>
+          <xacro:right_lwr_arm_gazebo_controller namespace="${prefix}a" port="49938"/>
         </xacro:if>
         <xacro:unless value="${is_right}" >
-          <xacro:left_lwr_arm_gazebo_controller namespace="${prefix}a" port="49938"/>
+          <xacro:left_lwr_arm_gazebo_controller namespace="${prefix}a" port="49940"/>
         </xacro:unless>
     </xacro:if>

File: agni_description/urdf/frame-half.urdf.xacro (robot description, xacro)
@@ -106,5 +106,5 @@
      <origin xyz="${cal_left_arm_x-cos30*0.01} ${cal_left_arm_y} ${cal_left_arm_z-sin30*0.01}"
         rpy="0 ${M_PI/3} 0"/>
-    <geometry><box size="${mount_triangle_length} ${mount_triangle_length} ${0.02}"/></geometry>
+    <geometry><box size="${mount_triangle_length} ${mount_triangle_length} ${0.015}"/></geometry>
    </collision>
    <visual>
@@ -117,5 +117,5 @@
        <origin xyz="${cal_right_arm_x+cos30*0.01} ${cal_right_arm_y} ${cal_right_arm_z-sin30*0.01}"
         rpy="0 ${-M_PI/3} 0"/>
-    <geometry><box size="${mount_triangle_length} ${mount_triangle_length} ${0.02}"/></geometry>
+    <geometry><box size="${mount_triangle_length} ${mount_triangle_length} ${0.015}"/></geometry>
    </collision>
    <visual>
@@ -128,5 +128,5 @@
       <origin xyz="0 ${cal_right_arm_y} ${cal_right_arm_z-sin30*0.02-mount_triangle_length/2*sin60-0.01}"
         rpy="0 0 0"/>
-    <geometry><box size="${mount_triangle_length} ${mount_triangle_length} ${0.02}"/></geometry>
+    <geometry><box size="${mount_triangle_length} ${mount_triangle_length} ${0.015}"/></geometry>
    </collision>
   <!-- table plane -->

Commit message: added missing xacro: prefixes

File: agni_description/kuka/kuka.urdf.xacro (robot description, xacro)
@@ -5,14 +5,14 @@
        xmlns:interface="http://playerstage.sourceforge.net/gazebo/xmlschema/#interface">
   <xacro:include filename="$(find agni_description)/urdf/util.urdf.xacro"/>
-  <property name="arm_elem_base_mass" value="2.0"/>
-  <property name="arm_elem_link_mass" value="2.0"/>
-  <property name="arm_elem_ball_link_mass" value="1.0"/>
-  <property name="arm_elem_end_link_mass" value="0.2"/>
-  <property name="safety_controller_k_pos" value="100" />
-  <property name="safety_controller_k_vel" value="2" />
-  <property name="joint_damping" value="1.0" />
-  <property name="arm_velocity_scale_factor" value="1"/>
+  <xacro:property name="arm_elem_base_mass" value="2.0"/>
+  <xacro:property name="arm_elem_link_mass" value="2.0"/>
+  <xacro:property name="arm_elem_ball_link_mass" value="1.0"/>
+  <xacro:property name="arm_elem_end_link_mass" value="0.2"/>
+  <xacro:property name="safety_controller_k_pos" value="100" />
+  <xacro:property name="safety_controller_k_vel" value="2" />
+  <xacro:property name="joint_damping" value="1.0" />
+  <xacro:property name="arm_velocity_scale_factor" value="1"/>
   <!-- reflect is either 1 (for right arm) or -1 (for left arm) -->
-  <macro name="kuka_lwr_arm" params="name reflect tool_name:=''">
+  <xacro:macro name="kuka_lwr_arm" params="name reflect tool_name:=''">
     <link name="${name}arm_base_link">
       <inertial>
@@ -377,4 +377,4 @@
     </joint>
     <link name="${name}arm_hand_mount" />
-  </macro>
+  </xacro:macro>
 </robot>

File: agni_description/robots/kuka_arm.urdf.xacro (robot description, xacro)
@@ -22,5 +22,5 @@
     <xacro:kuka_lwr_arm name="${prefix}_" reflect="${1 if side=='right' else -1}" tool_name=""/>
     <joint name="${prefix}_frame_placement" type="fixed">
-       <insert_block name="origin" />
+       <xacro:insert_block name="origin" />
       <parent link="${parent}"/>
       <child link="${prefix}_arm_base_link"/>

File: agni_description/robots/pa10_arm.urdf.xacro (robot description, xacro)
@@ -24,5 +24,5 @@
     <xacro:call macro="${armname[side]}_arm" name="${prefix}_" />
     <joint name="${prefix}_frame_placement" type="fixed">
-      <insert_block name="origin" />
+      <xacro:insert_block name="origin" />
       <parent link="${parent}"/>
       <child link="${prefix}_arm_base_link"/>

File: agni_description/urdf/camera.urdf.xacro (robot description, xacro)
@@ -1,4 +1,4 @@
 <robot xmlns:xacro="http://ros.org/wiki/xacro">
-  <property name="M_PI" value="3.1415926535"/>
+  <xacro:property name="M_PI" value="3.1415926535"/>
   <!-- The reference frame is the depth optical frame, all other frames are built around it -->
   <xacro:include filename="$(find agni_description)/urdf/gazebo_camera.urdf.xacro"/>

File: agni_description/urdf/frame-half.urdf.xacro (robot description, xacro)
@@ -7,5 +7,5 @@
 <xacro:include filename="$(find agni_description)/urdf/materials.urdf.xacro"/>
 <xacro:include filename="$(find agni_description)/calibration/kuka_cal.xml"/>
-  <property name="mount_triangle_length"     value="0.26" />
+  <xacro:property name="mount_triangle_length"     value="0.26" />
 <xacro:macro name="bar" params="thickness len *origin">
    <visual>

File: agni_description/urdf/sr_gazebo.urdf.xacro (robot description, xacro)
@@ -2,5 +2,5 @@
 <robot xmlns:xacro="http://ros.org/wiki/xacro">
 	<!-- namespace must be set up according to launch file namespace -->
-  <macro name="shadow_gazebo_controller_manager" params="namespace">
+  <xacro:macro name="shadow_gazebo_controller_manager" params="namespace">
 		<gazebo>
 			<plugin name="sr_gazebo_ros_controller_manager" filename="libsr_gazebo_ros_controller_manager.so">
@@ -10,4 +10,4 @@
 			</plugin>
 		</gazebo>
-  </macro>
+  </xacro:macro>
 </robot>

File: agni_description/urdf/util.urdf.xacro (robot description, xacro)
@@ -1,21 +1,21 @@
 <?xml version="1.0"?>
 <robot xmlns:xacro="http://www.ros.org/wiki/xacro">
-  <property name="M_PI" value="3.1415926535897931"/>
+  <xacro:property name="M_PI" value="3.1415926535897931"/>
   <!--
 		Little helper macro to define the inertia matrix needed
 		for links.
   -->
-  <macro name="cuboid_inertia_def" params="width height length mass">
+  <xacro:macro name="cuboid_inertia_def" params="width height length mass">
     <inertia ixx="${mass * (height * height + length * length) / 12}"
              iyy="${mass * (width * width + length * length) / 12}"
              izz="${mass * (width * width + height * height) / 12}"
              ixy="0" iyz="0" ixz="0"/>
-  </macro>
+  </xacro:macro>
   <!-- length is along the y-axis! -->
-  <macro name="cylinder_inertia_def" params="radius length mass">
+  <xacro:macro name="cylinder_inertia_def" params="radius length mass">
     <inertia ixx="${mass * (3 * radius * radius + length * length) / 12}"
              iyy="${mass * radius* radius / 2}"
              izz="${mass * (3 * radius * radius + length * length) / 12}"
              ixy="0" iyz="0" ixz="0"/>
-  </macro>
+  </xacro:macro>
 </robot>
