Commit message: replace M_PI with pi

File: agni_description/kuka/kuka.urdf.xacro (robot description, xacro)
@@ -43,8 +43,8 @@
       <origin xyz="0 0 0.11" rpy="0 0 0"/>
       <axis xyz="0 0 1"/>
-      <limit lower="${-170 * M_PI / 180}" upper="${170 * M_PI / 180}"
-             effort="204" velocity="${arm_velocity_scale_factor * 110 * M_PI / 180}" />
-      <safety_controller soft_lower_limit="${-168 * M_PI / 180}"
-                         soft_upper_limit="${168 * M_PI / 180}"
+      <limit lower="${-170 * pi / 180}" upper="${170 * pi / 180}"
+             effort="204" velocity="${arm_velocity_scale_factor * 110 * pi / 180}" />
+      <safety_controller soft_lower_limit="${-168 * pi / 180}"
+                         soft_upper_limit="${168 * pi / 180}"
                          k_position="${safety_controller_k_pos}"
                          k_velocity="${safety_controller_k_vel}"/>
@@ -70,5 +70,5 @@
       </inertial>
       <visual>
-        <origin xyz="0 0 0" rpy="0 0 ${M_PI}"/>
+        <origin xyz="0 0 0" rpy="0 0 ${pi}"/>
         <geometry>
           <mesh scale="100 100 100"  filename="package://agni_description/kuka/meshes/arm_segment_a.dae"/>
@@ -77,5 +77,5 @@
       </visual>
       <collision>
-        <origin xyz="0 0 0" rpy="0 0 ${M_PI}"/>
+        <origin xyz="0 0 0" rpy="0 0 ${pi}"/>
         <geometry>
           <mesh filename="package://agni_description/kuka/meshes/convex/arm_segment_a_convex.stl" scale="1.0 1.0 1.0"/>
@@ -89,8 +89,8 @@
       <origin xyz="0 0 0.20" rpy="0 0 0"/>
       <axis xyz="0 -1 0"/>
-      <limit lower="${-120 * M_PI / 180}" upper="${120 * M_PI / 180}"
-             effort="306" velocity="${arm_velocity_scale_factor * 110 * M_PI / 180}" />
-      <safety_controller soft_lower_limit="${-118 * M_PI / 180}"
-                         soft_upper_limit="${118 * M_PI / 180}"
+      <limit lower="${-120 * pi / 180}" upper="${120 * pi / 180}"
+             effort="306" velocity="${arm_velocity_scale_factor * 110 * pi / 180}" />
+      <safety_controller soft_lower_limit="${-118 * pi / 180}"
+                         soft_upper_limit="${118 * pi / 180}"
                          k_position="${safety_controller_k_pos}"
                          k_velocity="${safety_controller_k_vel}"/>
@@ -116,5 +116,5 @@
       </inertial>
       <visual>
-        <origin xyz="0 0 0.2" rpy="${M_PI} 0 ${M_PI}"/>
+        <origin xyz="0 0 0.2" rpy="${pi} 0 ${pi}"/>
         <geometry>
           <mesh scale="100 100 100"
@@ -124,5 +124,5 @@
       </visual>
       <collision>
-        <origin xyz="0 0 0.2" rpy="${M_PI} 0 ${M_PI}"/>
+        <origin xyz="0 0 0.2" rpy="${pi} 0 ${pi}"/>
         <geometry>
           <mesh filename="package://agni_description/kuka/meshes/convex/arm_segment_b_convex.stl" scale="1.0 1.0 1.0"/>
@@ -136,8 +136,8 @@
       <origin xyz="0 0 0.20" rpy="0 0 0"/>
       <axis xyz="0 0 1"/>
-      <limit lower="${-170 * M_PI / 180}" upper="${170 * M_PI / 180}"
-             effort="204" velocity="${arm_velocity_scale_factor * 130 * M_PI / 180}" />
-      <safety_controller soft_lower_limit="${-168 * M_PI / 180}"
-                         soft_upper_limit="${168 * M_PI / 180}"
+      <limit lower="${-170 * pi / 180}" upper="${170 * pi / 180}"
+             effort="204" velocity="${arm_velocity_scale_factor * 130 * pi / 180}" />
+      <safety_controller soft_lower_limit="${-168 * pi / 180}"
+                         soft_upper_limit="${168 * pi / 180}"
                          k_position="${safety_controller_k_pos}"
                          k_velocity="${safety_controller_k_vel}"/>
@@ -183,8 +183,8 @@
       <origin xyz="0 0 0.20" rpy="0 0 0"/>
       <axis xyz="0 1 0"/>
-      <limit lower="${-120 * M_PI / 180}" upper="${120 * M_PI / 180}"
-             effort="306" velocity="${arm_velocity_scale_factor * 130 * M_PI / 180}" />
-      <safety_controller soft_lower_limit="${-118 * M_PI / 180}"
-                         soft_upper_limit="${118 * M_PI / 180}"
+      <limit lower="${-120 * pi / 180}" upper="${120 * pi / 180}"
+             effort="306" velocity="${arm_velocity_scale_factor * 130 * pi / 180}" />
+      <safety_controller soft_lower_limit="${-118 * pi / 180}"
+                         soft_upper_limit="${118 * pi / 180}"
                          k_position="${safety_controller_k_pos}"
                          k_velocity="${safety_controller_k_vel}"/>
@@ -210,5 +210,5 @@
       </inertial>
       <visual>
-        <origin xyz="0 0 0.2" rpy="0 ${M_PI} ${M_PI}"/>
+        <origin xyz="0 0 0.2" rpy="0 ${pi} ${pi}"/>
         <geometry>
           <mesh scale="100 100 100"
@@ -218,5 +218,5 @@
       </visual>
       <collision>
-        <origin xyz="0 0 0.2" rpy="0 ${M_PI} ${M_PI}"/>
+        <origin xyz="0 0 0.2" rpy="0 ${pi} ${pi}"/>
         <geometry>
           <mesh filename="package://agni_description/kuka/meshes/convex/arm_segment_b_convex.stl" scale="1.0 1.0 1.0"/>
@@ -230,8 +230,8 @@
       <origin xyz="0 0 0.20" rpy="0 0 0"/>
       <axis xyz="0 0 1"/>
-      <limit lower="${-170 * M_PI / 180}" upper="${170 * M_PI / 180}"
-             effort="204" velocity="${arm_velocity_scale_factor * 130 * M_PI / 180}" />
-      <safety_controller soft_lower_limit="${-168 * M_PI / 180}"
-                         soft_upper_limit="${168 * M_PI / 180}"
+      <limit lower="${-170 * pi / 180}" upper="${170 * pi / 180}"
+             effort="204" velocity="${arm_velocity_scale_factor * 130 * pi / 180}" />
+      <safety_controller soft_lower_limit="${-168 * pi / 180}"
+                         soft_upper_limit="${168 * pi / 180}"
                          k_position="${safety_controller_k_pos}"
                          k_velocity="${safety_controller_k_vel}"/>
@@ -257,5 +257,5 @@
       </inertial>
       <visual>
-        <origin xyz="0 0 0" rpy="0 0 ${M_PI}"/>
+        <origin xyz="0 0 0" rpy="0 0 ${pi}"/>
         <geometry name="${name}arm_5_geom">
           <mesh scale="100 100 100"
@@ -265,5 +265,5 @@
       </visual>
       <collision>
-        <origin xyz="0 0 0" rpy="0 0 ${M_PI}"/>
+        <origin xyz="0 0 0" rpy="0 0 ${pi}"/>
         <geometry>
           <mesh filename="package://agni_description/kuka/meshes/convex/arm_segment_last_convex.stl" scale="1.0 1.0 1.0"/>
@@ -277,8 +277,8 @@
       <origin xyz="0 0 0.19" rpy="0 0 0"/>
       <axis xyz="0 -1 0"/>
-      <limit lower="${-120 * M_PI / 180}" upper="${120 * M_PI / 180}"
-             effort="306" velocity="${arm_velocity_scale_factor * 180 * M_PI / 180}" />
-      <safety_controller soft_lower_limit="${-118 * M_PI / 180}"
-                         soft_upper_limit="${118 * M_PI / 180}"
+      <limit lower="${-120 * pi / 180}" upper="${120 * pi / 180}"
+             effort="306" velocity="${arm_velocity_scale_factor * 180 * pi / 180}" />
+      <safety_controller soft_lower_limit="${-118 * pi / 180}"
+                         soft_upper_limit="${118 * pi / 180}"
                          k_position="${safety_controller_k_pos}"
                          k_velocity="${safety_controller_k_vel}"/>
@@ -304,5 +304,5 @@
       </inertial>
       <visual>
-        <origin xyz="0 0 0" rpy="0 0 ${M_PI}"/>
+        <origin xyz="0 0 0" rpy="0 0 ${pi}"/>
         <geometry>
           <mesh scale="100 100 100"
@@ -312,5 +312,5 @@
       </visual>
       <collision>
-        <origin xyz="0 0 0" rpy="0 0 ${M_PI}"/>
+        <origin xyz="0 0 0" rpy="0 0 ${pi}"/>
         <geometry>
           <mesh filename="package://agni_description/kuka/meshes/convex/arm_wrist_convex.stl" scale="1.0 1.0 1.0"/>
@@ -324,8 +324,8 @@
       <origin xyz="0 0 0.078" rpy="0 0 0"/>
       <axis xyz="0 0 1"/>
-      <limit lower="${-170 * M_PI / 180}" upper="${170 * M_PI / 180}"
-             effort="204" velocity="${arm_velocity_scale_factor * 180 * M_PI / 180}" />
-      <safety_controller soft_lower_limit="${-168 * M_PI / 180}"
-                         soft_upper_limit="${168 * M_PI / 180}"
+      <limit lower="${-170 * pi / 180}" upper="${170 * pi / 180}"
+             effort="204" velocity="${arm_velocity_scale_factor * 180 * pi / 180}" />
+      <safety_controller soft_lower_limit="${-168 * pi / 180}"
+                         soft_upper_limit="${168 * pi / 180}"
                          k_position="${safety_controller_k_pos}"
                          k_velocity="${safety_controller_k_vel}"/>
@@ -351,5 +351,5 @@
       </inertial>
       <visual>
-        <origin xyz="0 0 0" rpy="0 0 ${reflect * -1/4 * M_PI  +  M_PI}"/>
+        <origin xyz="0 0 0" rpy="0 0 ${reflect * -1/4 * pi  +  pi}"/>
         <geometry>
           <mesh scale="100 100 100"
@@ -359,5 +359,5 @@
       </visual>
       <collision>
-        <origin xyz="0 0 0" rpy="0 0 ${reflect * -1/4 * M_PI  +  M_PI}"/>
+        <origin xyz="0 0 0" rpy="0 0 ${reflect * -1/4 * pi  +  pi}"/>
         <geometry>
           <mesh filename="package://agni_description/kuka/meshes/convex/arm_flanche${tool_name}_convex.stl" scale="1.0 1.0 1.0"/>
@@ -371,5 +371,5 @@
 <!--
       <origin xyz="${-reflect * 0.075} -0.075 -0.094"
-              rpy="${0.5*reflect*M_PI} 0 ${(1.5 + 0.25*reflect)*M_PI}"/>
+              rpy="${0.5*reflect*pi} 0 ${(1.5 + 0.25*reflect)*pi}"/>
 -->
       <parent link="${name}arm_7_link"/>

File: agni_description/urdf/camera.urdf.xacro (robot description, xacro)
@@ -1,4 +1,3 @@
 <robot xmlns:xacro="http://ros.org/wiki/xacro">
-  <xacro:property name="M_PI" value="3.1415926535"/>
   <!-- The reference frame is the depth optical frame, all other frames are built around it -->
   <xacro:include filename="$(find agni_description)/urdf/gazebo_camera.urdf.xacro"/>
@@ -21,5 +20,5 @@
     </link>
     <joint name="${name}_camera_depth_joint" type="fixed">
-      <origin xyz="0 0 0" rpy="${M_PI/2} ${-M_PI/2} 0 " />
+      <origin xyz="0 0 0" rpy="${pi/2} ${-pi/2} 0 " />
       <parent link="${name}_camera_depth_optical_frame" />
       <child link="${name}_camera_depth_frame" />
@@ -75,5 +74,5 @@
     </link>
     <joint name="${name}_camera_rgb_optical_joint" type="fixed">
-      <origin xyz="0 0 0" rpy="${-M_PI/2} 0 ${-M_PI/2}" />
+      <origin xyz="0 0 0" rpy="${-pi/2} 0 ${-pi/2}" />
       <parent link="${name}_camera_rgb_frame" />
       <child link="${name}_camera_rgb_optical_frame" />

File: agni_description/urdf/frame-half.urdf.xacro (robot description, xacro)
@@ -29,13 +29,13 @@
    <!-- horizontal front bar-->
    <xacro:bar thickness="${thickness}" len="${width}">
-    <origin xyz="0 ${thickness/2} ${-thickness/2}" rpy="0 ${-M_PI/2} 0"/>
+    <origin xyz="0 ${thickness/2} ${-thickness/2}" rpy="0 ${-pi/2} 0"/>
    </xacro:bar>
    <!-- horizontal rear bar -->
    <xacro:bar thickness="${thickness}" len="${width}">
-    <origin xyz="0 ${depth+thickness/2} ${-thickness/2}" rpy="0 ${-M_PI/2} 0"/>
+    <origin xyz="0 ${depth+thickness/2} ${-thickness/2}" rpy="0 ${-pi/2} 0"/>
    </xacro:bar>
    <!-- horizontal rear bar top -->
    <xacro:bar thickness="${thickness}" len="${width}">
-    <origin xyz="0 ${depth+thickness/2} ${height+thickness/2}" rpy="0 ${-M_PI/2} 0"/>
+    <origin xyz="0 ${depth+thickness/2} ${height+thickness/2}" rpy="0 ${-pi/2} 0"/>
    </xacro:bar>
    <!-- left front pole -->
@@ -58,10 +58,10 @@
    <xacro:bar thickness="${thickness}" len="${depth}">
     <origin xyz="${-(width+thickness)/2} ${depth/2} ${-thickness/2}"
-          rpy="${-M_PI/2} 0 0"/>
+          rpy="${-pi/2} 0 0"/>
    </xacro:bar>
    <!-- right side bottom -->
    <xacro:bar thickness="${thickness}" len="${depth}">
     <origin xyz="${+(width+thickness)/2} ${depth/2} ${-thickness/2}"
-          rpy="${-M_PI/2} 0 0"/>
+          rpy="${-pi/2} 0 0"/>
    </xacro:bar>
    <!-- left central pole -->
@@ -96,5 +96,5 @@
    <visual>
      <origin xyz="${cal_arm_x['left']-cos(30/180.0*pi)*0.01} ${cal_arm_y['left']} ${cal_arm_z['left']-sin(30/180.0*pi)*0.01}"
-        rpy="0 ${M_PI/3} 0"/>
+        rpy="0 ${pi/3} 0"/>
     <geometry><box size="${mount_triangle_length} ${mount_triangle_length} ${0.02}"/></geometry>
     <material name="Silver"/>
@@ -102,10 +102,10 @@
    <collision>
      <origin xyz="${cal_arm_x['left']-cos(30/180.0*pi)*0.01} ${cal_arm_y['left']} ${cal_arm_z['left']-sin(30/180.0*pi)*0.01}"
-        rpy="0 ${M_PI/3} 0"/>
+        rpy="0 ${pi/3} 0"/>
     <geometry><box size="${mount_triangle_length} ${mount_triangle_length} ${0.015}"/></geometry>
    </collision>
    <visual>
      <origin xyz="${cal_arm_x['right']+cos(30/180.0*pi)*0.01} ${cal_arm_y['right']} ${cal_arm_z['right']-sin(30/180.0*pi)*0.01}"
-        rpy="0 ${-M_PI/3} 0"/>
+        rpy="0 ${-pi/3} 0"/>
     <geometry><box size="${mount_triangle_length} ${mount_triangle_length} ${0.02}"/></geometry>
     <material name="Silver"/>
@@ -113,5 +113,5 @@
     <collision>
        <origin xyz="${cal_arm_x['right']+cos(30/180.0*pi)*0.01} ${cal_arm_y['right']} ${cal_arm_z['right']-sin(30/180.0*pi)*0.01}"
-        rpy="0 ${-M_PI/3} 0"/>
+        rpy="0 ${-pi/3} 0"/>
     <geometry><box size="${mount_triangle_length} ${mount_triangle_length} ${0.015}"/></geometry>
    </collision>

File: agni_description/urdf/frame.urdf.xacro (robot description, xacro)
@@ -31,18 +31,18 @@
 	 <!-- horizontal front bar-->
 	 <xacro:bar thickness="${thickness}" len="${width}">
-		<origin xyz="0 ${-thickness/2} ${-thickness/2}" rpy="0 ${-M_PI/2} 0"/>
+		<origin xyz="0 ${-thickness/2} ${-thickness/2}" rpy="0 ${-pi/2} 0"/>
 	 </xacro:bar>
 	 <!-- horizontal rear bar -->
 	 <xacro:bar thickness="${thickness}" len="${width}">
-		<origin xyz="0 ${depth+thickness/2} ${-thickness/2}" rpy="0 ${-M_PI/2} 0"/>
+		<origin xyz="0 ${depth+thickness/2} ${-thickness/2}" rpy="0 ${-pi/2} 0"/>
 	 </xacro:bar>
     <!-- robot mounting bars -->
 	 <!-- horizontal front bar top -->
 	 <xacro:bar thickness="${thickness}" len="${width}">
-		<origin xyz="0 ${mountingYpos-mountingspacing/2 + thickness/2} ${height+thickness/2}" rpy="0 ${-M_PI/2} 0"/>
+		<origin xyz="0 ${mountingYpos-mountingspacing/2 + thickness/2} ${height+thickness/2}" rpy="0 ${-pi/2} 0"/>
 	 </xacro:bar>
 	 <!-- horizontal rear bar top -->
 	 <xacro:bar thickness="${thickness}" len="${width}">
-		<origin xyz="0 ${mountingYpos+mountingspacing/2 - thickness/2} ${height+thickness/2}" rpy="0 ${-M_PI/2} 0"/>
+		<origin xyz="0 ${mountingYpos+mountingspacing/2 - thickness/2} ${height+thickness/2}" rpy="0 ${-pi/2} 0"/>
 	 </xacro:bar>
     <!-- additional collision box inbetzeen the mounting bars at the top -->
@@ -71,20 +71,20 @@
 	 <xacro:bar thickness="${thickness}" len="${depth}">
 		<origin xyz="${-(width+thickness)/2} ${depth/2} ${-thickness/2}"
-				  rpy="${-M_PI/2} 0 0"/>
+				  rpy="${-pi/2} 0 0"/>
 	 </xacro:bar>
 	 <!-- right side bottom -->
 	 <xacro:bar thickness="${thickness}" len="${depth}">
 		<origin xyz="${+(width+thickness)/2} ${depth/2} ${-thickness/2}"
-				  rpy="${-M_PI/2} 0 0"/>
+				  rpy="${-pi/2} 0 0"/>
 	 </xacro:bar>
 	 <!-- left side top -->
 	 <xacro:bar thickness="${thickness}" len="${depth}">
 		<origin xyz="${-(width+thickness)/2} ${depth/2} ${height+thickness/2}"
-				  rpy="${-M_PI/2} 0 0"/>
+				  rpy="${-pi/2} 0 0"/>
 	 </xacro:bar>
 	 <!-- right side top -->
 	 <xacro:bar thickness="${thickness}" len="${depth}">
 		<origin xyz="${+(width+thickness)/2} ${depth/2} ${height+thickness/2}"
-				  rpy="${-M_PI/2} 0 0"/>
+				  rpy="${-pi/2} 0 0"/>
 	 </xacro:bar>
    <!-- table plane -->

File: agni_description/urdf/util.urdf.xacro (robot description, xacro)
@@ -1,5 +1,4 @@
 <?xml version="1.0"?>
 <robot xmlns:xacro="http://www.ros.org/wiki/xacro">
-  <xacro:property name="M_PI" value="3.1415926535897931"/>
   <!--
 		Little helper macro to define the inertia matrix needed
