Commit message: use yaml robots file
- helpers.urdf.xacro: generic macros arm(), tool(), arm_with_tool()
- calibration files use scheme <tool name>_cal.xml or <arm name>_cal.xml
  where <tool name> and <arm name> match the names in the yaml settings file
- renamed link "*arm_hand_mount" to more generic "*tool_mount"

File: agni_description/kuka/kuka.urdf.xacro (robot description, xacro)
@@ -13,6 +13,5 @@
   <xacro:property name="joint_damping" value="1.0" />
   <xacro:property name="arm_velocity_scale_factor" value="1"/>
-  <!-- reflect is either 1 (for right arm) or -1 (for left arm) -->
-  <xacro:macro name="kuka_lwr_arm" params="name reflect tool_name:=''">
+  <xacro:macro name="kuka_lwr_arm" params="name">
     <link name="${name}arm_base_link">
       <inertial>
@@ -351,15 +350,15 @@
       </inertial>
       <visual>
-        <origin xyz="0 0 0" rpy="0 0 ${reflect * -1/4 * pi  +  pi}"/>
-        <geometry>
-          <mesh scale="100 100 100"
-					 filename="package://agni_description/kuka/meshes/arm_flanche${tool_name}.dae"/>
+        <origin xyz="0 0 0" rpy="0 0 0"/>
+        <geometry>
+          <mesh scale="100 100 100"
+                filename="package://agni_description/kuka/meshes/arm_flanche.dae"/>
         </geometry>
         <material name="Grey"/>
       </visual>
       <collision>
-        <origin xyz="0 0 0" rpy="0 0 ${reflect * -1/4 * pi  +  pi}"/>
-        <geometry>
-          <mesh filename="package://agni_description/kuka/meshes/convex/arm_flanche${tool_name}_convex.stl" scale="1.0 1.0 1.0"/>
+        <origin xyz="0 0 0" rpy="0 0 0"/>
+        <geometry>
+          <mesh filename="package://agni_description/kuka/meshes/convex/arm_flanche_convex.stl" scale="1.0 1.0 1.0"/>
         </geometry>
       </collision>
@@ -369,12 +368,8 @@
     </gazebo>
     <joint name="${name}arm_hand_fixed_joint" type="fixed">
-<!--
-      <origin xyz="${-reflect * 0.075} -0.075 -0.094"
-              rpy="${0.5*reflect*pi} 0 ${(1.5 + 0.25*reflect)*pi}"/>
--->
       <parent link="${name}arm_7_link"/>
-      <child link="${name}arm_hand_mount"/>
-    </joint>
-    <link name="${name}arm_hand_mount" />
+      <child link="${name}tool_mount"/>
+    </joint>
+    <link name="${name}tool_mount" />
   </xacro:macro>
 </robot>

File: agni_description/kuka/lwr_controllers.gazebo.xacro (robot description, xacro)
@@ -1,47 +1,23 @@
 <?xml version="1.0"?>
 <robot xmlns:xacro="http://www.ros.org/wiki/xacro">
-  <!-- default port value. do not modify here.
-       If not correct, redefine your own property and pass the values through macro param -->
-  <xacro:property name="portlist" value="${dict(right=49938, left=49940)}"/>
-  <!-- namespace must be set up according to launch file namespace -->
-  <!-- port is the port number for the FRI UDP connection (be aware that port+1 is also used) -->
-  <xacro:macro name="left_lwr_arm_gazebo_controller" params="namespace port:=${portlist['left']}">
-    <xacro:property name="prefix"  value="${'' if namespace=='' else namespace}" />
+	<!-- namespace must be set up according to launch file namespace -->
+	<!-- port is the port number for the FRI UDP connection (be aware that port+1 is also used) -->
+	<xacro:macro name="lwr_arm_gazebo_controller" params="namespace port">
+		<xacro:property name="prefix"  value="${namespace + '_' if namespace else ''}" />
 		<gazebo>
-			<plugin name="left_lwr_arm_controller" filename="liblwr_controller.so">
+			<plugin name="${prefix}lwr_arm_controller" filename="liblwr_controller.so">
 				<alwaysOn>true</alwaysOn>
-				<robotPrefix>${prefix}</robotPrefix>
+				<robotPrefix>${namespace}</robotPrefix>
 				<robotNamespace>${namespace}</robotNamespace>
 				<remotePort>${port}</remotePort>
-				<baseLink>la_arm_base_link</baseLink>
-				<toolLink>la_arm_hand_mount</toolLink>
-				<la_arm_0_joint>0.0</la_arm_0_joint>
-				<la_arm_1_joint>0</la_arm_1_joint>
-				<la_arm_2_joint>0.0</la_arm_2_joint>
-				<la_arm_3_joint>0</la_arm_3_joint>
-				<la_arm_4_joint>0</la_arm_4_joint>
-				<la_arm_5_joint>0</la_arm_5_joint>
-				<la_arm_6_joint>0</la_arm_6_joint>
-			</plugin>
-		</gazebo>
-	</xacro:macro>
-	<!-- namespace must be set up according to launch file namespace -->
-  <!-- port is the port number for the FRI UDP connection (be aware that port+1 is also used) -->
-  <xacro:macro name="right_lwr_arm_gazebo_controller" params="namespace port:=${portlist['right']}">
-		<gazebo>
-			<plugin name="right_lwr_arm_controller" filename="liblwr_controller.so">
-				<alwaysOn>true</alwaysOn>
-				<robotPrefix>ra</robotPrefix>
-				<robotNamespace>${namespace}</robotNamespace>
-				<remotePort>${port}</remotePort>
-				<baseLink>ra_arm_base_link</baseLink>
-				<toolLink>ra_arm_hand_mount</toolLink>
-				<ra_arm_0_joint>0.0</ra_arm_0_joint>
-				<ra_arm_1_joint>0</ra_arm_1_joint>
-				<ra_arm_2_joint>0.0</ra_arm_2_joint>
-				<ra_arm_3_joint>0</ra_arm_3_joint>
-				<ra_arm_4_joint>0</ra_arm_4_joint>
-				<ra_arm_5_joint>0</ra_arm_5_joint>
-				<ra_arm_6_joint>0</ra_arm_6_joint>
+				<baseLink>${prefix}arm_base_link</baseLink>
+				<toolLink>${prefix}tool_mount</toolLink>
+				<xacro:rename xacro:name="${prefix}arm_0_joint">0</xacro:rename>
+				<xacro:rename xacro:name="${prefix}arm_1_joint">0</xacro:rename>
+				<xacro:rename xacro:name="${prefix}arm_2_joint">0</xacro:rename>
+				<xacro:rename xacro:name="${prefix}arm_3_joint">0</xacro:rename>
+				<xacro:rename xacro:name="${prefix}arm_4_joint">0</xacro:rename>
+				<xacro:rename xacro:name="${prefix}arm_5_joint">0</xacro:rename>
+				<xacro:rename xacro:name="${prefix}arm_6_joint">0</xacro:rename>
 			</plugin>
 		</gazebo>

File: agni_description/models/myrmex_quick_mount.urdf.xacro (robot description, xacro)
@@ -1,38 +1,42 @@
 <?xml version="1.0"?>
 <robot name="myrmex_quick_mount" xmlns:xacro="http://www.ros.org/wiki/xacro">
-  <xacro:macro name="myrmex_quick_mount" params="prefix tactile">
-  <link name="${prefix}myrmex_quick_mount">
-    <visual>
-      <origin xyz="0 0 0"
-          rpy="0 0 0"/>
-      <geometry>
-        <mesh scale="0.001 0.001 0.001"
-					 filename="package://agni_description/models/meshes/myrmex_quick_mount.dae"/>
-      </geometry>
-    </visual>
-    <collision>
-      <origin xyz="0 0 0.00797"
-          rpy="0 0 0"/>
-      <geometry>
-        <cylinder radius="0.06725" length="0.01584"/>
-      </geometry>
-    </collision>
-     <collision>
-      <origin xyz="0 0 0.02159"
-          rpy="0 0 0"/>
-      <geometry>
-        <cylinder radius="0.060" length="0.0115"/>
-      </geometry>
-    </collision>
-    <collision>
-      <origin xyz="0 0 0.03034"
-          rpy="0 0 0"/>
+  <xacro:macro name="myrmex_quick_mount" params="prefix:=''">
+    <link name="${prefix}myrmex_quick_mount">
+      <visual>
+        <origin xyz="0 0 0" rpy="0 0 0"/>
+        <geometry>
+          <mesh scale="0.001 0.001 0.001"
+                filename="package://agni_description/models/meshes/myrmex_quick_mount.dae"/>
+        </geometry>
+      </visual>
+      <collision>
+        <origin xyz="0 0 0.00797" rpy="0 0 0"/>
+        <geometry>
+          <cylinder radius="0.06725" length="0.01584"/>
+        </geometry>
+      </collision>
+      <collision>
+        <origin xyz="0 0 0.02159" rpy="0 0 0"/>
+        <geometry>
+          <cylinder radius="0.060" length="0.0115"/>
+        </geometry>
+      </collision>
+      <collision>
+        <origin xyz="0 0 0.03034" rpy="0 0 0"/>
         <geometry>
           <box size="0.095 0.095 0.006"/>
         </geometry>
-    </collision>
-  </link>
-  <gazebo reference="${prefix}myrmex_quick_mount">
-  </gazebo>
-    </xacro:macro>
+      </collision>
+    </link>
+    <gazebo reference="${prefix}myrmex_quick_mount"></gazebo>
+  </xacro:macro>
+  <xacro:macro name="myrmex_tactile_markers" params="parent topic *origin">
+    <!-- tactile marker mapping description -->
+    <tactile topic="${topic}" data="data" xs="0 4095" link="${parent}">
+      <geometry>
+        <grid size="16 16" spacing="0.005 0.005"/>
+      </geometry>
+      <xacro:insert_block name="origin"/>
+    </tactile>
+  </xacro:macro>
 </robot>

File: agni_description/robots/famula.urdf.xacro (robot description, xacro)
@@ -1,52 +1,20 @@
 <?xml version="1.0"?>
 <robot name="arm_hand_shadow" xmlns:xacro="http://www.ros.org/wiki/xacro">
+	<xacro:property name="settings" value="${load_yaml('robots.yaml')}" />
 	<xacro:arg name="SIM" default="1"/>
 	<xacro:arg name="CALIB" default="famula"/>
-	<!-- Frame -->
+	<!-- frame -->
 	<xacro:include filename="../urdf/frame-half.urdf.xacro"/>
-	<xacro:include filename="../calibration/kuka_frame_cal.xml"/>
-	<xacro:frame prefix="kuka"/>
-	<!-- arm with -->
-	<xacro:include filename="../robots/kuka_arm.urdf.xacro" />
-	<!-- end-effector -->
-	<xacro:include filename="../robots/shadow_hand_ee.urdf.xacro" />
-	<!-- Right -->
-	<!-- Arm -->
-	<xacro:include filename="../calibration/$(arg CALIB)/kuka_right_cal.xml"/>
-	<xacro:call macro="kuka_arm" parent="world" side="right" controller="$(arg SIM)">
-		<origin xyz="${cal_arm_x} ${cal_arm_y} ${cal_arm_z}"
-		        rpy="${cal_arm_roll} ${cal_arm_pitch} ${cal_arm_yaw}"/>
-	</xacro:call>
-	<!-- Effector -->
-	<xacro:call macro="shadow_hand" model="motor" side="right" tactile="ubi" prefix="rh" />
-	<!-- Link arm and effector -->
-	<xacro:include filename="../calibration/$(arg CALIB)/shadow_hand_motor_right_cal.xml"/>
-	<joint name="ra_arm_hand_mount" type="fixed">
-		<parent link="ra_${arm_mount['kuka']}"/>
-		<child link="rh_${ee_mount['shadow_hand']}"/>
-		<origin xyz="${cal_ee_x} ${cal_ee_y} ${cal_ee_z}"
-		        rpy="${cal_ee_roll} ${cal_ee_pitch} ${cal_ee_yaw}"/>
-	</joint>
-	<!-- Left -->
-	<!-- Arm -->
-	<xacro:include filename="../calibration/$(arg CALIB)/kuka_left_cal.xml"/>
-	<xacro:call macro="kuka_arm" parent="world" side="left" controller="$(arg SIM)">
-		<origin xyz="${cal_arm_x} ${cal_arm_y} ${cal_arm_z}"
-		        rpy="${cal_arm_roll} ${cal_arm_pitch} ${cal_arm_yaw}"/>
-	</xacro:call>
-	<!-- Effector -->
-	<xacro:call macro="shadow_hand" model="motor" side="left" tactile="ubi" prefix="lh" />
-	<!-- Link arm and effector -->
-	<xacro:include filename="../calibration/$(arg CALIB)/shadow_hand_motor_left_cal.xml"/>
-	<joint name="la_arm_hand_mount" type="fixed">
-		<parent link="la_${arm_mount['kuka']}"/>
-		<child link="lh_${ee_mount['shadow_hand']}"/>
-		<origin xyz="${cal_ee_x} ${cal_ee_y} ${cal_ee_z}"
-		        rpy="${cal_ee_roll} ${cal_ee_pitch} ${cal_ee_yaw}"/>
-	</joint>
+	<xacro:include filename="../calibration/famula_frame_cal.xml"/>
+	<xacro:frame/>
+	<xacro:include filename="../urdf/helpers.urdf.xacro" />
+	<xacro:arm_with_tool parent="frame" prefix="r"
+	                     arm_type="kukaR" tool_type="shadow_motor_right" />
+	<xacro:arm_with_tool parent="frame" prefix="l"
+	                     arm_type="kukaL" tool_type="shadow_motor_left"/>
 	<!-- flobi -->
 	<xacro:include filename="$(find flobi_sim)/defs/xacro/flobiv3.urdf.xacro" />
-	<xacro:flobi prefix="" neutral="1" gender="0" parent="kuka_frame" >
-		<origin xyz="0 ${cal_mount_triangle_offset[1]} ${cal_mount_triangle_offset[2]+mount_triangle_length/2*sin(60/180.0*pi)+0.01}"
+	<xacro:flobi parent="frame" prefix="" neutral="1" gender="0">
+		<origin xyz="${cal_flobi_pos['X']} ${cal_flobi_pos['Y']} ${cal_flobi_pos['Z']}"
 		        rpy="0 0 ${-pi/2.0}"/>
 	</xacro:flobi>

File: agni_description/robots/kuka_arm.urdf.xacro (robot description, xacro)
@@ -1,32 +1,13 @@
 <?xml version="1.0"?>
-<robot name="kuka_anytool"
-     xmlns:xacro="http://www.ros.org/wiki/xacro">
-  <xacro:include filename="../kuka/kuka.urdf.xacro"/>
-  <xacro:include filename="../kuka/lwr_controllers.gazebo.xacro"/>
-  <!-- arm_ee macro with the params
-         * parent : where it is attached
-         * side : right|left
-         * controller : should the controllers be loaded or not
-         * *origin : first block for the base offset -->
-  <xacro:property name="arm_mount"  value="${dict( kuka='arm_hand_mount' )}" />
-  <!-- default arm cal (so that the dict exists) but key right and left should be set at top level-->
-  <xacro:property name="cal_arm_x" value="${dict(default= 0.0)}" />
-  <xacro:property name="cal_arm_y" value="${dict(default= 0.0)}" />
-  <xacro:property name="cal_arm_z" value="${dict(default= 0.0)}" />
-  <xacro:property name="cal_arm_yaw" value="${dict(default= 0.0)}" />
-  <xacro:property name="cal_arm_pitch" value="${dict(default= 0.0)}" />
-  <xacro:property name="cal_arm_roll" value="${dict(default= 0.0)}" />
-  <xacro:macro name="kuka_arm" params="parent side controller *origin">
-  <!-- KUKA arm -->
-    <xacro:property name="prefix"  value="${'ra' if side=='right' else 'la'}" />
-    <xacro:kuka_lwr_arm name="${prefix}_" reflect="${1 if side=='right' else -1}" tool_name=""/>
-    <joint name="${prefix}_frame_placement" type="fixed">
-       <xacro:insert_block name="origin" />
-      <parent link="${parent}"/>
-      <child link="${prefix}_arm_base_link"/>
-    </joint>
+<robot name="kuka_arm" xmlns:xacro="http://www.ros.org/wiki/xacro">
+  <xacro:macro name="kuka_arm" params="prefix controller">
+    <!-- KUKA arm -->
+    <xacro:include filename="../kuka/kuka.urdf.xacro"/>
+    <xacro:kuka_lwr_arm name="${prefix + '_' if prefix else ''}"/>
     <xacro:if value="${controller}">
-      <!-- add controllers -->
-      <xacro:call macro="${side}_lwr_arm_gazebo_controller" namespace="${prefix}" port="${portlist[side]}"/>
+      <!-- add gazebo controllers -->
+      <xacro:include filename="../kuka/lwr_controllers.gazebo.xacro"/>
+      <xacro:lwr_arm_gazebo_controller namespace="${prefix}"
+                                       port="${props['port']}"/>
     </xacro:if>
   </xacro:macro>

File: agni_description/robots/pa10_arm.urdf.xacro (robot description, xacro)
@@ -1,34 +1,15 @@
 <?xml version="1.0"?>
-<robot name="kuka_anytool"
-     xmlns:xacro="http://www.ros.org/wiki/xacro">
-  <xacro:include filename="../pa10/pa10-a.urdf.xacro"/>
-  <xacro:include filename="../pa10/pa10-c.urdf.xacro"/>
-  <xacro:include filename="../pa10/pa10_shadow_controller_manager.xacro"/>
-  <!-- arm macro with the params
-         * parent : where it is attached
-         * side : right|left
-         * controller : should the controllers be loaded or not
-         * *origin : first block for the base offset -->
-  <xacro:property name="arm_mount"  value="${dict( pa10='arm_hand_mount' )}" />
-  <!-- default arm cal (so that the dict exists) but key right and left should be set at top level-->
-  <xacro:property name="cal_arm_x" value="${dict(default= 0.0)}" />
-  <xacro:property name="cal_arm_y" value="${dict(default= 0.0)}" />
-  <xacro:property name="cal_arm_z" value="${dict(default= 0.0)}" />
-  <xacro:property name="cal_arm_yaw" value="${dict(default= 0.0)}" />
-  <xacro:property name="cal_arm_pitch" value="${dict(default= 0.0)}" />
-  <xacro:property name="cal_arm_roll" value="${dict(default= 0.0)}" />
-  <xacro:macro name="pa10_arm" params="parent side controller *origin">
-  <!-- PA10 arm -->
-    <xacro:property name="armname" value="${dict( right='pa10c', left='pa10a')}"/>
-    <xacro:property name="prefix"  value="${'ra' if side=='right' else 'la'}" />
-    <xacro:call macro="${armname[side]}_arm" name="${prefix}_" />
-    <joint name="${prefix}_frame_placement" type="fixed">
-      <xacro:insert_block name="origin" />
-      <parent link="${parent}"/>
-      <child link="${prefix}_arm_base_link"/>
-    </joint>
+<robot name="pa10_arm" xmlns:xacro="http://www.ros.org/wiki/xacro">
+  <xacro:property name="filename" value="${dict([('7a', 'pa10-a'), ('7c', 'pa10-c')])}"/>
+  <xacro:property name="macroname" value="${dict([('7a', 'pa10a_arm'), ('7c', 'pa10c_arm')])}"/>
+  <xacro:macro name="pa10_arm" params="prefix controller">
+    <!-- PA10 arm -->
+    <xacro:include filename="../pa10/${filename[props['model']]}.urdf.xacro"/>
+    <xacro:call macro="${macroname[props['model']]}"
+                name="${prefix + '_' if prefix else ''}"/>
     <xacro:if value="${controller}">
-      <!-- add controllers -->
-       <xacro:pa10_shadow_gazebo_controller_manager namespace="${prefix}"/>
+      <!-- add gazebo controllers -->
+      <xacro:include filename="../pa10/pa10_shadow_controller_manager.xacro"/>
+      <xacro:pa10_shadow_gazebo_controller_manager namespace="${prefix}"/>
     </xacro:if>
   </xacro:macro>

File: agni_description/robots/sfb.urdf.xacro (robot description, xacro)
@@ -1,43 +1,15 @@
 <?xml version="1.0"?>
 <robot name="arm_hand_shadow" xmlns:xacro="http://www.ros.org/wiki/xacro">
+	<xacro:property name="settings" value="${load_yaml('robots.yaml')}" />
 	<xacro:arg name="SIM" default="1"/>
 	<xacro:arg name="CALIB" default="sfb"/>
 	<!-- Frame -->
 	<xacro:include filename="../urdf/frame.urdf.xacro"/>
-	<xacro:include filename="../calibration/pa10_frame_cal.xml"/>
-	<xacro:frame prefix="pa10"/>
-	<!-- arm  -->
-	<xacro:include filename="../robots/pa10_arm.urdf.xacro" />
-	<!-- end-effector -->
-	<xacro:include filename="../robots/shadow_hand_ee.urdf.xacro" />
-	<!-- Right -->
-	<!-- Arm -->
-	<xacro:include filename="../calibration/$(arg CALIB)/pa10_right_cal.xml"/>
-	<xacro:call macro="pa10_arm" parent="world" side="right" controller="$(arg SIM)">
-		<origin xyz="${cal_arm_x} ${cal_arm_y} ${cal_arm_z}" rpy="${cal_arm_roll} ${cal_arm_pitch} ${cal_arm_yaw}"/>
-	</xacro:call>
-	<!-- Effector -->
-	<xacro:call macro="shadow_hand" model="motor" side="right" tactile="ubi" prefix="rh" />
-	<!-- Link arm and effector -->
-	<xacro:include filename="../calibration/$(arg CALIB)/shadow_hand_motor_right_cal.xml"/>
-	<joint name="ra_arm_hand_mount" type="fixed">
-		<parent link="ra_${arm_mount['pa10']}"/>
-		<child link="rh_${ee_mount['shadow_hand']}"/>
-		<origin xyz="${cal_ee_x} ${cal_ee_y} ${cal_ee_z}" rpy="${cal_ee_roll} ${cal_ee_pitch} ${cal_ee_yaw}"/>
-	</joint>
-	<!-- Left -->
-	<!-- Arm -->
-	<xacro:include filename="../calibration/$(arg CALIB)/pa10_left_cal.xml"/>
-	<xacro:call macro="pa10_arm" parent="world" side="left" controller="$(arg SIM)">
-		<origin xyz="${cal_arm_x} ${cal_arm_y} ${cal_arm_z}" rpy="${cal_arm_roll} ${cal_arm_pitch} ${cal_arm_yaw}"/>
-	</xacro:call>
-	<!-- Effector -->
-	<xacro:call macro="shadow_hand" model="motor" side="left" tactile="ubi" prefix="lh" />
-	<!-- Link arm and effector -->
-	<xacro:include filename="../calibration/$(arg CALIB)/shadow_hand_motor_left_cal.xml"/>
-	<joint name="la_arm_hand_mount" type="fixed">
-		<parent link="la_${arm_mount['pa10']}"/>
-		<child link="lh_${ee_mount['shadow_hand']}"/>
-		<origin xyz="${cal_ee_x} ${cal_ee_y} ${cal_ee_z}" rpy="${cal_ee_roll} ${cal_ee_pitch} ${cal_ee_yaw}"/>
-	</joint>
+	<xacro:include filename="../calibration/sfb_frame_cal.xml"/>
+	<xacro:frame/>
+	<xacro:include filename="../urdf/helpers.urdf.xacro" />
+	<xacro:arm_with_tool parent="frame" prefix="r"
+	                     arm_type="pa10c" tool_type="shadow_motor_right"/>
+	<xacro:arm_with_tool parent="frame" prefix="l"
+	                     arm_type="pa10a" tool_type="shadow_motor_left"/>
 </robot>
