Commit message: use yaml robots file
- helpers.urdf.xacro: generic macros arm(), tool(), arm_with_tool()
- calibration files use scheme <tool name>_cal.xml or <arm name>_cal.xml
  where <tool name> and <arm name> match the names in the yaml settings file
- renamed link "*arm_hand_mount" to more generic "*tool_mount"

File: agni_description/urdf/frame-half.urdf.xacro (robot description, xacro)
@@ -4,5 +4,4 @@
       xmlns:controller="http://playerstage.sourceforge.net/gazebo/xmlschema/#controller"
       xmlns:interface="http://playerstage.sourceforge.net/gazebo/xmlschema/#interface">
-	<xacro:property name="mount_triangle_length" value="0.26" />
 	<xacro:include filename="../urdf/materials.urdf.xacro"/>
 	<xacro:macro name="bar" params="thickness len *origin">
@@ -17,10 +16,11 @@
 		</collision>
 	</xacro:macro>
-	<xacro:macro name="frame" params="prefix thickness:=${cal_frame_thick}
+	<xacro:macro name="frame" params="prefix:='' thickness:=${cal_frame_thick}
 	   width:=${cal_frame_width} depth:=${cal_frame_depth} height:=${cal_frame_height}
-	   tableHeight:=${cal_frame_table_height}
-	   triangle_offset:=${cal_mount_triangle_offset}">
+	   tableHeight:=${cal_frame_table_height} triangle_pos:=${cal_triangle_pos}">
+		<xacro:property name="mount_triangle_length" value="0.26" />
+		<xacro:property name="mount_triangle_thickness" value="0.02"/>
 		<link name="world"/>
-		<link name="${prefix}_frame">
+		<link name="${prefix}frame">
 			<inertial>
 				<mass value="100.0" />
@@ -95,45 +95,38 @@
 			</collision>
 			<!-- kuka mount triangle -->
-			<visual>
-				<origin xyz="${triangle_offset[0]-0.01*cos(30/180.0*pi)}
-				             ${triangle_offset[1]}
-				             ${triangle_offset[2]-0.01*sin(30/180.0*pi)}"
+			<xacro:macro name="plate"
+			             params="thickness:=${mount_triangle_thickness}
+			                     length:=${mount_triangle_length} *origin">
+				<visual>
+					<xacro:insert_block name="origin"/>
+					<geometry><box size="${length} ${length} ${thickness}"/></geometry>
+					<material name="Silver"/>
+				</visual>
+				<collision>
+					<xacro:insert_block name="origin"/>
+					<geometry><box size="${length} ${length} ${thickness - 0.005}"/></geometry>
+				</collision>
+			</xacro:macro>
+			<xacro:property name="mtth" value="${mount_triangle_thickness}"/>
+			<xacro:property name="mtlen" value="${mount_triangle_length}"/>
+			<!-- left plate -->
+			<xacro:plate>
+				<origin xyz="${triangle_pos['leftX']-mtth/2*cos(30/180.0*pi)}
+				             ${triangle_pos['Y']}
+				             ${triangle_pos['Z']-mtth/2*sin(30/180.0*pi)}"
 				        rpy="0 ${pi/3} 0"/>
-				<geometry><box size="${mount_triangle_length} ${mount_triangle_length} ${0.02}"/></geometry>
-				<material name="Silver"/>
-			</visual>
-			<collision>
-				<origin xyz="${triangle_offset[0]-0.01*cos(30/180.0*pi)}
-				             ${triangle_offset[1]}
-				             ${triangle_offset[2]-0.01*sin(30/180.0*pi)}"
-				        rpy="0 ${pi/3} 0"/>
-				<geometry><box size="${mount_triangle_length} ${mount_triangle_length} ${0.015}"/></geometry>
-			</collision>
-			<visual>
-				<origin xyz="-${triangle_offset[0]+0.01*cos(30/180.0*pi)}
-				             ${triangle_offset[1]}
-				             ${triangle_offset[2]-0.01*sin(30/180.0*pi)}"
+			</xacro:plate>
+			<!-- right plate -->
+			<xacro:plate>
+				<origin xyz="${triangle_pos['rightX']+mtth/2*cos(30/180.0*pi)}
+				             ${triangle_pos['Y']}
+				             ${triangle_pos['Z']-mtth/2*sin(30/180.0*pi)}"
 				        rpy="0 ${-pi/3} 0"/>
-				<geometry><box size="${mount_triangle_length} ${mount_triangle_length} ${0.02}"/></geometry>
-				<material name="Silver"/>
-			</visual>
-			<collision>
-				<origin xyz="-${triangle_offset[0]+0.01*cos(30/180.0*pi)}
-				             ${triangle_offset[1]}
-				             ${triangle_offset[2]-0.01*sin(30/180.0*pi)}"
-				        rpy="0 ${-pi/3} 0"/>
-				<geometry><box size="${mount_triangle_length} ${mount_triangle_length} ${0.015}"/></geometry>
-			</collision>
-			<visual>
-				<origin xyz="0 ${triangle_offset[1]} ${triangle_offset[2]-sin(30/180.0*pi)*0.02-mount_triangle_length/2*sin(60/180.0*pi)-0.01}"
+			</xacro:plate>
+			<!-- lower plate -->
+			<xacro:plate>
+				<origin xyz="0 ${triangle_pos['Y']} ${triangle_pos['Z']-sin(30/180.0*pi)*mtth-mtlen/2*sin(60/180.0*pi)-mtth/2}"
 				        rpy="0 0 0"/>
-				<geometry><box size="${mount_triangle_length} ${mount_triangle_length} ${0.02}"/></geometry>
-				<material name="Silver"/>
-			</visual>
-			<collision>
-				<origin xyz="0 ${triangle_offset[1]} ${triangle_offset[2]-sin(30/180.0*pi)*0.02-mount_triangle_length/2*sin(60/180.0*pi)-0.01}"
-				        rpy="0 0 0"/>
-				<geometry><box size="${mount_triangle_length} ${mount_triangle_length} ${0.015}"/></geometry>
-			</collision>
+			</xacro:plate>
 			<!-- table plane -->
 			<visual>
@@ -149,11 +142,11 @@
 			</collision>
 		</link>
-		<gazebo reference="${prefix}_frame">
+		<gazebo reference="${prefix}frame">
 			<material value="Gazebo/Grey"/>
 		</gazebo>
-		<joint name="${prefix}_frame_joint" type="fixed">
+		<joint name="${prefix}frame_joint" type="fixed">
 			<origin xyz="0 0 0" rpy="0 0 0"/>
 			<parent link="world"/>
-			<child link="${prefix}_frame"/>
+			<child link="${prefix}frame"/>
 		</joint>
 	</xacro:macro>

File: agni_description/urdf/frame.urdf.xacro (robot description, xacro)
@@ -20,5 +20,5 @@
 		</visual>
 	</xacro:macro>
-	<xacro:macro name="frame" params="prefix thickness:=${cal_frame_thick}
+	<xacro:macro name="frame" params="prefix:='' thickness:=${cal_frame_thick}
 	   width:=${cal_frame_width} depth:=${cal_frame_depth} height:=${cal_frame_height}
 	   tableHeight:=${cal_frame_table_height}
@@ -26,5 +26,5 @@
 	   mountingspacing:=${cal_frame_mounting_spacing}">
 		<link name="world"/>
-		<link name="${prefix}_frame">
+		<link name="${prefix}frame">
 			<inertial>
 				<mass value="100.0" />
@@ -149,8 +149,8 @@
 			</collision>
 		</link>
-		<joint name="${prefix}_frame_joint" type="fixed">
+		<joint name="${prefix}frame_joint" type="fixed">
 			<origin xyz="0 0 0" rpy="0 0 0"/>
 			<parent link="world"/>
-			<child link="${prefix}_frame"/>
+			<child link="${prefix}frame"/>
 		</joint>
 	</xacro:macro>

Commit message: Added gravity compensation support (parameter passing to lwr_controller) Fixed damping

File: agni_description/kuka/kuka.urdf.xacro (robot description, xacro)
@@ -5,5 +5,5 @@
        xmlns:interface="http://playerstage.sourceforge.net/gazebo/xmlschema/#interface">
   <xacro:include filename="../urdf/util.urdf.xacro"/>
-  <xacro:property name="arm_elem_base_mass" value="2.0"/>
+  <xacro:property name="arm_elem_base_mass" value="1.2"/>
   <xacro:property name="arm_elem_link_mass" value="2.0"/>
   <xacro:property name="arm_elem_ball_link_mass" value="1.0"/>
@@ -11,5 +11,5 @@
   <xacro:property name="safety_controller_k_pos" value="100" />
   <xacro:property name="safety_controller_k_vel" value="2" />
-  <xacro:property name="joint_damping" value="1.0" />
+  <xacro:property name="joint_damping_factor" value="1.0" />
   <xacro:property name="arm_velocity_scale_factor" value="1"/>
   <xacro:macro name="kuka_lwr_arm" params="name">
@@ -48,5 +48,5 @@
                          k_position="${safety_controller_k_pos}"
                          k_velocity="${safety_controller_k_vel}"/>
-      <dynamics damping="${joint_damping}"/>
+      <dynamics damping="${joint_damping_factor*5.0}"/>
       <parent link="${name}arm_base_link"/>
       <child link="${name}arm_1_link"/>
@@ -94,5 +94,5 @@
                          k_position="${safety_controller_k_pos}"
                          k_velocity="${safety_controller_k_vel}"/>
-      <dynamics damping="${joint_damping}"/>
+      <dynamics damping="${joint_damping_factor*5.0}"/>
       <parent link="${name}arm_1_link"/>
       <child link="${name}arm_2_link"/>
@@ -141,5 +141,5 @@
                          k_position="${safety_controller_k_pos}"
                          k_velocity="${safety_controller_k_vel}"/>
-      <dynamics damping="${joint_damping}"/>
+      <dynamics damping="${joint_damping_factor*3.0}"/>
       <parent link="${name}arm_2_link"/>
       <child link="${name}arm_3_link"/>
@@ -188,5 +188,5 @@
                          k_position="${safety_controller_k_pos}"
                          k_velocity="${safety_controller_k_vel}"/>
-      <dynamics damping="${joint_damping}"/>
+      <dynamics damping="${joint_damping_factor*3.0}"/>
       <parent link="${name}arm_3_link"/>
       <child link="${name}arm_4_link"/>
@@ -235,5 +235,5 @@
                          k_position="${safety_controller_k_pos}"
                          k_velocity="${safety_controller_k_vel}"/>
-      <dynamics damping="${joint_damping}"/>
+      <dynamics damping="${joint_damping_factor*1.0}"/>
       <parent link="${name}arm_4_link"/>
       <child link="${name}arm_5_link"/>
@@ -282,5 +282,5 @@
                          k_position="${safety_controller_k_pos}"
                          k_velocity="${safety_controller_k_vel}"/>
-      <dynamics damping="${joint_damping}"/>
+      <dynamics damping="${joint_damping_factor*1.0}"/>
       <parent link="${name}arm_5_link"/>
       <child link="${name}arm_6_link"/>
@@ -329,5 +329,5 @@
                          k_position="${safety_controller_k_pos}"
                          k_velocity="${safety_controller_k_vel}"/>
-      <dynamics damping="${joint_damping}"/>
+      <dynamics damping="${joint_damping_factor*1.0}"/>
       <parent link="${name}arm_6_link"/>
       <child link="${name}arm_7_link"/>

File: agni_description/kuka/lwr_controllers.gazebo.xacro (robot description, xacro)
@@ -3,5 +3,6 @@
 	<!-- namespace must be set up according to launch file namespace -->
 	<!-- port is the port number for the FRI UDP connection (be aware that port+1 is also used) -->
-	<xacro:macro name="lwr_arm_gazebo_controller" params="namespace port">
+	<xacro:macro name="lwr_arm_gazebo_controller" params="namespace port gravity_dir:=^|-
+		                                                    payload_mass:=^|- payload_cog:=^|-">
 		<xacro:property name="prefix"  value="${namespace + '_' if namespace else ''}" />
 		<gazebo>
@@ -13,4 +14,13 @@
 				<baseLink>${prefix}arm_base_link</baseLink>
 				<toolLink>${prefix}tool_mount</toolLink>
+				<xacro:if value="${gravity_dir not in ['','-']}" >
+					<gravityDirection>${gravity_dir}</gravityDirection>
+				</xacro:if>
+				<xacro:if value="${payload_mass not in ['','-']}" >
+					<payloadMass>${payload_mass}</payloadMass>
+				</xacro:if>
+				<xacro:if value="${payload_cog not in ['','-']}" >
+					<payloadCOG>${payload_cog}</payloadCOG>
+				</xacro:if>
 				<xacro:element xacro:name="${prefix}arm_0_joint">0</xacro:element>
 				<xacro:element xacro:name="${prefix}arm_1_joint">0</xacro:element>

File: agni_description/urdf/helpers.urdf.xacro (robot description, xacro)
@@ -47,4 +47,9 @@
     <xacro:property name="arm_prefix_" value="${arm_prefix + '_' if arm_prefix else ''}"/>
     <xacro:property name="tool_prefix_" value="${tool_prefix + '_' if tool_prefix else ''}"/>
+    <!-- add payload mass if relevant -->
+    <xacro:if value="${tool_type not in ['','-']}">
+      <xacro:property name="payload_mass" value="${settings['tools'][tool_type]['props']['mass']}"/>
+      <xacro:property name="payload_cog" value="${settings['tools'][tool_type]['props']['cog']}"/>
+    </xacro:if>
     <xacro:property name="tool_parent" value="${parent}"/>
     <xacro:if value="${arm_type not in ['','-']}">
