Commit message: Modified camera_urdf to support single camera or depth camera or depth with color together (not yet supported inside the plugin but frames are correct now)

File: agni_description/urdf/camera.urdf.xacro (robot description, xacro)
@@ -1,41 +1,47 @@
 <robot xmlns:xacro="http://www.ros.org/wiki/xacro">
-  <!-- The reference frame is the depth optical frame, all other frames are built around it -->
+  <!-- The reference frame is depth optical frame if has_depth, otherwise camera_rgb_optical, all other frames are built around it -->
   <xacro:include filename="../urdf/gazebo_camera.urdf.xacro"/>
   <!-- do not name the macro 'camera', it conflicts with gazebo camera tag -->
-  <xacro:macro name="camera_body" params="parent name fps hfov width height has_depth *origin">
-    <link name="world" />
-    <joint name="${name}_camera_depth_optical_joint" type="fixed">
-      <xacro:insert_block name="origin"/>
-      <parent link="world"/>
-      <child link="${name}_camera_depth_optical_frame" />
-    </joint>
-    <link name="${name}_camera_depth_optical_frame">
-      <inertial>
-        <mass value="0.001" />
-        <origin xyz="0 0 0" />
-        <inertia ixx="0.000002" ixy="0.0" ixz="0.0"
-           iyy="0.00001" iyz="0.0"
-           izz="0.000002" />
-      </inertial>
-    </link>
-    <joint name="${name}_camera_depth_joint" type="fixed">
-      <origin xyz="0 0 0" rpy="${pi/2} ${-pi/2} 0 " />
-      <parent link="${name}_camera_depth_optical_frame" />
-      <child link="${name}_camera_depth_frame" />
-    </joint>
-    <link name="${name}_camera_depth_frame">
-      <inertial>
-        <mass value="0.01" />
-        <origin xyz="0 0 0" />
-        <inertia ixx="0.00001" ixy="0.0" ixz="0.0"
-        iyy="0.0001" iyz="0.0"
-        izz="0.00001" />
-      </inertial>
-    </link>
-    <joint name="base_${name}_camera_depth_joint" type="fixed">
-      <origin xyz="0 -0.018 0" rpy="0 0 0" />
-      <parent link="${name}_camera_depth_frame" />
-      <child link="${name}_camera_link" />
-    </joint>
+  <xacro:macro name="camera_body" params="parent name fps hfov width height has_depth *origin has_second_origin:=0 *second_origin">
+    <xacro:if value="${1 if 'world' in parent else 0}">
+      <link name="${parent}" />
+    </xacro:if>
+    <!-- do not name the macro 'camera', it conflicts with gazebo camera tag -->
+    <xacro:if value="${has_depth}">
+      <!-- attach depth to parent -->
+      <joint name="${name}_camera_depth_optical_joint" type="fixed">
+        <xacro:insert_block name="origin"/>
+        <parent link="${parent}"/>
+        <child link="${name}_camera_depth_optical_frame" />
+      </joint>
+      <link name="${name}_camera_depth_optical_frame">
+        <inertial>
+          <mass value="0.001" />
+          <origin xyz="0 0 0" />
+          <inertia ixx="0.000002" ixy="0.0" ixz="0.0"
+             iyy="0.00001" iyz="0.0"
+             izz="0.000002" />
+        </inertial>
+      </link>
+      <joint name="${name}_camera_depth_joint" type="fixed">
+        <origin xyz="0 0 0" rpy="${pi/2} ${-pi/2} 0 " />
+        <parent link="${name}_camera_depth_optical_frame" />
+        <child link="${name}_camera_depth_frame" />
+      </joint>
+      <link name="${name}_camera_depth_frame">
+        <inertial>
+          <mass value="0.01" />
+          <origin xyz="0 0 0" />
+          <inertia ixx="0.00001" ixy="0.0" ixz="0.0"
+          iyy="0.0001" iyz="0.0"
+          izz="0.00001" />
+        </inertial>
+      </link>
+      <joint name="base_${name}_camera_depth_joint" type="fixed">
+        <origin xyz="0 -0.018 0" rpy="0 0 0" />
+        <parent link="${name}_camera_depth_frame" />
+        <child link="${name}_camera_link" />
+      </joint>
+    </xacro:if>
     <link name="${name}_camera_link">
       <inertial>
@@ -59,9 +65,21 @@
       </collision>
     </link>
-    <joint name="${name}_camera_rgb_joint" type="fixed">
-      <origin xyz="0 -0.005 0" rpy="0 0 0" />
-      <parent link="${name}_camera_link" />
-      <child link="${name}_camera_rgb_frame" />
-    </joint>
+    <xacro:if value="${has_depth}">
+      <xacro:unless value="${has_second_origin}">
+        <!-- attach rgb to camera_link if has depth but not attached to parent -->
+        <joint name="base_${name}_camera_rgb_joint" type="fixed">
+          <origin xyz="0 -0.005 0" rpy="0 0 0" /> <!-- CHECK THIS OFFSET -->
+          <parent link="${name}_camera_link" />
+          <child link="${name}_camera_rgb_frame" />
+        </joint>
+      </xacro:unless>
+    </xacro:if>
+    <xacro:unless value="${has_depth}">
+      <joint name="base_${name}_camera_rgb_joint" type="fixed">
+        <origin xyz="0 0.005 0" rpy="0 0 0" /> <!-- CHECK THIS OFFSET -->
+        <parent link="${name}_camera_rgb_frame" />
+        <child link="${name}_camera_link" />
+      </joint>
+    </xacro:unless>
     <link name="${name}_camera_rgb_frame">
       <inertial>
@@ -73,9 +91,4 @@
       </inertial>
     </link>
-    <joint name="${name}_camera_rgb_optical_joint" type="fixed">
-      <origin xyz="0 0 0" rpy="${-pi/2} 0 ${-pi/2}" />
-      <parent link="${name}_camera_rgb_frame" />
-      <child link="${name}_camera_rgb_optical_frame" />
-    </joint>
     <link name="${name}_camera_rgb_optical_frame">
       <inertial>
@@ -87,6 +100,55 @@
       </inertial>
     </link>
+    <xacro:if value="${has_depth}">
+      <xacro:if value="${has_second_origin}">
+        <!-- attach in this order if rgb attached to parent -->
+        <joint name="${name}_camera_rgb_joint" type="fixed">
+          <origin xyz="0 0 0" rpy="${pi/2} ${-pi/2} 0 " />
+          <parent link="${name}_camera_rgb_optical_frame" />
+          <child link="${name}_camera_rgb_frame" />
+        </joint>
+      </xacro:if>
+      <xacro:unless value="${has_second_origin}">
+        <!-- attach in this order if rgb not attached to parent -->
+        <joint name="${name}_camera_rgb__joint" type="fixed">
+          <origin xyz="0 0 0" rpy="${-pi/2} 0 ${-pi/2}" />
+          <parent link="${name}_camera_rgb_frame" />
+          <child link="${name}_camera_rgb_optical_frame" />
+        </joint>
+      </xacro:unless>
+    </xacro:if>
+    <xacro:unless value="${has_depth}">
+      <!-- attach in this order if rgb attached to parent -->
+      <joint name="${name}_camera_rgb_joint" type="fixed">
+        <origin xyz="0 0 0" rpy="${pi/2} ${-pi/2} 0 " />
+        <parent link="${name}_camera_rgb_optical_frame" />
+        <child link="${name}_camera_rgb_frame" />
+      </joint>
+    </xacro:unless>
+    <xacro:if value="${has_depth}">
+      <xacro:if value="${has_second_origin}">
+        <!-- attach rgb to parent -->
+        <joint name="${name}_camera_rgb_optical_joint" type="fixed">
+          <xacro:insert_block name="second_origin"/>
+          <parent link="${parent}"/>
+          <child link="${name}_camera_rgb_optical_frame" />
+        </joint>
+      </xacro:if>
+    </xacro:if>
+    <xacro:unless value="${has_depth}">
+      <!-- attach rgb to parent -->
+      <joint name="${name}_camera_rgb_optical_joint" type="fixed">
+        <xacro:insert_block name="origin"/>
+        <parent link="${parent}"/>
+        <child link="${name}_camera_rgb_optical_frame" />
+      </joint>
+    </xacro:unless>
     <!-- Gazebo camera sensor for simulation -->
-   <gazebo_camera linkref="${name}_camera_depth_frame" name="${name}" fps="${fps}" hfov="${hfov}" width="${width}" height="${height}" has_depth="1"/>
+    <xacro:if value="${has_depth}">
+      <gazebo_camera linkref="${name}_camera_depth_frame" name="${name}" fps="${fps}" hfov="${hfov}" width="${width}" height="${height}" has_depth="${has_depth}"/>
+    </xacro:if>
+    <xacro:unless value="${has_depth}">
+      <gazebo_camera linkref="${name}_camera_rgb_frame" name="${name}" fps="${fps}" hfov="${hfov}" width="${width}" height="${height}" has_depth="${has_depth}"/>
+    </xacro:unless>
   </xacro:macro>
 </robot>

File: agni_description/urdf/gazebo_camera.urdf.xacro (robot description, xacro)
@@ -1,6 +1,6 @@
 <robot xmlns:controller="http://playerstage.sourceforge.net/gazebo/xmlschema/#controller" xmlns:interface="http://playerstage.sourceforge.net/gazebo/xmlschema/#interface" xmlns:sensor="http://playerstage.sourceforge.net/gazebo/xmlschema/#sensor" xmlns:xacro="http://www.ros.org/wiki/xacro" name="gazebo_camera">
-  <xacro:macro name="gazebo_camera" params="linkref name fps hfov width:=640 height:=480 has_depth:=1">
+  <xacro:macro name="gazebo_camera" params="linkref name fps hfov width:=640 height:=480 has_depth:=0">
     <gazebo reference="${linkref}">
-       <xacro:if value="${has_depth}">
+      <xacro:if value="${has_depth}">
         <sensor type="depth" name="${name}">
           <always_on>true</always_on>
@@ -39,4 +39,41 @@
         </sensor>
       </xacro:if>
+      <xacro:unless value="${has_depth}">
+        <sensor type="camera" name="${name}">
+          <always_on>true</always_on>
+          <update_rate>${fps}</update_rate>
+          <camera>
+            <horizontal_fov>${hfov}</horizontal_fov>
+            <image>
+              <format>B8G8R8</format>
+              <width>${width}</width>
+              <height>${height}</height>
+            </image>
+            <clip>
+              <near>0.05</near>
+              <far>3.0</far>
+            </clip>
+          </camera>
+          <!--noise>
+            <type>gaussian</type>
+            <mean>0.0</mean>
+            <stddev>0.007</stddev>
+          </noise-->
+          <plugin name="camera_controller" filename="libgazebo_ros_camera.so">
+            <cameraName>camera</cameraName>
+            <alwaysOn>true</alwaysOn>
+            <updateRate>20</updateRate>
+            <imageTopicName>image_raw</imageTopicName>
+            <cameraInfoTopicName>camera_info</cameraInfoTopicName>
+            <frameName>${name}_camera_rgb_optical_frame</frameName>
+            <hackBaseline>0.07</hackBaseline>
+            <distortion_k1>0.0</distortion_k1>
+            <distortion_k2>0.0</distortion_k2>
+            <distortion_k3>0.0</distortion_k3>
+            <distortion_t1>0.0</distortion_t1>
+            <distortion_t2>0.0</distortion_t2>
+          </plugin>
+        </sensor>
+      </xacro:unless>
     </gazebo>
   </xacro:macro>

Commit message: Fixed camera spawning with two different calibrations (fixes #7951)

File: agni_description/urdf/camera.urdf.xacro (robot description, xacro)
@@ -3,9 +3,8 @@
   <xacro:include filename="../urdf/gazebo_camera.urdf.xacro"/>
   <!-- do not name the macro 'camera', it conflicts with gazebo camera tag -->
-  <xacro:macro name="camera_body" params="parent name fps hfov width height has_depth *origin has_second_origin:=0 *second_origin">
+  <xacro:macro name="camera_body" params="parent name fps hfov width height hfov2:=- width2:=- height2:=- has_depth *origin has_second_origin:=0 *second_origin">
     <xacro:if value="${1 if 'world' in parent else 0}">
       <link name="${parent}" />
     </xacro:if>
-    <!-- do not name the macro 'camera', it conflicts with gazebo camera tag -->
     <xacro:if value="${has_depth}">
       <!-- attach depth to parent -->
@@ -145,10 +144,18 @@
     </xacro:unless>
     <!-- Gazebo camera sensor for simulation -->
-    <xacro:if value="${has_depth}">
-      <gazebo_camera linkref="${name}_camera_depth_frame" name="${name}" fps="${fps}" hfov="${hfov}" width="${width}" height="${height}" has_depth="${has_depth}"/>
+    <!-- if second origin is given, then create separate sensors (one depth, one rgb) and not a kinect with embedded color/depth -->
+    <xacro:if value="${has_depth and not has_second_origin}">
+      <gazebo_camera linkref="${name}_camera_depth_frame" name="${name}" fps="${fps}" hfov="${hfov}" width="${width}" height="${height}" has_depth="1" has_color="1"/>
     </xacro:if>
-    <xacro:unless value="${has_depth}">
-      <gazebo_camera linkref="${name}_camera_rgb_frame" name="${name}" fps="${fps}" hfov="${hfov}" width="${width}" height="${height}" has_depth="${has_depth}"/>
-    </xacro:unless>
+    <xacro:if value="${has_depth and has_second_origin}">
+      <xacro:property name="second_hfov" value="${hfov if hfov2=='-' else hfov2}" />
+      <xacro:property name="second_width" value="${width if width2=='-' else width2}" />
+      <xacro:property name="second_height" value="${height if height2=='-' else height2}" />
+      <gazebo_camera linkref="${name}_camera_depth_frame" name="${name}" fps="${fps}" hfov="${hfov}" width="${width}" height="${height}" has_depth="1" has_color="0"/>
+      <gazebo_camera linkref="${name}_camera_rgb_frame" name="${name}" fps="${fps}" hfov="${second_hfov}" width="${second_width}" height="${second_height}" has_depth="0" has_color="1"/>
+    </xacro:if>
+    <xacro:if value="${not has_depth}">
+      <gazebo_camera linkref="${name}_camera_rgb_frame" name="${name}" fps="${fps}" hfov="${hfov}" width="${width}" height="${height}" has_depth="0" has_color="1"/>
+    </xacro:if>
   </xacro:macro>
 </robot>

File: agni_description/urdf/gazebo_camera.urdf.xacro (robot description, xacro)
@@ -1,6 +1,6 @@
 <robot xmlns:controller="http://playerstage.sourceforge.net/gazebo/xmlschema/#controller" xmlns:interface="http://playerstage.sourceforge.net/gazebo/xmlschema/#interface" xmlns:sensor="http://playerstage.sourceforge.net/gazebo/xmlschema/#sensor" xmlns:xacro="http://www.ros.org/wiki/xacro" name="gazebo_camera">
-  <xacro:macro name="gazebo_camera" params="linkref name fps hfov width:=640 height:=480 has_depth:=0">
+  <xacro:macro name="gazebo_camera" params="linkref name fps hfov width:=640 height:=480 has_depth:=0 has_color:=1">
     <gazebo reference="${linkref}">
-      <xacro:if value="${has_depth}">
+      <xacro:if value="${has_depth and has_color}">
         <sensor type="depth" name="${name}">
           <always_on>true</always_on>
@@ -19,7 +19,7 @@
           </camera>
           <plugin name="kinect_camera_controller" filename="libgazebo_ros_openni_kinect.so">
-            <cameraName>camera</cameraName>
+            <cameraName>kinect</cameraName>
             <alwaysOn>true</alwaysOn>
-            <updateRate>20</updateRate>
+            <updateRate>0</updateRate>
             <imageTopicName>rgb/image_raw</imageTopicName>
             <depthImageTopicName>depth/image_raw</depthImageTopicName>
@@ -39,5 +39,5 @@
         </sensor>
       </xacro:if>
-      <xacro:unless value="${has_depth}">
+      <xacro:if value="${not has_depth and has_color}">
         <sensor type="camera" name="${name}">
           <always_on>true</always_on>
@@ -63,9 +63,9 @@
             <cameraName>camera</cameraName>
             <alwaysOn>true</alwaysOn>
-            <updateRate>20</updateRate>
-            <imageTopicName>image_raw</imageTopicName>
-            <cameraInfoTopicName>camera_info</cameraInfoTopicName>
+            <updateRate>0</updateRate>
+            <imageTopicName>rgb/image_raw</imageTopicName>
+            <cameraInfoTopicName>rgb/camera_info</cameraInfoTopicName>
             <frameName>${name}_camera_rgb_optical_frame</frameName>
-            <hackBaseline>0.07</hackBaseline>
+            <hackBaseline>0.0</hackBaseline>
             <distortion_k1>0.0</distortion_k1>
             <distortion_k2>0.0</distortion_k2>
@@ -75,5 +75,46 @@
           </plugin>
         </sensor>
-      </xacro:unless>
+      </xacro:if>
+      <xacro:if value="${has_depth and not has_color}">
+        <sensor type="depth" name="${name}">
+          <always_on>true</always_on>
+          <update_rate>${fps}</update_rate>
+          <camera>
+            <horizontal_fov>${hfov}</horizontal_fov>
+            <image>
+              <format>B8G8R8</format>
+              <width>${width}</width>
+              <height>${height}</height>
+            </image>
+            <clip>
+              <near>0.05</near>
+              <far>3.0</far>
+            </clip>
+          </camera>
+          <plugin name="depth_camera_controller" filename="libgazebo_ros_depth_camera.so">
+            <cameraName>camera</cameraName>
+            <alwaysOn>true</alwaysOn>
+            <updateRate>0</updateRate>
+            <imageTopicName>ir/image_raw</imageTopicName>
+            <depthImageTopicName>depth/image_raw</depthImageTopicName>
+            <pointCloudTopicName>depth/points</pointCloudTopicName>
+            <cameraInfoTopicName>ir/camera_info</cameraInfoTopicName>
+            <depthImageCameraInfoTopicName>depth/camera_info</depthImageCameraInfoTopicName>
+            <frameName>${name}_camera_depth_optical_frame</frameName>
+            <baseline>0.1</baseline>
+            <distortion_k1>0.0</distortion_k1>
+            <distortion_k2>0.0</distortion_k2>
+            <distortion_k3>0.0</distortion_k3>
+            <distortion_t1>0.0</distortion_t1>
+            <distortion_t2>0.0</distortion_t2>
+            <pointCloudCutoff>0.4</pointCloudCutoff>
+            <CxPrime>0</CxPrime>
+            <Cx>0</Cx>
+            <Cy>0</Cy>
+            <focalLength>0</focalLength>
+            <hackBaseline>0</hackBaseline>
+          </plugin>
+        </sensor>
+      </xacro:if>
     </gazebo>
   </xacro:macro>

Commit message: Added support for principal point cx/cy parameters in camera_urdf

File: agni_description/urdf/camera.urdf.xacro (robot description, xacro)
@@ -3,5 +3,6 @@
   <xacro:include filename="../urdf/gazebo_camera.urdf.xacro"/>
   <!-- do not name the macro 'camera', it conflicts with gazebo camera tag -->
-  <xacro:macro name="camera_body" params="parent name fps hfov width height hfov2:=- width2:=- height2:=- has_depth *origin has_second_origin:=0 *second_origin">
+  <xacro:macro name="camera_body" params="parent name fps hfov width height cx:=0 cy:=0 hfov2:=- width2:=- height2:=- cx2:=- cy2:=-
+                                          has_depth *origin has_second_origin:=0 *second_origin">
     <xacro:if value="${1 if 'world' in parent else 0}">
       <link name="${parent}" />
@@ -146,5 +147,5 @@
     <!-- if second origin is given, then create separate sensors (one depth, one rgb) and not a kinect with embedded color/depth -->
     <xacro:if value="${has_depth and not has_second_origin}">
-      <gazebo_camera linkref="${name}_camera_depth_frame" name="${name}" fps="${fps}" hfov="${hfov}" width="${width}" height="${height}" has_depth="1" has_color="1"/>
+      <gazebo_camera linkref="${name}_camera_depth_frame" name="${name}" fps="${fps}" hfov="${hfov}" width="${width}" height="${height}" cx="${cx}" cy="${cy}" has_depth="1" has_color="1"/>
     </xacro:if>
     <xacro:if value="${has_depth and has_second_origin}">
@@ -152,9 +153,11 @@
       <xacro:property name="second_width" value="${width if width2=='-' else width2}" />
       <xacro:property name="second_height" value="${height if height2=='-' else height2}" />
-      <gazebo_camera linkref="${name}_camera_depth_frame" name="${name}" fps="${fps}" hfov="${hfov}" width="${width}" height="${height}" has_depth="1" has_color="0"/>
-      <gazebo_camera linkref="${name}_camera_rgb_frame" name="${name}" fps="${fps}" hfov="${second_hfov}" width="${second_width}" height="${second_height}" has_depth="0" has_color="1"/>
+      <xacro:property name="second_cx" value="${cx if cx2=='-' else cx2}" />
+      <xacro:property name="second_cy" value="${cy if cy2=='-' else cy2}" />
+      <gazebo_camera linkref="${name}_camera_depth_frame" name="${name}" fps="${fps}" hfov="${hfov}" width="${width}" height="${height}" cx="${cx}" cy="${cy}" has_depth="1" has_color="0"/>
+      <gazebo_camera linkref="${name}_camera_rgb_frame" name="${name}" fps="${fps}" hfov="${second_hfov}" width="${second_width}" height="${second_height}" cx="${second_cx}" cy="${second_cy}" has_depth="0" has_color="1"/>
     </xacro:if>
     <xacro:if value="${not has_depth}">
-      <gazebo_camera linkref="${name}_camera_rgb_frame" name="${name}" fps="${fps}" hfov="${hfov}" width="${width}" height="${height}" has_depth="0" has_color="1"/>
+      <gazebo_camera linkref="${name}_camera_rgb_frame" name="${name}" fps="${fps}" hfov="${hfov}" width="${width}" height="${height}" cx="${cx}" cy="${cy}" has_depth="0" has_color="1"/>
     </xacro:if>
   </xacro:macro>

File: agni_description/urdf/gazebo_camera.urdf.xacro (robot description, xacro)
@@ -1,4 +1,4 @@
 <robot xmlns:controller="http://playerstage.sourceforge.net/gazebo/xmlschema/#controller" xmlns:interface="http://playerstage.sourceforge.net/gazebo/xmlschema/#interface" xmlns:sensor="http://playerstage.sourceforge.net/gazebo/xmlschema/#sensor" xmlns:xacro="http://www.ros.org/wiki/xacro" name="gazebo_camera">
-  <xacro:macro name="gazebo_camera" params="linkref name fps hfov width:=640 height:=480 has_depth:=0 has_color:=1">
+  <xacro:macro name="gazebo_camera" params="linkref name fps hfov width:=640 height:=480 cx:=0 cy:=0 has_depth:=0 has_color:=1">
     <gazebo reference="${linkref}">
       <xacro:if value="${has_depth and has_color}">
@@ -21,5 +21,5 @@
             <cameraName>kinect</cameraName>
             <alwaysOn>true</alwaysOn>
-            <updateRate>0</updateRate>
+            <updateRate>0</updateRate> <!-- 0 will make the plugin use the sensor update_rate -->
             <imageTopicName>rgb/image_raw</imageTopicName>
             <depthImageTopicName>depth/image_raw</depthImageTopicName>
@@ -36,4 +36,8 @@
             <pointCloudCutoff>0.4</pointCloudCutoff>
             <pointCloudCutoffMax>2.0</pointCloudCutoffMax>
+            <CxPrime>${cx}</CxPrime>
+            <Cx>${cx}</Cx>
+            <Cy>${cy}</Cy>
+            <focalLength>0</focalLength> <!-- 0 forces calculation from hfov -->
           </plugin>
         </sensor>
@@ -63,5 +67,5 @@
             <cameraName>camera</cameraName>
             <alwaysOn>true</alwaysOn>
-            <updateRate>0</updateRate>
+            <updateRate>0</updateRate> <!-- 0 will make the plugin use the sensor update_rate -->
             <imageTopicName>rgb/image_raw</imageTopicName>
             <cameraInfoTopicName>rgb/camera_info</cameraInfoTopicName>
@@ -73,4 +77,8 @@
             <distortion_t1>0.0</distortion_t1>
             <distortion_t2>0.0</distortion_t2>
+            <CxPrime>${cx}</CxPrime>
+            <Cx>${cx}</Cx>
+            <Cy>${cy}</Cy>
+            <focalLength>0</focalLength> <!-- 0 forces calculation from hfov -->
           </plugin>
         </sensor>
@@ -109,8 +117,8 @@
             <distortion_t2>0.0</distortion_t2>
             <pointCloudCutoff>0.4</pointCloudCutoff>
-            <CxPrime>0</CxPrime>
-            <Cx>0</Cx>
-            <Cy>0</Cy>
-            <focalLength>0</focalLength>
+            <CxPrime>${cx}</CxPrime>
+            <Cx>${cx}</Cx>
+            <Cy>${cy}</Cy>
+            <focalLength>0</focalLength> <!-- 0 forces calculation from hfov -->
             <hackBaseline>0</hackBaseline>
           </plugin>
