Commit message: Added a cover to the triangle (camera mounted there)

File: agni_description/urdf/frame-moveable.urdf.xacro (robot description, xacro)
@@ -71,4 +71,12 @@
 				        rpy="0 0 0"/>
 			</xacro:plate>
+			<!-- cover front plate (no visual which would require a mesh) -->
+			<collision>
+					<origin xyz="${(triangle_pos['leftX']+triangle_pos['rightX'])/2.0}
+				               ${triangle_pos['Y']-mtlen/2-mtth/2.0}
+				               ${triangle_pos['Z']-0.01}"
+				        rpy="0 0 0"/>
+					<geometry><box size="${mtlen*2*sin(30/180.0*pi)} ${mtth} ${mtlen*cos(30/180.0*pi)} "/></geometry>
+			</collision>
 			<!-- table plane -->
 			<visual>

Commit message: Added collision box for camera

File: agni_description/urdf/frame-moveable.urdf.xacro (robot description, xacro)
@@ -79,4 +79,12 @@
 					<geometry><box size="${mtlen*2*sin(30/180.0*pi)} ${mtth} ${mtlen*cos(30/180.0*pi)} "/></geometry>
 			</collision>
+			<!-- zone for the camera -->
+			<collision>
+					<origin xyz="${(triangle_pos['leftX']+triangle_pos['rightX'])/2.0}
+				               ${triangle_pos['Y'] - mtlen/2 - 0.04}
+				               ${triangle_pos['Z'] + mount_triangle_length/2*sin(60/180.0*pi) + mount_triangle_thickness/2}"
+				        rpy="0 0 0"/>
+					<geometry><box size="0.2 0.1 0.1"/></geometry>
+			</collision>
 			<!-- table plane -->
 			<visual>
