Commit message: remove virtual collision box: only keep back and top plane

File: agni_description/urdf/frame.urdf.xacro (robot description, xacro)
@@ -104,23 +104,12 @@
 			</collision>
 			<!-- virtual fence -->
-			<!-- left pane -->
+			<!-- top plane -->
 			<collision>
-				<origin xyz="${-(width+thickness)/2} ${depth/2} ${height/2}"
+				<xacro:property name="rearBarY" value="${mountingYpos + mountingspacing/2}"/>
+				<origin xyz="0 ${rearBarY + (depth-rearBarY)/2} ${height+(thickness-0.35)/2}"
 				        rpy="0 0 0"/>
-				<geometry><box size="${thickness} ${depth} ${height}"/></geometry>
+				<geometry><box size="${width} ${depth-rearBarY} ${0.02}"/></geometry>
 			</collision>
-			<!-- right pane -->
-			<collision>
-				<origin xyz="${+(width+thickness)/2} ${depth/2} ${height/2}"
-				        rpy="0 0 0"/>
-				<geometry><box size="${thickness} ${depth} ${height}"/></geometry>
-			</collision>
-			<!-- front pane -->
-			<collision>
-				<origin xyz="0 ${-thickness/2} ${height/2}"
-				        rpy="0 0 0"/>
-				<geometry><box size="${width} ${thickness} ${height}"/></geometry>
-			</collision>
-			<!-- back pane -->
+			<!-- back plane -->
 			<collision>
 				<origin xyz="0 ${depth + thickness/2} ${height/2}"

Commit message: frame: add front plane

File: agni_description/urdf/frame.urdf.xacro (robot description, xacro)
@@ -106,12 +106,17 @@
 			<!-- top plane -->
 			<collision>
-				<xacro:property name="rearBarY" value="${mountingYpos + mountingspacing/2}"/>
-				<origin xyz="0 ${rearBarY + (depth-rearBarY)/2} ${height+(thickness-0.35)/2}"
+				<origin xyz="0 ${depth/2} ${height+(thickness-0.35)/2}"
 				        rpy="0 0 0"/>
-				<geometry><box size="${width} ${depth-rearBarY} ${0.02}"/></geometry>
+				<geometry><box size="${width} ${depth} ${0.02}"/></geometry>
 			</collision>
 			<!-- back plane -->
 			<collision>
 				<origin xyz="0 ${depth + thickness/2} ${height/2}"
+				        rpy="0 0 0"/>
+				<geometry><box size="${width} ${thickness} ${height}"/></geometry>
+			</collision>
+			<!-- front plane -->
+			<collision>
+				<origin xyz="0 ${-thickness/2} ${height/2}"
 				        rpy="0 0 0"/>
 				<geometry><box size="${width} ${thickness} ${height}"/></geometry>

Commit message: Fixed pa10 frame collision (lower ceiling), and hand home/open to not request zeros for xFJ0

File: agni_description/urdf/frame.urdf.xacro (robot description, xacro)
@@ -106,5 +106,5 @@
 			<!-- top plane -->
 			<collision>
-				<origin xyz="0 ${depth/2} ${height+(thickness-0.35)/2}"
+				<origin xyz="0 ${depth/2} ${height+(thickness)/2-0.27}"
 				        rpy="0 0 0"/>
 				<geometry><box size="${width} ${depth} ${0.02}"/></geometry>

Commit message: Added the full fence back for pa10

File: agni_description/urdf/frame.urdf.xacro (robot description, xacro)
@@ -104,4 +104,16 @@
 			</collision>
 			<!-- virtual fence -->
+			<!-- left pane -->
+			<collision>
+				<origin xyz="${-(width+thickness)/2} ${depth/2} ${height/2}"
+				        rpy="0 0 0"/>
+				<geometry><box size="${thickness} ${depth} ${height}"/></geometry>
+			</collision>
+			<!-- right pane -->
+			<collision>
+				<origin xyz="${+(width+thickness)/2} ${depth/2} ${height/2}"
+				        rpy="0 0 0"/>
+				<geometry><box size="${thickness} ${depth} ${height}"/></geometry>
+			</collision>
 			<!-- top plane -->
 			<collision>
