Commit message: len -> length to avoid redefinition of python's len()

File: agni_description/urdf/frame-half.urdf.xacro (robot description, xacro)
@@ -5,13 +5,17 @@
       xmlns:interface="http://playerstage.sourceforge.net/gazebo/xmlschema/#interface">
 	<xacro:include filename="../urdf/materials.urdf.xacro"/>
-	<xacro:macro name="bar" params="thickness len *origin">
+	<xacro:macro name="bar" params="thickness length *origin">
 		<visual>
 			<xacro:insert_block name="origin"/>
-			<geometry><box size="${thickness} ${thickness} ${len}"/></geometry>
+			<geometry>
+				<box size="${thickness} ${thickness} ${length}" />
+			</geometry>
 			<material name="Silver"/>
 		</visual>
 		<collision>
 			<xacro:insert_block name="origin"/>
-			<geometry><box size="${thickness} ${thickness} ${len}"/></geometry>
+			<geometry>
+				<box size="${thickness} ${thickness} ${length}" />
+			</geometry>
 		</collision>
 	</xacro:macro>
@@ -29,47 +33,47 @@
 			</inertial>
 			<!-- horizontal front bar-->
-			<xacro:bar thickness="${thickness}" len="${width}">
+			<xacro:bar thickness="${thickness}" length="${width}">
 				<origin xyz="0 ${thickness/2} ${-thickness/2}" rpy="0 ${-pi/2} 0"/>
 			</xacro:bar>
 			<!-- horizontal rear bar -->
-			<xacro:bar thickness="${thickness}" len="${width}">
+			<xacro:bar thickness="${thickness}" length="${width}">
 				<origin xyz="0 ${depth+thickness/2} ${-thickness/2}" rpy="0 ${-pi/2} 0"/>
 			</xacro:bar>
 			<!-- horizontal rear bar top -->
-			<xacro:bar thickness="${thickness}" len="${width}">
+			<xacro:bar thickness="${thickness}" length="${width}">
 				<origin xyz="0 ${depth+thickness/2} ${height+thickness/2}" rpy="0 ${-pi/2} 0"/>
 			</xacro:bar>
 			<!-- left front pole -->
-			<xacro:bar thickness="${thickness}" len="${thickness+tableHeight}">
+			<xacro:bar thickness="${thickness}" length="${thickness+tableHeight}">
 				<origin xyz="${-(width+thickness)/2} ${thickness/2} ${-(thickness+tableHeight)/2}"/>
 			</xacro:bar>
 			<!-- right front pole -->
-			<xacro:bar thickness="${thickness}" len="${thickness+tableHeight}">
+			<xacro:bar thickness="${thickness}" length="${thickness+tableHeight}">
 				<origin xyz="${+(width+thickness)/2} ${thickness/2} ${-(thickness+tableHeight)/2}"/>
 			</xacro:bar>
 			<!-- left rear pole -->
-			<xacro:bar thickness="${thickness}" len="${height+2*thickness+tableHeight}">
+			<xacro:bar thickness="${thickness}" length="${height+2*thickness+tableHeight}">
 				<origin xyz="${-(width+thickness)/2} ${depth+thickness/2} ${(height-tableHeight)/2}"/>
 			</xacro:bar>
 			<!-- right rear pole -->
-			<xacro:bar thickness="${thickness}" len="${height+2*thickness+tableHeight}">
+			<xacro:bar thickness="${thickness}" length="${height+2*thickness+tableHeight}">
 				<origin xyz="${+(width+thickness)/2} ${depth+thickness/2} ${(height-tableHeight)/2}"/>
 			</xacro:bar>
 			<!-- left side bottom -->
-			<xacro:bar thickness="${thickness}" len="${depth}">
+			<xacro:bar thickness="${thickness}" length="${depth}">
 				<origin xyz="${-(width+thickness)/2} ${depth/2} ${-thickness/2}"
 				        rpy="${-pi/2} 0 0"/>
 			</xacro:bar>
 			<!-- right side bottom -->
-			<xacro:bar thickness="${thickness}" len="${depth}">
+			<xacro:bar thickness="${thickness}" length="${depth}">
 				<origin xyz="${+(width+thickness)/2} ${depth/2} ${-thickness/2}"
 				        rpy="${-pi/2} 0 0"/>
 			</xacro:bar>
 			<!-- left central pole -->
-			<xacro:bar thickness="${thickness}" len="${thickness+tableHeight+(height)/2}">
+			<xacro:bar thickness="${thickness}" length="${thickness+tableHeight+(height)/2}">
 				<origin xyz="${-thickness} ${(depth)/2+2*thickness} ${-(2*tableHeight-height)/4-thickness/2}"/>
 			</xacro:bar>
 			<!-- right central pole -->
-			<xacro:bar thickness="${thickness}" len="${thickness+tableHeight+(height)/2}">
+			<xacro:bar thickness="${thickness}" length="${thickness+tableHeight+(height)/2}">
 				<origin xyz="${thickness} ${(depth)/2+2*thickness} ${-(2*tableHeight-height)/4-thickness/2}"/>
 			</xacro:bar>
@@ -95,6 +99,5 @@
 			</collision>
 			<!-- kuka mount triangle -->
-			<xacro:macro name="plate"
-			             params="thickness:=${mount_triangle_thickness}
+			<xacro:macro name="plate" params="thickness:=${mount_triangle_thickness}
 			                     length:=${mount_triangle_length} *origin">
 				<visual>

File: agni_description/urdf/frame-half_mesh.urdf.xacro (robot description, xacro)
@@ -5,8 +5,10 @@
       xmlns:interface="http://playerstage.sourceforge.net/gazebo/xmlschema/#interface">
 	<xacro:include filename="../urdf/materials.urdf.xacro"/>
-	<xacro:macro name="bar" params="thickness len *origin">
+	<xacro:macro name="bar" params="thickness length *origin">
 		<visual>
 			<xacro:insert_block name="origin"/>
-			<geometry><box size="${thickness} ${thickness} ${len}"/></geometry>
+			<geometry>
+				<box size="${thickness} ${thickness} ${length}" />
+			</geometry>
 			<material name="Silver"/>
 		</visual>
@@ -25,47 +27,47 @@
 			</inertial>
 			<!-- horizontal front bar-->
-			<xacro:bar thickness="${thickness}" len="${width}">
+			<xacro:bar thickness="${thickness}" length="${width}">
 				<origin xyz="0 ${thickness/2} ${-thickness/2}" rpy="0 ${-pi/2} 0"/>
 			</xacro:bar>
 			<!-- horizontal rear bar -->
-			<xacro:bar thickness="${thickness}" len="${width}">
+			<xacro:bar thickness="${thickness}" length="${width}">
 				<origin xyz="0 ${depth+thickness/2} ${-thickness/2}" rpy="0 ${-pi/2} 0"/>
 			</xacro:bar>
 			<!-- horizontal rear bar top -->
-			<xacro:bar thickness="${thickness}" len="${width}">
+			<xacro:bar thickness="${thickness}" length="${width}">
 				<origin xyz="0 ${depth+thickness/2} ${height+thickness/2}" rpy="0 ${-pi/2} 0"/>
 			</xacro:bar>
 			<!-- left front pole -->
-			<xacro:bar thickness="${thickness}" len="${thickness+tableHeight}">
+			<xacro:bar thickness="${thickness}" length="${thickness+tableHeight}">
 				<origin xyz="${-(width+thickness)/2} ${thickness/2} ${-(thickness+tableHeight)/2}"/>
 			</xacro:bar>
 			<!-- right front pole -->
-			<xacro:bar thickness="${thickness}" len="${thickness+tableHeight}">
+			<xacro:bar thickness="${thickness}" length="${thickness+tableHeight}">
 				<origin xyz="${+(width+thickness)/2} ${thickness/2} ${-(thickness+tableHeight)/2}"/>
 			</xacro:bar>
 			<!-- left rear pole -->
-			<xacro:bar thickness="${thickness}" len="${height+2*thickness+tableHeight}">
+			<xacro:bar thickness="${thickness}" length="${height+2*thickness+tableHeight}">
 				<origin xyz="${-(width+thickness)/2} ${depth+thickness/2} ${(height-tableHeight)/2}"/>
 			</xacro:bar>
 			<!-- right rear pole -->
-			<xacro:bar thickness="${thickness}" len="${height+2*thickness+tableHeight}">
+			<xacro:bar thickness="${thickness}" length="${height+2*thickness+tableHeight}">
 				<origin xyz="${+(width+thickness)/2} ${depth+thickness/2} ${(height-tableHeight)/2}"/>
 			</xacro:bar>
 			<!-- left side bottom -->
-			<xacro:bar thickness="${thickness}" len="${depth}">
+			<xacro:bar thickness="${thickness}" length="${depth}">
 				<origin xyz="${-(width+thickness)/2} ${depth/2} ${-thickness/2}"
 				        rpy="${-pi/2} 0 0"/>
 			</xacro:bar>
 			<!-- right side bottom -->
-			<xacro:bar thickness="${thickness}" len="${depth}">
+			<xacro:bar thickness="${thickness}" length="${depth}">
 				<origin xyz="${+(width+thickness)/2} ${depth/2} ${-thickness/2}"
 				        rpy="${-pi/2} 0 0"/>
 			</xacro:bar>
 			<!-- left central pole -->
-			<xacro:bar thickness="${thickness}" len="${thickness+tableHeight+(height)/2}">
+			<xacro:bar thickness="${thickness}" length="${thickness+tableHeight+(height)/2}">
 				<origin xyz="${-thickness} ${(depth)/2+2*thickness} ${-(2*tableHeight-height)/4-thickness/2}"/>
 			</xacro:bar>
 			<!-- right central pole -->
-			<xacro:bar thickness="${thickness}" len="${thickness+tableHeight+(height)/2}">
+			<xacro:bar thickness="${thickness}" length="${thickness+tableHeight+(height)/2}">
 				<origin xyz="${thickness} ${(depth)/2+2*thickness} ${-(2*tableHeight-height)/4-thickness/2}"/>
 			</xacro:bar>
@@ -94,6 +96,5 @@
 			</collision>
 			<!-- kuka mount triangle -->
-			<xacro:macro name="plate"
-			             params="thickness:=${mount_triangle_thickness}
+			<xacro:macro name="plate" params="thickness:=${mount_triangle_thickness}
 			                     length:=${mount_triangle_length} *origin">
 				<visual>

File: agni_description/urdf/frame-moveable.urdf.xacro (robot description, xacro)
@@ -5,13 +5,13 @@
       xmlns:interface="http://playerstage.sourceforge.net/gazebo/xmlschema/#interface">
 	<xacro:include filename="../urdf/materials.urdf.xacro"/>
-	<xacro:macro name="bar" params="thickness len *origin">
+	<xacro:macro name="bar" params="thickness length *origin">
 		<visual>
 			<xacro:insert_block name="origin"/>
-			<geometry><box size="${thickness} ${thickness} ${len}"/></geometry>
+			<geometry><box size="${thickness} ${thickness} ${length}"/></geometry>
 			<material name="Silver"/>
 		</visual>
 		<collision>
 			<xacro:insert_block name="origin"/>
-			<geometry><box size="${thickness} ${thickness} ${len}"/></geometry>
+			<geometry><box size="${thickness} ${thickness} ${length}"/></geometry>
 		</collision>
 	</xacro:macro>
@@ -29,9 +29,9 @@
 			</inertial>
 			<!-- left central pole -->
-			<xacro:bar thickness="${thickness}" len="${thickness+tableHeight+(height)/2}">
+			<xacro:bar thickness="${thickness}" length="${thickness+tableHeight+(height)/2}">
 				<origin xyz="${-thickness} ${pole_front_dist+thickness/2} ${-(2*tableHeight-height)/4-thickness/2}"/>
 			</xacro:bar>
 			<!-- right central pole -->
-			<xacro:bar thickness="${thickness}" len="${thickness+tableHeight+(height)/2}">
+			<xacro:bar thickness="${thickness}" length="${thickness+tableHeight+(height)/2}">
 				<origin xyz="${thickness} ${pole_front_dist+thickness/2} ${-(2*tableHeight-height)/4-thickness/2}"/>
 			</xacro:bar>

File: agni_description/urdf/frame.urdf.xacro (robot description, xacro)
@@ -2,19 +2,25 @@
 <root xmlns:xacro="http://www.ros.org/wiki/xacro">
 	<xacro:include filename="../urdf/materials.urdf.xacro"/>
-	<xacro:macro name="barcollision" params="thickness len *origin">
+	<xacro:macro name="barcollision" params="thickness length *origin">
 		<visual>
 			<xacro:insert_block name="origin"/>
-			<geometry><box size="${thickness} ${thickness} ${len}"/></geometry>
+			<geometry>
+				<box size="${thickness} ${thickness} ${length}" />
+			</geometry>
 			<material name="Silver"/>
 		</visual>
 		<collision>
 			<xacro:insert_block name="origin"/>
-			<geometry><box size="${thickness} ${thickness} ${len}"/></geometry>
+			<geometry>
+				<box size="${thickness} ${thickness} ${length}" />
+			</geometry>
 		</collision>
 	</xacro:macro>
-	<xacro:macro name="bar" params="thickness len *origin">
+	<xacro:macro name="bar" params="thickness length *origin">
 		<visual>
 			<xacro:insert_block name="origin"/>
-			<geometry><box size="${thickness} ${thickness} ${len}"/></geometry>
+			<geometry>
+				<box size="${thickness} ${thickness} ${length}" />
+			</geometry>
 			<material name="Silver"/>
 		</visual>
@@ -33,18 +39,18 @@
 			</inertial>
 			<!-- horizontal front bar-->
-			<xacro:bar thickness="${thickness}" len="${width}">
+			<xacro:bar thickness="${thickness}" length="${width}">
 				<origin xyz="0 ${-thickness/2} ${-thickness/2}" rpy="0 ${-pi/2} 0"/>
 			</xacro:bar>
 			<!-- horizontal rear bar -->
-			<xacro:bar thickness="${thickness}" len="${width}">
+			<xacro:bar thickness="${thickness}" length="${width}">
 				<origin xyz="0 ${depth+thickness/2} ${-thickness/2}" rpy="0 ${-pi/2} 0"/>
 			</xacro:bar>
 			<!-- robot mounting bars -->
 			<!-- horizontal front bar top -->
-			<xacro:bar thickness="${thickness}" len="${width}">
+			<xacro:bar thickness="${thickness}" length="${width}">
 				<origin xyz="0 ${mountingYpos-mountingspacing/2 + thickness/2} ${height+thickness/2}" rpy="0 ${-pi/2} 0"/>
 			</xacro:bar>
 			<!-- horizontal rear bar top -->
-			<xacro:bar thickness="${thickness}" len="${width}">
+			<xacro:bar thickness="${thickness}" length="${width}">
 				<origin xyz="0 ${mountingYpos+mountingspacing/2 - thickness/2} ${height+thickness/2}" rpy="0 ${-pi/2} 0"/>
 			</xacro:bar>
@@ -56,36 +62,36 @@
 			</collision>
 			<!-- left front pole -->
-			<xacro:bar thickness="${thickness}" len="${height+2*thickness+tableHeight}">
+			<xacro:bar thickness="${thickness}" length="${height+2*thickness+tableHeight}">
 				<origin xyz="${-(width+thickness)/2} ${-thickness/2} ${(height-tableHeight)/2}"/>
 			</xacro:bar>
 			<!-- right front pole -->
-			<xacro:bar thickness="${thickness}" len="${height+2*thickness+tableHeight}">
+			<xacro:bar thickness="${thickness}" length="${height+2*thickness+tableHeight}">
 				<origin xyz="${+(width+thickness)/2} ${-thickness/2} ${(height-tableHeight)/2}"/>
 			</xacro:bar>
 			<!-- left rear pole -->
-			<xacro:bar thickness="${thickness}" len="${height+2*thickness+tableHeight}">
+			<xacro:bar thickness="${thickness}" length="${height+2*thickness+tableHeight}">
 				<origin xyz="${-(width+thickness)/2} ${depth+thickness/2} ${(height-tableHeight)/2}"/>
 			</xacro:bar>
 			<!-- right rear pole -->
-			<xacro:bar thickness="${thickness}" len="${height+2*thickness+tableHeight}">
+			<xacro:bar thickness="${thickness}" length="${height+2*thickness+tableHeight}">
 				<origin xyz="${+(width+thickness)/2} ${depth+thickness/2} ${(height-tableHeight)/2}"/>
 			</xacro:bar>
 			<!-- left side bottom -->
-			<xacro:bar thickness="${thickness}" len="${depth}">
+			<xacro:bar thickness="${thickness}" length="${depth}">
 				<origin xyz="${-(width+thickness)/2} ${depth/2} ${-thickness/2}"
 				        rpy="${-pi/2} 0 0"/>
 			</xacro:bar>
 			<!-- right side bottom -->
-			<xacro:bar thickness="${thickness}" len="${depth}">
+			<xacro:bar thickness="${thickness}" length="${depth}">
 				<origin xyz="${+(width+thickness)/2} ${depth/2} ${-thickness/2}"
 				        rpy="${-pi/2} 0 0"/>
 			</xacro:bar>
 			<!-- left side top -->
-			<xacro:bar thickness="${thickness}" len="${depth}">
+			<xacro:bar thickness="${thickness}" length="${depth}">
 				<origin xyz="${-(width+thickness)/2} ${depth/2} ${height+thickness/2}"
 				        rpy="${-pi/2} 0 0"/>
 			</xacro:bar>
 			<!-- right side top -->
-			<xacro:bar thickness="${thickness}" len="${depth}">
+			<xacro:bar thickness="${thickness}" length="${depth}">
 				<origin xyz="${+(width+thickness)/2} ${depth/2} ${height+thickness/2}"
 				        rpy="${-pi/2} 0 0"/>
