Commit message: Added support for bimanual hand only attached to parent (creates a parent to tool mount if arm is not instantiated) Added calibration for two hands (move them appart so they do not collide is attached to parent such as world)

File: agni_description/urdf/helpers.urdf.xacro (robot description, xacro)
@@ -58,4 +58,8 @@
       <xacro:property name="tool_parent" value="${arm_prefix_}tool_mount"/>
     </xacro:if>
+    <xacro:unless value="${arm_type not in ['','-']}">
+      <!-- use parent as tool mount -->
+      <xacro:property name="tool_parent" value="${parent}"/>
+    </xacro:unless>
     <xacro:if value="${tool_type not in ['','-']}">
       <!-- load tool calibration and instantiate tool -->

Commit message: fixed checking availability of props entries

File: agni_description/urdf/helpers.urdf.xacro (robot description, xacro)
@@ -3,5 +3,5 @@
   <xacro:macro name="arm" params="type prefix:='' parent:='world' controller *origin">
     <xacro:property name="prefix_" value="${prefix + '_' if prefix else ''}"/>
-    <xacro:property name="props" value="${settings['arms'][type]['props'] if settings['arms'][type]['props'] else dict()}"/>
+    <xacro:property name="props" value="${settings['arms'][type]['props'] if 'props' in settings['arms'][type] else dict()}"/>
     <!-- include urdf file and call macro to generate arm -->
     <xacro:include filename="${settings['arms'][type]['file']}"/>
@@ -19,5 +19,5 @@
   <xacro:macro name="tool" params="type prefix:='' parent:='world' *origin">
     <xacro:property name="prefix_" value="${prefix + '_' if prefix else ''}"/>
-    <xacro:property name="props" value="${settings['tools'][type]['props'] if settings['tools'][type]['props'] else dict()}"/>
+    <xacro:property name="props" value="${settings['tools'][type]['props'] if 'props' in settings['tools'][type] else dict()}"/>
     <!-- include urdf file and call macro to generate tool -->
     <xacro:include filename="${settings['tools'][type]['file']}"/>
@@ -47,6 +47,8 @@
     <xacro:property name="arm_prefix_" value="${arm_prefix + '_' if arm_prefix else ''}"/>
     <xacro:property name="tool_prefix_" value="${tool_prefix + '_' if tool_prefix else ''}"/>
-    <!-- add payload mass if relevant -->
-    <xacro:if value="${tool_type not in ['','-']}">
+    <!-- add payload mass if available -->
+    <xacro:if value="${(tool_type not in ['','-']) and
+                     ('props' in settings['tools'][tool_type]) and
+                     ('mass' in settings['tools'][tool_type]['props'])}">
       <xacro:property name="payload_mass" value="${settings['tools'][tool_type]['props']['mass']}"/>
       <xacro:property name="payload_cog" value="${settings['tools'][tool_type]['props']['cog']}"/>

Commit message: Use new yaml parameter to specify cal_file and avoid many symlinks

File: agni_description/urdf/helpers.urdf.xacro (robot description, xacro)
@@ -56,6 +56,22 @@
     <xacro:property name="tool_parent" value="${parent}"/>
     <xacro:if value="${arm_type not in ['','-']}">
-      <!-- load arm calibration and instantiate arm -->
-      <xacro:include filename="../calibration/$(arg CALIB)/${arm_type}_cal.xml"/>
+      <!-- load arm calibration -->
+      <xacro:if value="${('cal_file' in settings['arms'][arm_type])}">
+        <!-- auto = use tool name for calib_file -->
+        <xacro:if value="${('auto' in settings['arms'][arm_type]['cal_file'])}">
+          <!-- in the future, test if exist and have a fallback to default -->
+          <xacro:property name="arm_cal_filename" value="../calibration/$(arg CALIB)/${arm_type}_cal.xml"/>
+        </xacro:if>
+        <xacro:unless value="${('auto' in settings['arms'][arm_type]['cal_file'])}">
+          <!-- in the future, test if exist and have a fallback to default -->
+          <xacro:property name="arm_cal_filename" value="../calibration/$(arg CALIB)/${settings['arms'][arm_type]['cal_file']}"/>
+        </xacro:unless>
+      </xacro:if>
+      <!-- no cal_file given use origin -->
+      <xacro:unless value="${('cal_file' in settings['arms'][arm_type])}">
+        <xacro:property name="arm_cal_filename" value="../calibration/$(arg CALIB)/origin.xml"/>
+      </xacro:unless>
+      <xacro:include filename="${arm_cal_filename}"/>
+      <!-- instantiate arm -->
       <xacro:arm type="${arm_type}" prefix="${arm_prefix}" controller="$(arg SIM)">
         <origin xyz="${cal_x} ${cal_y} ${cal_z}"
@@ -70,6 +86,22 @@
     </xacro:unless>
     <xacro:if value="${tool_type not in ['','-']}">
-      <!-- load tool calibration and instantiate tool -->
-      <xacro:include filename="../calibration/$(arg CALIB)/${tool_type}_cal.xml"/>
+      <!-- load tool calibration -->
+      <xacro:if value="${('cal_file' in settings['tools'][tool_type])}">
+        <!-- auto = use tool name for calib_file -->
+        <xacro:if value="${('auto' in settings['tools'][tool_type]['cal_file'])}">
+          <!-- in the future, test if exist and have a fallback to default -->
+          <xacro:property name="tool_cal_filename" value="../calibration/$(arg CALIB)/${tool_type}_cal.xml"/>
+        </xacro:if>
+        <xacro:unless value="${('auto' in settings['tools'][tool_type]['cal_file'])}">
+          <!-- in the future, test if exist and have a fallback to default -->
+          <xacro:property name="tool_cal_filename" value="../calibration/$(arg CALIB)/${settings['tools'][tool_type]['cal_file']}"/>
+        </xacro:unless>
+      </xacro:if>
+      <!-- no cal_file given use origin -->
+      <xacro:unless value="${('cal_file' in settings['tools'][tool_type])}">
+        <xacro:property name="tool_cal_filename" value="../calibration/$(arg CALIB)/origin.xml"/>
+      </xacro:unless>
+      <xacro:include filename="${tool_cal_filename}"/>
+      <!-- instantiate tool -->
       <xacro:tool type="${tool_type}" prefix="${tool_prefix}" parent="${tool_parent}">
         <origin xyz="${cal_x} ${cal_y} ${cal_z}"

Commit message: Exploit dotified dict syntax
settings['xxx'] -> settings.xxx

File: agni_description/urdf/helpers.urdf.xacro (robot description, xacro)
@@ -3,8 +3,8 @@
   <xacro:macro name="arm" params="type prefix:='' parent:='world' controller *origin">
     <xacro:property name="prefix_" value="${prefix + '_' if prefix else ''}"/>
-    <xacro:property name="props" value="${settings['arms'][type]['props'] if 'props' in settings['arms'][type] else dict()}"/>
+    <xacro:property name="props" value="${settings.arms[type].props if 'props' in settings.arms[type] else dict()}"/>
     <!-- include urdf file and call macro to generate arm -->
-    <xacro:include filename="${settings['arms'][type]['file']}"/>
-    <xacro:call macro="${settings['arms'][type]['macro']}"
+    <xacro:include filename="${settings.arms[type].file}"/>
+    <xacro:call macro="${settings.arms[type].macro}"
                 prefix="${prefix}" controller="${controller}"/>
     <!-- attach arm to parent link -->
@@ -19,8 +19,8 @@
   <xacro:macro name="tool" params="type prefix:='' parent:='world' *origin">
     <xacro:property name="prefix_" value="${prefix + '_' if prefix else ''}"/>
-    <xacro:property name="props" value="${settings['tools'][type]['props'] if 'props' in settings['tools'][type] else dict()}"/>
+    <xacro:property name="props" value="${settings.tools[type].props if 'props' in settings.tools[type] else dict()}"/>
     <!-- include urdf file and call macro to generate tool -->
-    <xacro:include filename="${settings['tools'][type]['file']}"/>
-    <xacro:call macro="${settings['tools'][type]['macro']}"
+    <xacro:include filename="${settings.tools[type].file}"/>
+    <xacro:call macro="${settings.tools[type].macro}"
                 prefix="${prefix}" />
     <!-- attach tool to parent link -->
@@ -28,5 +28,5 @@
       <joint name="${prefix_}tool_mount" type="fixed">
         <parent link="${parent}"/>
-        <child link="${prefix_}${settings['tools'][type]['mount']}"/>
+        <child link="${prefix_}${settings.tools[type].mount}"/>
         <xacro:insert_block name="origin" />
       </joint>
@@ -49,25 +49,25 @@
     <!-- add payload mass if available -->
     <xacro:if value="${(tool_type not in ['','-']) and
-                     ('props' in settings['tools'][tool_type]) and
-                     ('mass' in settings['tools'][tool_type]['props'])}">
-      <xacro:property name="payload_mass" value="${settings['tools'][tool_type]['props']['mass']}"/>
-      <xacro:property name="payload_cog" value="${settings['tools'][tool_type]['props']['cog']}"/>
+                     ('props' in settings.tools[tool_type]) and
+                     ('mass' in settings.tools[tool_type].props)}">
+      <xacro:property name="payload_mass" value="${settings.tools[tool_type].props['mass']}"/>
+      <xacro:property name="payload_cog" value="${settings.tools[tool_type].props['cog']}"/>
     </xacro:if>
     <xacro:property name="tool_parent" value="${parent}"/>
     <xacro:if value="${arm_type not in ['','-']}">
       <!-- load arm calibration -->
-      <xacro:if value="${('cal_file' in settings['arms'][arm_type])}">
+      <xacro:if value="${('cal_file' in settings.arms[arm_type])}">
         <!-- auto = use tool name for calib_file -->
-        <xacro:if value="${('auto' in settings['arms'][arm_type]['cal_file'])}">
+        <xacro:if value="${('auto' in settings.arms[arm_type].cal_file)}">
           <!-- in the future, test if exist and have a fallback to default -->
           <xacro:property name="arm_cal_filename" value="../calibration/$(arg CALIB)/${arm_type}_cal.xml"/>
         </xacro:if>
-        <xacro:unless value="${('auto' in settings['arms'][arm_type]['cal_file'])}">
+        <xacro:unless value="${('auto' in settings.arms[arm_type].cal_file)}">
           <!-- in the future, test if exist and have a fallback to default -->
-          <xacro:property name="arm_cal_filename" value="../calibration/$(arg CALIB)/${settings['arms'][arm_type]['cal_file']}"/>
+          <xacro:property name="arm_cal_filename" value="../calibration/$(arg CALIB)/${settings.arms[arm_type].cal_file}"/>
         </xacro:unless>
       </xacro:if>
       <!-- no cal_file given use origin -->
-      <xacro:unless value="${('cal_file' in settings['arms'][arm_type])}">
+      <xacro:unless value="${('cal_file' in settings.arms[arm_type])}">
         <xacro:property name="arm_cal_filename" value="../calibration/$(arg CALIB)/origin.xml"/>
       </xacro:unless>
@@ -87,17 +87,17 @@
     <xacro:if value="${tool_type not in ['','-']}">
       <!-- load tool calibration -->
-      <xacro:if value="${('cal_file' in settings['tools'][tool_type])}">
+      <xacro:if value="${('cal_file' in settings.tools[tool_type])}">
         <!-- auto = use tool name for calib_file -->
-        <xacro:if value="${('auto' in settings['tools'][tool_type]['cal_file'])}">
+        <xacro:if value="${('auto' in settings.tools[tool_type].cal_file)}">
           <!-- in the future, test if exist and have a fallback to default -->
           <xacro:property name="tool_cal_filename" value="../calibration/$(arg CALIB)/${tool_type}_cal.xml"/>
         </xacro:if>
-        <xacro:unless value="${('auto' in settings['tools'][tool_type]['cal_file'])}">
+        <xacro:unless value="${('auto' in settings.tools[tool_type].cal_file)}">
           <!-- in the future, test if exist and have a fallback to default -->
-          <xacro:property name="tool_cal_filename" value="../calibration/$(arg CALIB)/${settings['tools'][tool_type]['cal_file']}"/>
+          <xacro:property name="tool_cal_filename" value="../calibration/$(arg CALIB)/${settings.tools[tool_type].cal_file}"/>
         </xacro:unless>
       </xacro:if>
       <!-- no cal_file given use origin -->
-      <xacro:unless value="${('cal_file' in settings['tools'][tool_type])}">
+      <xacro:unless value="${('cal_file' in settings.tools[tool_type])}">
         <xacro:property name="tool_cal_filename" value="../calibration/$(arg CALIB)/origin.xml"/>
       </xacro:unless>

Commit message: Simplify dict access with fallback
Replace regex:
([^} ]*?\w\.\w+?\[\w+?\])\.(\w+) +if +'\2' +in +\1 +else +([^}]*)
with:
$1.get('$2', $3)

File: agni_description/urdf/helpers.urdf.xacro (robot description, xacro)
@@ -3,5 +3,5 @@
   <xacro:macro name="arm" params="type prefix:='' parent:='world' controller *origin">
     <xacro:property name="prefix_" value="${prefix + '_' if prefix else ''}"/>
-    <xacro:property name="props" value="${settings.arms[type].props if 'props' in settings.arms[type] else dict()}"/>
+    <xacro:property name="props" value="${settings.arms[type].get('props', dict())}" />
     <!-- include urdf file and call macro to generate arm -->
     <xacro:include filename="${settings.arms[type].file}"/>
@@ -19,5 +19,5 @@
   <xacro:macro name="tool" params="type prefix:='' parent:='world' *origin">
     <xacro:property name="prefix_" value="${prefix + '_' if prefix else ''}"/>
-    <xacro:property name="props" value="${settings.tools[type].props if 'props' in settings.tools[type] else dict()}"/>
+    <xacro:property name="props" value="${settings.tools[type].get('props', dict())}" />
     <!-- include urdf file and call macro to generate tool -->
     <xacro:include filename="${settings.tools[type].file}"/>
