Commit message: Fixed ati collision model

File: agni_description/models/ati_sensor.urdf.xacro (robot description, xacro)
@@ -20,5 +20,5 @@
       </visual>
       <collision>
-        <origin xyz="0 0 0" rpy="0 0 0"/>
+        <origin xyz="0 0 ${ati_offset/2.0}" rpy="0 0 0"/>
         <geometry>
           <cylinder radius="0.038" length="${ati_offset}" />
