Commit message: Added a new setup with poking stick and myrmex Converted new models to macros

File: agni_description/models/myrmex_quick_mount.urdf.xacro (robot description, xacro)
@@ -1,4 +1,5 @@
 <?xml version="1.0"?>
 <robot name="myrmex_quick_mount" xmlns:xacro="http://www.ros.org/wiki/xacro">
+  <xacro:macro name="myrmex_quick_mount" params="">
   <link name="myrmex_quick_mount">
      <visual>
@@ -19,3 +20,4 @@
   <gazebo reference="myrmex_quick_mount">
   </gazebo>
+    </xacro:macro>
 </robot>

File: agni_description/models/poking_stick.urdf.xacro (robot description, xacro)
@@ -1,5 +1,5 @@
 <?xml version="1.0"?>
 <robot name="poking_stick" xmlns:xacro="http://www.ros.org/wiki/xacro">
-<xacro:include filename="$(find agni_description)/urdf/materials.urdf.xacro"/>
+  <xacro:macro name="poking_stick" params="">
   <link name="poking_stick">
      <visual>
@@ -20,3 +20,4 @@
   <gazebo reference="poking_stick">
   </gazebo>
+  </xacro:macro>
 </robot>

Commit message: Added collision to new models

File: agni_description/models/myrmex_quick_mount.urdf.xacro (robot description, xacro)
@@ -3,18 +3,33 @@
   <xacro:macro name="myrmex_quick_mount" params="">
   <link name="myrmex_quick_mount">
-     <visual>
-    <origin xyz="0 0 0"
+    <visual>
+      <origin xyz="0 0 0"
           rpy="0 0 0"/>
-    <geometry>
+      <geometry>
         <mesh scale="0.001 0.001 0.001"
 					 filename="package://agni_description/models/meshes/myrmex_quick_mount.dae"/>
-    </geometry>
-   </visual>
-     	 <!--
-   <collision>
-      <origin xyz="0 0 0"
+      </geometry>
+    </visual>
+    <collision>
+      <origin xyz="0 0 0.00797"
           rpy="0 0 0"/>
-      <geometry><box size="${width+2*thickness} ${0.01} ${height+0.4+2*thickness}"/></geometry>
-    </collision>-->
+      <geometry>
+        <cylinder radius="0.06725" length="0.01584"/>
+      </geometry>
+    </collision>
+     <collision>
+      <origin xyz="0 0 0.02159"
+          rpy="0 0 0"/>
+      <geometry>
+        <cylinder radius="0.060" length="0.0115"/>
+      </geometry>
+    </collision>
+    <collision>
+      <origin xyz="0 0 0.03034"
+          rpy="0 0 0"/>
+        <geometry>
+          <box size="0.095 0.095 0.006"/>
+        </geometry>
+    </collision>
   </link>
   <gazebo reference="myrmex_quick_mount">

File: agni_description/models/poking_stick.urdf.xacro (robot description, xacro)
@@ -3,18 +3,33 @@
   <xacro:macro name="poking_stick" params="">
   <link name="poking_stick">
-     <visual>
-    <origin xyz="0 0 0"
+    <visual>
+      <origin xyz="0 0 0"
           rpy="0 0 0"/>
-    <geometry>
+      <geometry>
         <mesh scale="0.001 0.001 0.001"
 					 filename="package://agni_description/models/meshes/poking_stick.dae"/>
-    </geometry>
-   </visual>
-     	 <!--
-   <collision>
-      <origin xyz="0 0 0"
+      </geometry>
+    </visual>
+    <collision>
+      <origin xyz="0 0 0.0075"
           rpy="0 0 0"/>
-      <geometry><box size="${width+2*thickness} ${0.01} ${height+0.4+2*thickness}"/></geometry>
-    </collision>-->
+      <geometry>
+        <cylinder radius="0.06725" length="0.015"/>
+      </geometry>
+    </collision>
+    <collision>
+      <origin xyz="0 0 0.08875"
+          rpy="0 0 0"/>
+      <geometry>
+        <cylinder radius="0.0075" length="0.1475"/>
+      </geometry>
+    </collision>
+    <collision>
+      <origin xyz="0 0 0.1625"
+          rpy="0 0 0"/>
+      <geometry>
+        <sphere radius="0.0075"/>
+      </geometry>
+    </collision>
   </link>
   <gazebo reference="poking_stick">

Commit message: Reworked end-effector selection. New argument to select side of end-effector is necessary to be able to load two left hands or a left hand on a right arm Added pa10 support, fixed is_right usage, fixed frame loading Added myrmex as end-effector Cleaned up and added comments

File: agni_description/models/myrmex_quick_mount.urdf.xacro (robot description, xacro)
@@ -1,6 +1,6 @@
 <?xml version="1.0"?>
 <robot name="myrmex_quick_mount" xmlns:xacro="http://www.ros.org/wiki/xacro">
-  <xacro:macro name="myrmex_quick_mount" params="">
-  <link name="myrmex_quick_mount">
+  <xacro:macro name="myrmex_quick_mount" params="prefix">
+  <link name="${prefix}myrmex_quick_mount">
     <visual>
       <origin xyz="0 0 0"
@@ -33,5 +33,5 @@
     </collision>
   </link>
-  <gazebo reference="myrmex_quick_mount">
+  <gazebo reference="${prefix}myrmex_quick_mount">
   </gazebo>
     </xacro:macro>

File: agni_description/robots/left_myrmex_ee.urdf.xacro (robot description, xacro)
@@ -1,5 +1,5 @@
 <?xml version="1.0"?>
 <robot xmlns:xacro="http://www.ros.org/wiki/xacro">
-  <xacro:include filename="$(find agni_description)/models/poking_stick.urdf.xacro" />
+  <xacro:include filename="$(find agni_description)/models/myrmex_quick_mount.urdf.xacro" />
   <xacro:property name="cal_left_ee_x" value="0.0" />
   <xacro:property name="cal_left_ee_y" value="0.0" />
@@ -8,10 +8,10 @@
   <xacro:property name="cal_left_ee_pitch" value="0.0" />
   <xacro:property name="cal_left_ee_roll" value="0.0" />
-  <xacro:property name="l_ee_base_link" value="poking_stick" />
-  <xacro:macro name="right_poking_stick" params="prefix" >
-    <xacro:poking_stick prefix="${prefix}" />
+  <xacro:property name="l_ee_base_link" value="myrmex_quick_mount" />
+  <xacro:macro name="right_myrmex" params="prefix" >
+    <xacro:myrmex_quick_mount prefix="${prefix}" />
   </xacro:macro>
-  <xacro:macro name="left_poking_stick" params="prefix" >
-    <xacro:poking_stick prefix="${prefix}" />
+  <xacro:macro name="left_myrmex" params="prefix" >
+    <xacro:myrmex_quick_mount prefix="${prefix}" />
   </xacro:macro>
 </robot>

File: agni_description/robots/left_shadow_muscle_ee.urdf.xacro (robot description, xacro)
@@ -7,5 +7,5 @@
   <xacro:property name="cal_left_ee_x" value="0.0" />
   <xacro:property name="cal_left_ee_y" value="0.0" />
-  <xacro:property name="cal_left_ee_z" value="0.0151" />
+  <xacro:property name="cal_left_ee_z" value="0.0" />
   <xacro:property name="cal_left_ee_yaw" value="0.0" />
   <xacro:property name="cal_left_ee_pitch" value="0.0" />

File: agni_description/robots/pa10_anytool.urdf.xacro (robot description, xacro)
@@ -1,8 +1,10 @@
 <?xml version="1.0"?>
-<robot name="kuka_anytool"
+<robot name="pa10_anytool"
      xmlns:xacro="http://www.ros.org/wiki/xacro">
   <!-- all necessary includes for end-effectors must be done outside -->
-  <xacro:include filename="$(find agni_description)/kuka/kuka.urdf.xacro"/>
-  <xacro:include filename="$(find agni_description)/kuka/lwr_controllers.gazebo.xacro"/>
+  <xacro:include filename="$(find agni_description)/pa10/pa10-a.urdf.xacro"/>
+  <xacro:include filename="$(find agni_description)/pa10/pa10-c.urdf.xacro"/>
+  <xacro:include filename="$(find agni_description)/pa10/pa10_shadow_controller_manager.xacro"/>
+  <xacro:include filename="$(find agni_description)/calibration/pa10_cal.xml"/>
   <!-- arm_ee macro with the params
          * parent : where it is attached
@@ -17,6 +19,11 @@
          * *ee_offset : second block for the end-effector offset -->
   <xacro:macro name="arm_ee" params="parent arm is_right ee_macro ee_base_link use_prefix prefix controller *origin *ee_offset ">
-  <!-- KUKA arm -->
-    <xacro:kuka_lwr_arm name="${prefix}a_" reflect="${-1+2*is_right}" tool_name=""/>
+  <!-- PA10 arm -->
+    <xacro:if value="${is_right}" >
+      <xacro:call macro="pa10c_arm" name="${prefix}a_"/>
+    </xacro:if>
+    <xacro:unless value="${is_right}" >
+      <xacro:call macro="pa10a_arm" name="${prefix}a_"/>
+    </xacro:unless>
     <joint name="${prefix}a_frame_placement" type="fixed">
        <insert_block name="origin" />
@@ -26,5 +33,8 @@
     <xacro:if value="${controller}">
       <!-- add controllers -->
-      <xacro:right_lwr_arm_gazebo_controller namespace="${prefix}a" port="49940"/>
+       <!-- add controllers -->
+      <!-- pa10 controllers HERE
+      <xacro:pa10_gazebo_controller_manager namespace="${prefix}a"/> ros-hydro-gazebo-ros-control missing-->
+      <xacro:pa10_shadow_gazebo_controller_manager namespace="${prefix}a"/>
     </xacro:if>
     <xacro:if value="${use_prefix}">

File: agni_description/robots/platforms.urdf.xacro (robot description, xacro)
@@ -4,21 +4,57 @@
   <xacro:arg name="R" default="1"/>
   <xacro:arg name="L" default="1"/>
-  <xacro:arg name="R_EE" default="right_shadow_motor"/>
-  <xacro:arg name="L_EE" default="left_shadow_motor"/>
+  <xacro:arg name="R_EE_TYPE" default="shadow_motor"/>
+  <xacro:arg name="L_EE_TYPE" default="shadow_motor"/>
+  <xacro:arg name="R_EE_SIDE" default="right"/>
+  <xacro:arg name="L_EE_SIDE" default="left"/>
   <xacro:arg name="FLOBI" default="0"/>
+  <xacro:arg name="USE_PREFIX" default="true"/>
+  <!-- USE_PREFIX [true|false] to tell to use prefix for the end-effector or not.
+       Is mandatory if using two hands -->
+  <!-- ARM to select the arm type.
+       files called <ARM>.urdf.xacro and <ARM>_cal.xml should exist and provide
+       - offset of the base relatively to the <ARM>_frame
+       - arm_ee macro with the params
+         * parent : where it is attached
+         * arm : arm type
+         * is_right : 1 if arm is the right one
+         * ee_macro : name of the end-effector macro
+         * ee_base_link : name of the base_link of the end-effector to link to
+         * use_prefix : should we use prefix for the end-effector
+         * prefix : the prefix (for instance "r")
+         * controller : should the controllers be loaded or not
+         * *origin : first block for the base offset
+         * *ee_offset : second block for the end-effector offset -->
+  <!-- FLOBI to select if flobi should be added to the setup -->
+  <!-- R and L to select left or right or both arm and hand -->
+  <!-- R_EE_TYPE and L_EE_TYPE are the names of the end-effectors
+       mounted on right and left arms respectively -->
+  <!-- R_EE_SIDE and L_EE_SIDE are the variants of the end-effectors
+       for right and left arms respectively
+       Note a left hand can be mounted on the right arm
+       with R_EE_SIDE:=left -->
+  <!-- file called right_<R_EE_TYPE>_ee.urdf.xacro should exist and provide
+        - a macro called <R_EE_SIDE>_<R_EE_TYPE>
+        - a property r_ee_base_link with the name of the attachement link
+          for this end-effector type
+        - offset properties cal_right_ee_x|y|z|yaw|pitch|roll of the mounting
+          part of this effector when attached at the right arm
+       The same for left
+          -->
+  <!-- arm with end-effector -->
   <xacro:include filename="$(find agni_description)/robots/$(arg ARM)_anytool.urdf.xacro" />
-  <xacro:include filename="$(find agni_description)/$(arg ARM)/$(arg ARM).urdf.xacro" />
-  <xacro:include filename="$(find agni_description)/robots/$(arg R_EE)_ee.urdf.xacro" />
-  <xacro:include filename="$(find agni_description)/robots/$(arg L_EE)_ee.urdf.xacro" />
+  <!-- arm calibration -->
   <xacro:include filename="$(find agni_description)/calibration/$(arg ARM)_cal.xml"/>
-  <xacro:include filename="$(find agni_description)/urdf/frame-half.urdf.xacro"/>
-  <!--
-  <xacro:frame-half prefix="$(arg ARM)" thickness="${cal_frame_thick}" width="${cal_frame_width}" depth="${cal_frame_depth}"
-              height="${cal_frame_height}" tableHeight="${cal_frame_table_height}"/>
-  arm and hand -->
-    <xacro:frame-half prefix="kuka" thickness="0.09" width="1.92" depth="1.82"
-              height="1.26" tableHeight="1.00"/>
+  <!-- right end-effector -->
+  <xacro:include filename="$(find agni_description)/robots/right_$(arg R_EE_TYPE)_ee.urdf.xacro" />
+  <!-- left enf-effector -->
+  <xacro:include filename="$(find agni_description)/robots/left_$(arg L_EE_TYPE)_ee.urdf.xacro" />
+  <!-- frame -->
+  <xacro:include filename="$(find agni_description)/urdf/$(arg ARM)_frame.urdf.xacro"/>
+  <!-- frame generation -->
+  <xacro:call macro="$(arg ARM)_frame" prefix="$(arg ARM)" />
+  <!-- right arm with a right end-effector (can be of type left if needed, but must profide r_ee_base_link and cal_right_ee_x|y|z|yaw|pitch|roll) -->
   <xacro:if value="$(arg R)">
-    <xacro:arm_ee parent="$(arg ARM)_frame" arm="$(arg ARM)" prefix="r" is_right="1" ee_macro="$(arg R_EE)" ee_base_link="${r_ee_base_link}" use_prefix="$(arg USE_PREFIX)" controller="false">
+    <xacro:arm_ee parent="$(arg ARM)_frame" arm="$(arg ARM)" prefix="r" is_right="1" ee_macro="$(arg R_EE_SIDE)_$(arg R_EE_TYPE)" ee_base_link="${r_ee_base_link}" use_prefix="$(arg USE_PREFIX)" controller="false">
       <origin xyz="${cal_right_arm_x} ${cal_right_arm_y} ${cal_right_arm_z}"
       rpy="${cal_right_arm_roll} ${cal_right_arm_pitch} ${cal_right_arm_yaw}"/>
@@ -27,6 +63,7 @@
     </xacro:arm_ee>
   </xacro:if>
+  <!--left arm with a left end-effector (can be of type right if needed, but must profide l_ee_base_link and cal_left_ee_x|y|z|yaw|pitch|roll) -->
   <xacro:if value="$(arg L)">
-    <xacro:arm_ee parent="$(arg ARM)_frame" arm="$(arg ARM)" prefix="l" is_right="0" ee_macro="$(arg L_EE)" ee_base_link="${l_ee_base_link}" use_prefix="$(arg USE_PREFIX)" controller="false">
+    <xacro:arm_ee parent="$(arg ARM)_frame" arm="$(arg ARM)" prefix="l" is_right="0" ee_macro="$(arg L_EE_SIDE)_$(arg L_EE_TYPE)" ee_base_link="${l_ee_base_link}" use_prefix="$(arg USE_PREFIX)" controller="false">
       <origin xyz="${cal_left_arm_x} ${cal_left_arm_y} ${cal_left_arm_z}"
           rpy="${cal_left_arm_roll} ${cal_left_arm_pitch} ${cal_left_arm_yaw}"/>
@@ -35,4 +72,5 @@
     </xacro:arm_ee>
   </xacro:if>
+  <!-- flobi -->
   <xacro:if value="$(arg FLOBI)">
     <xacro:flobi prefix="" neutral="1" gender="0" parent="$(arg ARM)_frame" >

File: agni_description/robots/right_myrmex_ee.urdf.xacro (robot description, xacro)
@@ -1,5 +1,5 @@
 <?xml version="1.0"?>
 <robot xmlns:xacro="http://www.ros.org/wiki/xacro">
-  <xacro:include filename="$(find agni_description)/models/poking_stick.urdf.xacro" />
+  <xacro:include filename="$(find agni_description)/models/myrmex_quick_mount.urdf.xacro" />
   <xacro:property name="cal_right_ee_x" value="0.0" />
   <xacro:property name="cal_right_ee_y" value="0.0" />
@@ -8,10 +8,10 @@
   <xacro:property name="cal_right_ee_pitch" value="0.0" />
   <xacro:property name="cal_right_ee_roll" value="0.0" />
-  <xacro:property name="r_ee_base_link" value="poking_stick" />
-  <xacro:macro name="right_poking_stick" params="prefix" >
-    <xacro:poking_stick prefix="${prefix}" />
+  <xacro:property name="r_ee_base_link" value="myrmex_quick_mount" />
+  <xacro:macro name="right_myrmex" params="prefix" >
+    <xacro:myrmex_quick_mount prefix="${prefix}" />
   </xacro:macro>
-  <xacro:macro name="left_poking_stick" params="prefix" >
-    <xacro:poking_stick prefix="${prefix}" />
+  <xacro:macro name="left_myrmex" params="prefix" >
+    <xacro:myrmex_quick_mount prefix="${prefix}" />
   </xacro:macro>
 </robot>

File: agni_description/robots/right_shadow_muscle_ee.urdf.xacro (robot description, xacro)
@@ -7,5 +7,5 @@
   <xacro:property name="cal_right_ee_x" value="0.0" />
   <xacro:property name="cal_right_ee_y" value="0.0" />
-  <xacro:property name="cal_right_ee_z" value="0.0151" />
+  <xacro:property name="cal_right_ee_z" value="0.0" />
   <xacro:property name="cal_right_ee_yaw" value="0.0" />
   <xacro:property name="cal_right_ee_pitch" value="0.0" />

Commit message: Support for new tactile msgs in myrmex and hand wrapper

File: agni_description/models/myrmex_quick_mount.urdf.xacro (robot description, xacro)
@@ -32,11 +32,17 @@
   </xacro:macro>
   <xacro:macro name="myrmex_tactile_markers" params="parent topic *origin">
+    <xacro:property name="cell_size" value="0.005" />
+    <xacro:property name="myrmex_size" value="16" />
     <!-- tactile marker mapping description -->
-    <tactile topic="${topic}" data="data" xs="0 4095" link="${parent}">
-      <geometry>
-        <grid size="16 16" spacing="0.005 0.005"/>
-      </geometry>
+    <sensor name="myrmex_sensor" update_rate="100">
+      <parent link="${parent}"/>
       <xacro:insert_block name="origin"/>
-    </tactile>
+      <tactile>
+        <array rows="${myrmex_size}" cols="${myrmex_size}"
+            order="row-major" size="${cell_size} ${cell_size}"
+            offset="${cell_size * myrmex_size/2.0} ${cell_size * myrmex_size/2.0}">
+        </array>
+      </tactile>
+    </sensor>
   </xacro:macro>
 </robot>

File: agni_description/robots/shadow_hand.urdf.xacro (robot description, xacro)
@@ -26,6 +26,5 @@
     <!-- add tactile markers -->
     <xacro:shadowhand_tactile reflect="${1 if side=='right' else -1}"
-                              prefix="${'' if prefix=='' else prefix+'_'}"
-                              meshes="1" normals="1"/>
+                              prefix="${'' if prefix=='' else prefix+'_'}" />
     <xacro:shadow_gazebo_controller_manager namespace="${prefix}" />
   </xacro:macro>

Commit message: Added a contact plugin to myrmex

File: agni_description/models/myrmex_quick_mount.urdf.xacro (robot description, xacro)
@@ -24,10 +24,25 @@
       <collision>
         <origin xyz="0 0 0.03034" rpy="0 0 0"/>
-        <geometry>
+        <geometry name="${prefix}foam_collision_geom">
           <box size="0.095 0.095 0.006"/>
         </geometry>
       </collision>
     </link>
-    <gazebo reference="${prefix}myrmex_quick_mount"></gazebo>
+    <gazebo reference="${prefix}myrmex_quick_mount">
+      <sensor type="contact" name="${prefix}myrmex_contact">
+        <always_on>1</always_on>
+        <update_rate>1000.0</update_rate>
+        <contact>
+          <collision>${prefix}foam_collision</collision>
+          <topic>${prefix}foam_collision</topic>
+        </contact>
+        <plugin name="${prefix}myrmex_gazebo_ros_contact_controller" filename="libgazebo_ros_contact.so">
+          <alwaysOn>true</alwaysOn>
+          <frameName>${prefix}myrmex</frameName>
+          <updateRate>100.0</updateRate>
+          <bumperTopicName>contacts/${prefix}myrmex</bumperTopicName>
+        </plugin>
+      </sensor>
+    </gazebo>
   </xacro:macro>
   <xacro:macro name="myrmex_tactile_markers" params="parent topic *origin">

Commit message: Added intermediate prismatic link on myrmex (workaround due to gazebo bug generating bad collision name if links attached with fixed joints)

File: agni_description/models/myrmex_quick_mount.urdf.xacro (robot description, xacro)
@@ -3,4 +3,10 @@
   <xacro:macro name="myrmex_quick_mount" params="prefix:=''">
     <link name="${prefix}myrmex_quick_mount">
+       <inertial>
+        <origin xyz="0 0 0.03" rpy="0 0 0" />
+        <mass value="0.180" />
+        <inertia ixx="0.0002" ixy="0.0" ixz="0.0"
+        iyy="0.0002" iyz="0.0" izz="0.0001" />
+      </inertial>
       <visual>
         <origin xyz="0 0 0" rpy="0 0 0"/>
@@ -22,22 +28,44 @@
         </geometry>
       </collision>
-      <collision>
-        <origin xyz="0 0 0.03034" rpy="0 0 0"/>
-        <geometry name="${prefix}foam_collision_geom">
+    </link>
+    <joint name="${prefix}myrmex_bumper_joint" type="prismatic">
+      <parent link="${prefix}myrmex_quick_mount" />
+      <child link="${prefix}myrmex_foam" />
+      <origin xyz="0 0 0.03034" rpy="0 0 0"/>
+      <axis xyz="0 0 1" />
+       <limit lower="0.0" upper="0.001" effort="1" velocity="0.1" />
+    </joint>
+    <link name="${prefix}myrmex_foam">
+      <inertial>
+        <origin xyz="0 0 0.0" rpy="0 0 0" />
+        <mass value="0.005" />
+        <inertia ixx="0.000002" ixy="0.0" ixz="0.0"
+        iyy="0.000002" iyz="0.0" izz="0.000001" />
+      </inertial>
+      <visual>
+        <origin xyz="0 0 0" rpy="0 0 0"/>
+        <geometry>
+          <box size="0.095 0.095 0.006"/>
+        </geometry>
+      </visual>
+      <collision name="${prefix}myrmex_foam_collision">
+        <origin xyz="0 0 0" rpy="0 0 0"/>
+        <geometry>
           <box size="0.095 0.095 0.006"/>
         </geometry>
       </collision>
     </link>
-    <gazebo reference="${prefix}myrmex_quick_mount">
-      <sensor type="contact" name="${prefix}myrmex_contact">
+    <gazebo reference="${prefix}myrmex_foam">
+      <material>Gazebo/Black</material>
+      <sensor type="contact" name="${prefix}myrmex_foam_contact">
         <always_on>1</always_on>
         <update_rate>1000.0</update_rate>
         <contact>
-          <collision>${prefix}foam_collision</collision>
-          <topic>${prefix}foam_collision</topic>
+          <collision>${prefix}myrmex_foam_collision</collision>
+          <topic>${prefix}myrmex_foam_collision</topic>
         </contact>
         <plugin name="${prefix}myrmex_gazebo_ros_contact_controller" filename="libgazebo_ros_contact.so">
           <alwaysOn>true</alwaysOn>
-          <frameName>${prefix}myrmex</frameName>
+          <frameName>${prefix}myrmex_foam</frameName>
           <updateRate>100.0</updateRate>
           <bumperTopicName>contacts/${prefix}myrmex</bumperTopicName>

Commit message: Replaced foam collision box by collision mesh to improve contact accuracy

File: agni_description/models/myrmex_quick_mount.urdf.xacro (robot description, xacro)
@@ -52,5 +52,7 @@
         <origin xyz="0 0 0" rpy="0 0 0"/>
         <geometry>
-          <box size="0.095 0.095 0.006"/>
+          <mesh scale="1.0 1.0 1.0"
+                filename="package://agni_description/models/meshes/myrmex_foam.stl"/>
+          <!--box size="0.095 0.095 0.006"/-->
         </geometry>
       </collision>

File: agni_description/models/tactile_tool.urdf.xacro (robot description, xacro)
@@ -71,5 +71,7 @@
         <origin xyz="0 0 0" rpy="0 0 0"/>
         <geometry>
-          <box size="0.095 0.095 0.006"/>
+          <!--box size="0.095 0.095 0.006"/-->
+          <mesh scale="1.0 1.0 1.0"
+                filename="package://agni_description/models/meshes/myrmex_foam.stl"/>
         </geometry>
       </collision>

Commit message: Fixed collision naming of myrmex (gazebo adds _collision automatically now)

File: agni_description/models/myrmex_quick_mount.urdf.xacro (robot description, xacro)
@@ -49,5 +49,5 @@
         </geometry>
       </visual>
-      <collision name="${prefix}myrmex_foam_collision">
+      <collision name="${prefix}myrmex_foam">
         <origin xyz="0 0 0" rpy="0 0 0"/>
         <geometry>

File: agni_description/models/tactile_tool.urdf.xacro (robot description, xacro)
@@ -68,5 +68,5 @@
         </geometry>
       </visual>
-      <collision name="${prefix}myrmex_foam_collision">
+      <collision name="${prefix}myrmex_foam">
         <origin xyz="0 0 0" rpy="0 0 0"/>
         <geometry>
