Commit message: Fixed namings for consistency and added poking_stick end-effector Working base concept.

File: agni_description/models/poking_stick.urdf.xacro (robot description, xacro)
@@ -1,6 +1,6 @@
 <?xml version="1.0"?>
 <robot name="poking_stick" xmlns:xacro="http://www.ros.org/wiki/xacro">
-  <xacro:macro name="poking_stick" params="">
-  <link name="poking_stick">
+  <xacro:macro name="poking_stick" params="prefix">
+  <link name="${prefix}poking_stick">
     <visual>
       <origin xyz="0 0 0"
@@ -33,5 +33,5 @@
     </collision>
   </link>
-  <gazebo reference="poking_stick">
+  <gazebo reference="${prefix}poking_stick">
   </gazebo>
   </xacro:macro>

File: agni_description/robots/kuka_anytool.urdf.xacro (robot description, xacro)
@@ -17,5 +17,5 @@
       <xacro:if value="${use_prefix}">
         <!-- Effector -->
-        <xacro:call macro="${ee_macro}" prefix="${prefix}h_"/>
+        <xacro:call macro="${ee_macro}_ee" prefix="${prefix}h_"/>
         <!-- Link arm and effector -->
       <joint name="${prefix}a_arm_hand_mount" type="fixed">
@@ -27,5 +27,5 @@
     <xacro:unless value="${use_prefix}">
         <!-- Effector -->
-        <xacro:call macro="${ee_macro}" prefix=""/>
+        <xacro:call macro="${ee_macro}_ee" prefix=""/>
       <!-- Link arm and hand -->
       <joint name="${prefix}a_arm_hand_mount" type="fixed">

File: agni_description/robots/left_shadow_motor_ee.urdf.xacro (robot description, xacro)
@@ -12,5 +12,5 @@
   <xacro:property name="cal_left_ee_pitch" value="0.0" />
   <xacro:property name="cal_left_ee_roll" value="0.0" />
-  <xacro:macro name="left_shadow_motor" params="prefix">
+  <xacro:macro name="left_shadow_motor_ee" params="prefix">
     <xacro:shadowhand muscletrans="false" muscle="false" bio="false" ubi="$(arg USE_UBI)" eli="false" reflect="-1.0" prefix="${prefix}"  />
   </xacro:macro>

File: agni_description/robots/platforms.urdf.xacro (robot description, xacro)
@@ -1,6 +1,7 @@
 <?xml version="1.0"?>
-<robot name="$(arg ARM)_$(arg R_EE)_flobi"
-     xmlns:xacro="http://www.ros.org/wiki/xacro">
+<robot name="toto" xmlns:xacro="http://www.ros.org/wiki/xacro">
   <xacro:arg name="ARM" default="kuka"/>
+  <xacro:arg name="R" default="1"/>
+  <xacro:arg name="L" default="1"/>
   <xacro:arg name="R_EE" default="right_shadow_motor"/>
   <xacro:arg name="L_EE" default="left_shadow_motor"/>
@@ -16,4 +17,6 @@
               height="${cal_frame_height}" tableHeight="${cal_frame_table_height}"/>
   arm and hand -->
+    <xacro:frame-half prefix="kuka" thickness="0.09" width="1.92" depth="1.82"
+              height="1.26" tableHeight="1.00"/>
   <xacro:if value="$(arg R)">
     <xacro:arm_ee parent="$(arg ARM)_frame" arm="$(arg ARM)" prefix="r" is_right="1" ee_macro="$(arg R_EE)" ee_base_link="${r_ee_base_link}" use_prefix="$(arg USE_PREFIX)" controller="false">

File: agni_description/robots/right_shadow_motor_ee.urdf.xacro (robot description, xacro)
@@ -12,5 +12,5 @@
   <xacro:property name="cal_right_ee_pitch" value="0.0" />
   <xacro:property name="cal_right_ee_roll" value="0.0" />
-  <xacro:macro name="right_shadow_motor" params="prefix">
+  <xacro:macro name="right_shadow_motor_ee" params="prefix">
     <xacro:shadowhand muscletrans="false" muscle="false" bio="false" ubi="$(arg USE_UBI)" eli="false" reflect="1.0" prefix="${prefix}"  />
   </xacro:macro>

File: agni_description/urdf/frame-half.urdf.xacro (robot description, xacro)
@@ -6,5 +6,5 @@
 <xacro:include filename="$(find agni_description)/urdf/util.urdf.xacro"/>
 <xacro:include filename="$(find agni_description)/urdf/materials.urdf.xacro"/>
-<xacro:include filename="$(find agni_description)/calibration/default_cal.xml"/>
+<xacro:include filename="$(find agni_description)/calibration/kuka_cal.xml"/>
   <property name="cos30"     value="0.866025404" />
   <property name="sin30"     value="0.5" />

Commit message: Fixed platforms_setup.launch and platforms_urdf.xacro to work with other end-effectors without model Fixed poking stick and end-effector redefining same macro name, added dual hand robot_description

File: agni_description/models/poking_stick.urdf.xacro (robot description, xacro)
@@ -1,5 +1,5 @@
 <?xml version="1.0"?>
 <robot name="poking_stick" xmlns:xacro="http://www.ros.org/wiki/xacro">
-  <xacro:macro name="poking_stick" params="prefix tactile">
+  <xacro:macro name="poking_stick_generic" params="prefix tactile">
   <link name="${prefix}poking_stick">
     <visual>

File: agni_description/robots/platforms.urdf.xacro (robot description, xacro)
@@ -9,5 +9,5 @@
   <xacro:arg name="R_EE_TACTILE" default="-"/>
   <xacro:arg name="L_EE_TYPE" default="-"/>
-  <xacro:arg name="L_EE_MODEL" default=""/>
+  <xacro:arg name="L_EE_MODEL" default="-"/>
   <xacro:arg name="L_EE_SIDE" default="left"/>
   <xacro:arg name="L_EE_TACTILE" default="-"/>
@@ -75,6 +75,6 @@
      <!-- right end-effector -->
       <xacro:include filename="${agni_description_path}/robots/${r_ee_type}_ee.urdf.xacro" />
-      <xacro:include filename="${agni_description_path}/calibration/${r_ee_type}_${r_ee_model}_cal.xml"/>
-      <xacro:call macro="${r_ee_type}" model="$(arg R_EE_MODEL)" tactile="${r_ee_tactile if r_ee_tactile!='-' else ''}" side="${r_ee_side}" prefix="${r_ee_prefix}"/>
+      <xacro:include filename="${agni_description_path}/calibration/${r_ee_type}${('_'+r_ee_model) if r_ee_model!='-' else ''}_cal.xml"/>
+      <xacro:call macro="${r_ee_type}" model="${r_ee_model}" tactile="${r_ee_tactile if r_ee_tactile!='-' else ''}" side="${r_ee_side}" prefix="${r_ee_prefix}"/>
      <!-- Link arm and effector -->
       <joint name="ra_arm_hand_mount" type="fixed">
@@ -101,7 +101,7 @@
       <xacro:if value="${1 if (r_ee_type!=l_ee_type or r==0) else 0}">
         <xacro:include filename="${agni_description_path}/robots/${l_ee_type}_ee.urdf.xacro" />
-        <xacro:include filename="${agni_description_path}/calibration/${l_ee_type}_${l_ee_model}_cal.xml"/>
+        <xacro:include filename="${agni_description_path}/calibration/${l_ee_type}${('_'+l_ee_model) if l_ee_model!='-' else ''}_cal.xml"/>
       </xacro:if>
-      <xacro:call macro="${l_ee_type}" model="$(arg L_EE_MODEL)" tactile="${l_ee_tactile if l_ee_tactile!='-' else ''}" side="${l_ee_side}" prefix="${l_ee_prefix}"/>
+      <xacro:call macro="${l_ee_type}" model="${l_ee_model}" tactile="${l_ee_tactile if l_ee_tactile!='-' else ''}" side="${l_ee_side}" prefix="${l_ee_prefix}"/>
       <!-- Link arm and effector -->
       <joint name="la_arm_hand_mount" type="fixed">

File: agni_description/robots/poking_stick_ee.urdf.xacro (robot description, xacro)
@@ -11,5 +11,5 @@
   <xacro:macro name="poking_stick" params="model:='-' tactile:='-' side prefix:=rh" >
     <xacro:include filename="$(find agni_description)/models/poking_stick.urdf.xacro" />
-    <xacro:poking_stick prefix="${prefix}_" tactile="${tactile}" />
+    <xacro:poking_stick_generic prefix="${prefix}_" tactile="${tactile}" />
     <xacro:if value="${tactile!='-'}">
       <xacro:include filename="$(find sr_description)/hand/xacro/finger/distal/distal.tactile.xacro" />

Commit message: Added inertia to poking_stick and fixed masses of tools

File: agni_description/models/poking_stick.urdf.xacro (robot description, xacro)
@@ -3,4 +3,10 @@
   <xacro:macro name="poking_stick_generic" params="prefix tactile">
   <link name="${prefix}poking_stick">
+    <inertial>
+        <mass value="0.492" /> <!-- to get a total mass of the real assembly with distal of 505g -->
+        <origin xyz="0 0 0.092" />
+        <inertia ixx="0.000651" ixy="0.0" ixz="0.0"
+		 iyy="0.000651" iyz="0.0" izz="0.000896" />
+    </inertial>
     <visual>
       <origin xyz="0 0 0"

Commit message: Fixed pocking stick inertia according to real world values and better weighted average calculations

File: agni_description/models/poking_stick.urdf.xacro (robot description, xacro)
@@ -3,10 +3,20 @@
   <xacro:macro name="poking_stick_generic" params="prefix tactile">
   <link name="${prefix}poking_stick">
-    <inertial>
-        <mass value="0.492" /> <!-- to get a total mass of the real assembly with distal of 505g -->
-        <origin xyz="0 0 0.092" />
-        <inertia ixx="0.000651" ixy="0.0" ixz="0.0"
-		 iyy="0.000651" iyz="0.0" izz="0.000896" />
-    </inertial>
+    <xacro:if value="${'ubi' in tactile}">
+      <inertial>
+          <mass value="0.505" /> <!-- mass of metal + stick + ubi -->
+          <origin xyz="0 0 0.0161" /> <!-- from bottom of poking stick = mount flange -->
+          <inertia ixx="0.000651" ixy="0.0" ixz="0.0"
+       iyy="0.000651" iyz="0.0" izz="0.000896" />
+      </inertial>
+    </xacro:if>
+    <xacro:unless value="${'ubi' in tactile}">
+      <inertial>
+          <mass value="0.427" /> <!-- mass of metal + stick -->
+          <origin xyz="0 0 0.0124" /> <!-- from bottom of poking stick = mount flange -->
+          <inertia ixx="0.000651" ixy="0.0" ixz="0.0"
+       iyy="0.000651" iyz="0.0" izz="0.000896" />
+      </inertial>
+    </xacro:unless>
     <visual>
       <origin xyz="0 0 0"

Commit message: Added more collision cylinders to cover the roundish part of the poking stick

File: agni_description/models/poking_stick.urdf.xacro (robot description, xacro)
@@ -38,4 +38,18 @@
       <geometry>
         <cylinder radius="0.06725" length="0.015"/>
+      </geometry>
+    </collision>
+    <collision>
+      <origin xyz="0 0 ${0.005+0.015}"
+          rpy="0 0 0"/>
+      <geometry>
+        <cylinder radius="0.05" length="0.01"/>
+      </geometry>
+    </collision>
+    <collision>
+      <origin xyz="0 0 ${0.005+0.010+0.015}"
+          rpy="0 0 0"/>
+      <geometry>
+        <cylinder radius="0.025" length="0.01"/>
       </geometry>
     </collision>

Commit message: Added parameters for new sensor selection

File: agni_description/models/poking_stick.urdf.xacro (robot description, xacro)
@@ -1,7 +1,7 @@
 <?xml version="1.0"?>
 <robot name="poking_stick" xmlns:xacro="http://www.ros.org/wiki/xacro">
-  <xacro:macro name="poking_stick_generic" params="prefix tactile">
+  <xacro:macro name="poking_stick_generic" params="prefix tip_sensor">
   <link name="${prefix}poking_stick">
-    <xacro:if value="${'ubi' in tactile}">
+    <xacro:if value="${'ubi' in tip_sensor}">
       <inertial>
           <mass value="0.505" /> <!-- mass of metal + stick + ubi -->
@@ -11,5 +11,5 @@
       </inertial>
     </xacro:if>
-    <xacro:unless value="${'ubi' in tactile}">
+    <xacro:unless value="${'ubi' in tip_sensor}">
       <inertial>
           <mass value="0.427" /> <!-- mass of metal + stick -->
@@ -23,9 +23,9 @@
           rpy="0 0 0"/>
       <geometry>
-        <xacro:if value="${'ubi' in tactile}">
+        <xacro:if value="${'ubi' in tip_sensor}">
         <mesh scale="0.001 0.001 0.001"
 					 filename="package://agni_description/models/meshes/poking_stick_for_ubi.dae"/>
         </xacro:if>
-        <xacro:unless value="${'ubi' in tactile}">
+        <xacro:unless value="${'ubi' in tip_sensor}">
         <mesh scale="0.001 0.001 0.001"
 					 filename="package://agni_description/models/meshes/poking_stick.dae"/>
@@ -54,5 +54,5 @@
       </geometry>
     </collision>
-    <xacro:if value="${'ubi' in tactile}">
+    <xacro:if value="${'ubi' in tip_sensor}">
       <collision>
         <origin xyz="0 0 0.07375"
@@ -63,5 +63,5 @@
       </collision>
     </xacro:if>
-    <xacro:unless value="${'ubi' in tactile}">
+    <xacro:unless value="${'ubi' in tip_sensor}">
       <collision>
         <origin xyz="0 0 0.08875"
@@ -80,5 +80,5 @@
     </xacro:unless>
   </link>
-  <xacro:if value="${'ubi' in tactile}">
+  <xacro:if value="${'ubi' in tip_sensor}">
     <joint name="${prefix}stick_to_ubi" type="fixed">
       <origin xyz="0 0 0.13605" rpy="0 0 0"/>

File: agni_description/robots/poking_stick.urdf.xacro (robot description, xacro)
@@ -5,7 +5,7 @@
     <!-- poking stick -->
     <xacro:include filename="../models/poking_stick.urdf.xacro" />
-    <xacro:poking_stick_generic prefix="${prefix_}" tactile="${props['tactile']}"/>
-    <xacro:if value="${props['tactile'] in ['bio', 'ubi', 'eli']}">
-      <xacro:include filename="$(find sr_description)/hand/xacro/tactile.${props['tactile']}.xacro" />
+    <xacro:poking_stick_generic prefix="${prefix_}" tip_sensor="${props['tip_sensor']}"/>
+    <xacro:if value="${props['tip_sensor'] in ['bio', 'ubi', 'eli']}">
+      <xacro:include filename="$(find sr_description)/hand/xacro/tactile.${props['tip_sensor']}.xacro" />
       <!-- tactile marker mapping description -->
       <xacro:property name="prefix" value="${prefix_}"/>

File: agni_description/robots/poking_stick_ati.urdf.xacro (robot description, xacro)
@@ -8,7 +8,7 @@
     <!-- poking stick -->
     <xacro:include filename="../models/poking_stick.urdf.xacro" />
-    <xacro:poking_stick_generic prefix="${prefix_}" tactile="${props['tactile']}"/>
-    <xacro:if value="${props['tactile'] in ['bio', 'ubi', 'eli']}">
-      <xacro:include filename="$(find sr_description)/hand/xacro/tactile.${props['tactile']}.xacro" />
+    <xacro:poking_stick_generic prefix="${prefix_}" tip_sensor="${props['tip_sensor']}"/>
+    <xacro:if value="${props['tip_sensor'] in ['bio', 'ubi', 'eli']}">
+      <xacro:include filename="$(find sr_description)/hand/xacro/tactile.${props['tip_sensor']}.xacro" />
       <!-- tactile marker mapping description -->
       <xacro:property name="prefix" value="${prefix_}"/>

File: agni_description/robots/shadow_hand.urdf.xacro (robot description, xacro)
@@ -5,5 +5,8 @@
   <xacro:include filename="$(find sr_description)/hand/xacro/full_hand.tactile.xacro" />
   <xacro:macro name="shadow_hand" params="model:=${props.get('model','motor')}
-                                          tactile:=${props.get('tactile','ubi')}
+                                          tip_sensor:=${props.get('tip_sensor','ubi')}
+                                          mid_sensor:=${props.get('mid_sensor','ubi')}
+                                          prox_sensor:=${props.get('prox_sensor','ubi')}
+                                          palm_sensor:=${props.get('palm_sensor','ubi_fabric')}
                                           side:=${props.get('side','right')}
                                           prefix:=''
@@ -13,11 +16,10 @@
     <xacro:shadowhand muscletrans="${'trans' in model}"
                       muscle="${'muscle' in model}"
-                      bio="${'bio' in tactile}"
-                      bt_sp="${'bt_stp' in tactile}"
-                      ubi="${'ubi' in tactile}"
-                      eli="${'eli' in tactile}"
+                      tip_sensor="${tip_sensor}"
+                      mid_sensor="${mid_sensor}"
+                      prox_sensor="${prox_sensor}"
+                      palm_sensor="${palm_sensor}"
                       reflect="${1 if side=='right' else -1}"
-                      prefix="${prefix_}"
-                      lf="${lf}" />
+                      prefix="${prefix_}" />
     <!-- add tool frame -->
     <joint name="${prefix_}tool_frame" type="fixed">

File: agni_description/robots/shadow_hand_ati.urdf.xacro (robot description, xacro)
@@ -5,5 +5,8 @@
   <xacro:include filename="$(find sr_description)/hand/xacro/full_hand.tactile.xacro" />
   <xacro:macro name="shadow_hand" params="model:=${props.get('model','motor')}
-                                          tactile:=${props.get('tactile','ubi')}
+                                          tip_sensor:=${props.get('tip_sensor','ubi')}
+                                          mid_sensor:=${props.get('mid_sensor','ubi')}
+                                          prox_sensor:=${props.get('prox_sensor','ubi')}
+                                          palm_sensor:=${props.get('palm_sensor','ubi_fabric')}
                                           side:=${props.get('side','right')}
                                           prefix:=''
@@ -13,8 +16,8 @@
     <xacro:shadowhand muscletrans="${'trans' in model}"
                       muscle="${'muscle' in model}"
-                      bio="${'bio' in tactile}"
-                      bt_sp="${'bt_stp' in tactile}"
-                      ubi="${'ubi' in tactile}"
-                      eli="${'eli' in tactile}"
+                      tip_sensor="${tip_sensor}"
+                      mid_sensor="${mid_sensor}"
+                      prox_sensor="${prox_sensor}"
+                      palm_sensor="${palm_sensor}"
                       reflect="${1 if side=='right' else -1}"
                       prefix="${prefix_}"
