Commit message: More specific variable tests
Using `'text' in variable` is a rather sloppy equivalence check.

File: agni_description/models/poking_stick.urdf.xacro (robot description, xacro)
@@ -3,5 +3,5 @@
   <xacro:macro name="poking_stick_generic" params="prefix tip_sensor">
   <link name="${prefix}poking_stick">
-    <xacro:if value="${'ubi' in tip_sensor}">
+    <xacro:if value="${tip_sensor == 'ubi'}">
       <inertial>
           <mass value="0.505" /> <!-- mass of metal + stick + ubi -->
@@ -11,5 +11,5 @@
       </inertial>
     </xacro:if>
-    <xacro:unless value="${'ubi' in tip_sensor}">
+    <xacro:unless value="${tip_sensor == 'ubi'}">
       <inertial>
           <mass value="0.427" /> <!-- mass of metal + stick -->
@@ -23,9 +23,9 @@
           rpy="0 0 0"/>
       <geometry>
-        <xacro:if value="${'ubi' in tip_sensor}">
+        <xacro:if value="${tip_sensor == 'ubi'}">
         <mesh scale="0.001 0.001 0.001"
 					 filename="package://agni_description/models/meshes/poking_stick_for_ubi.dae"/>
         </xacro:if>
-        <xacro:unless value="${'ubi' in tip_sensor}">
+        <xacro:unless value="${tip_sensor == 'ubi'}">
         <mesh scale="0.001 0.001 0.001"
 					 filename="package://agni_description/models/meshes/poking_stick.dae"/>
@@ -54,5 +54,5 @@
       </geometry>
     </collision>
-    <xacro:if value="${'ubi' in tip_sensor}">
+    <xacro:if value="${tip_sensor == 'ubi'}">
       <collision>
         <origin xyz="0 0 0.07375"
@@ -63,5 +63,5 @@
       </collision>
     </xacro:if>
-    <xacro:unless value="${'ubi' in tip_sensor}">
+    <xacro:unless value="${tip_sensor == 'ubi'}">
       <collision>
         <origin xyz="0 0 0.08875"
@@ -80,5 +80,5 @@
     </xacro:unless>
   </link>
-  <xacro:if value="${'ubi' in tip_sensor}">
+  <xacro:if value="${tip_sensor == 'ubi'}">
     <joint name="${prefix}stick_to_ubi" type="fixed">
       <origin xyz="0 0 0.13605" rpy="0 0 0"/>

File: agni_description/robots/bimanual.urdf.xacro (robot description, xacro)
@@ -1,5 +1,5 @@
 <?xml version="1.0"?>
 <robot name="bimanual" xmlns:xacro="http://www.ros.org/wiki/xacro">
-	<xacro:property name="settings" value="${load_yaml('robots.yaml')}" />
+	<xacro:property name="settings" value="${xacro.load_yaml('robots.yaml')}" />
 	<xacro:arg name="FRAME" default="-"/>
 	<xacro:arg name="ARM_L" default="-"/>

File: agni_description/robots/famula.urdf.xacro (robot description, xacro)
@@ -1,5 +1,5 @@
 <?xml version="1.0"?>
 <robot name="arm_hand_shadow" xmlns:xacro="http://www.ros.org/wiki/xacro">
-	<xacro:property name="settings" value="${load_yaml('robots.yaml')}" />
+	<xacro:property name="settings" value="${xacro.load_yaml('robots.yaml')}" />
 	<xacro:arg name="SIM" default="1"/>
 	<xacro:arg name="CALIB" default="famula"/>

File: agni_description/robots/moveable_famula.urdf.xacro (robot description, xacro)
@@ -1,5 +1,5 @@
 <?xml version="1.0"?>
 <robot name="arm_hand_shadow" xmlns:xacro="http://www.ros.org/wiki/xacro">
-	<xacro:property name="settings" value="${load_yaml('robots.yaml')}" />
+	<xacro:property name="settings" value="${xacro.load_yaml('robots.yaml')}" />
 	<xacro:arg name="SIM" default="1"/>
 	<xacro:arg name="CALIB" default="moveable_famula"/>

File: agni_description/robots/poking_stick.urdf.xacro (robot description, xacro)
@@ -12,5 +12,5 @@
       <xacro:property name="xs" value="1023 0"/>
       <xacro:property name="taxel_dir" value="$(find sr_description)/hand/xacro/finger"/>
-      <xacro:distal_tactile finger="ff" taxel_data="${load_yaml(taxel_dir + '/distal/distal.taxels.ubi.yaml')}"/>
+      <xacro:distal_tactile finger="ff" taxel_data="${xacro.load_yaml(taxel_dir + '/distal/distal.taxels.ubi.yaml')}" />
     </xacro:if>
   </xacro:macro>

File: agni_description/robots/poking_stick_ati.urdf.xacro (robot description, xacro)
@@ -15,5 +15,5 @@
       <xacro:property name="xs" value="1023 0"/>
       <xacro:property name="taxel_dir" value="$(find sr_description)/hand/xacro/finger"/>
-      <xacro:distal_tactile finger="ff" taxel_data="${load_yaml(taxel_dir + '/distal/distal.taxels.ubi.yaml')}"/>
+      <xacro:distal_tactile finger="ff" taxel_data="${xacro.load_yaml(taxel_dir + '/distal/distal.taxels.ubi.yaml')}" />
     </xacro:if>
   </xacro:macro>

File: agni_description/robots/sfb.urdf.xacro (robot description, xacro)
@@ -1,5 +1,5 @@
 <?xml version="1.0"?>
 <robot name="arm_hand_shadow" xmlns:xacro="http://www.ros.org/wiki/xacro">
-	<xacro:property name="settings" value="${load_yaml('robots.yaml')}" />
+	<xacro:property name="settings" value="${xacro.load_yaml('robots.yaml')}" />
 	<xacro:arg name="SIM" default="1"/>
 	<xacro:arg name="CALIB" default="sfb"/>

File: agni_description/robots/shadow_hand.urdf.xacro (robot description, xacro)
@@ -5,7 +5,7 @@
   <xacro:include filename="$(find sr_description)/hand/xacro/full_hand.tactile.xacro" />
   <xacro:macro name="shadow_hand" params="model:=${props.get('model','motor')}
-                                          tip_sensors:=${props.get('tip_sensor',['ubi','ubi','ubi','ubi','ubi'])}
-                                          mid_sensors:=${props.get('mid_sensor',['ubi','ubi','ubi','ubi','ubi'])}
-                                          prox_sensors:=${props.get('prox_sensor',['ubi','ubi','ubi','ubi','ubi'])}
+                                          tip_sensors:=${props.get('tip_sensor','ubi')}
+                                          mid_sensors:=${props.get('mid_sensor','ubi')}
+                                          prox_sensors:=${props.get('prox_sensor','ubi')}
                                           palm_sensor:=${props.get('palm_sensor','ubi_fabric')}
                                           side:=${props.get('side','right')}

File: agni_description/robots/shadow_hand_ati.urdf.xacro (robot description, xacro)
@@ -5,7 +5,7 @@
   <xacro:include filename="$(find sr_description)/hand/xacro/full_hand.tactile.xacro" />
   <xacro:macro name="shadow_hand" params="model:=${props.get('model','motor')}
-                                          tip_sensors:=${props.get('tip_sensor',['ubi','ubi','ubi','ubi','ubi'])}
-                                          mid_sensors:=${props.get('mid_sensor',['ubi','ubi','ubi','ubi','ubi'])}
-                                          prox_sensors:=${props.get('prox_sensor',['ubi','ubi','ubi','ubi','ubi'])}
+                                          tip_sensors:=${props.get('tip_sensor','ubi')}
+                                          mid_sensors:=${props.get('mid_sensor','ubi')}
+                                          prox_sensors:=${props.get('prox_sensor','ubi')}
                                           palm_sensor:=${props.get('palm_sensor','ubi_fabric')}
                                           side:=${props.get('side','right')}

File: agni_description/robots/single.urdf.xacro (robot description, xacro)
@@ -1,5 +1,5 @@
 <?xml version="1.0"?>
 <robot name="single" xmlns:xacro="http://www.ros.org/wiki/xacro">
-	<xacro:property name="settings" value="${load_yaml('robots.yaml')}" />
+	<xacro:property name="settings" value="${xacro.load_yaml('robots.yaml')}" />
 	<xacro:arg name="FRAME" default="-"/>
 	<xacro:arg name="ARM" default="-"/>

File: agni_description/urdf/camera.urdf.xacro (robot description, xacro)
@@ -5,5 +5,5 @@
   <xacro:macro name="camera_body" params="parent name fps hfov width height cx:=0 cy:=0 hfov2:=- width2:=- height2:=- cx2:=- cy2:=-
                                           has_depth *origin has_second_origin:=0 *second_origin">
-    <xacro:if value="${1 if 'world' in parent else 0}">
+    <xacro:if value="${1 if parent == 'world' else 0}">
       <link name="${parent}" />
     </xacro:if>
