Commit message: Formatting

File: agni_description/models/calibration_tool.urdf.xacro (robot description, xacro)
@@ -4,6 +4,5 @@
   <link name="${prefix}calibration_tool">
     <visual>
-      <origin xyz="0 0 0"
-          rpy="0 0 0"/>
+      <origin xyz="0 0 0" rpy="0 0 0" />
       <geometry>
         <mesh scale="0.001 0.001 0.001"
@@ -12,6 +11,5 @@
     </visual>
       <collision>
-        <origin xyz="0 0 0.0"
-            rpy="0 0 0"/>
+        <origin xyz="0 0 0.0" rpy="0 0 0" />
         <geometry>
           <mesh scale="0.001 0.001 0.001"

File: agni_description/models/poking_stick.urdf.xacro (robot description, xacro)
@@ -20,6 +20,5 @@
     </xacro:unless>
     <visual>
-      <origin xyz="0 0 0"
-          rpy="0 0 0"/>
+      <origin xyz="0 0 0" rpy="0 0 0" />
       <geometry>
         <xacro:if value="${tip_sensor == 'ubi'}">
@@ -34,6 +33,5 @@
     </visual>
     <collision>
-      <origin xyz="0 0 0.0075"
-          rpy="0 0 0"/>
+      <origin xyz="0 0 0.0075" rpy="0 0 0" />
       <geometry>
         <cylinder radius="0.06725" length="0.015"/>
@@ -41,6 +39,5 @@
     </collision>
     <collision>
-      <origin xyz="0 0 ${0.005+0.015}"
-          rpy="0 0 0"/>
+      <origin xyz="0 0 ${0.005+0.015}" rpy="0 0 0" />
       <geometry>
         <cylinder radius="0.05" length="0.01"/>
@@ -48,6 +45,5 @@
     </collision>
     <collision>
-      <origin xyz="0 0 ${0.005+0.010+0.015}"
-          rpy="0 0 0"/>
+      <origin xyz="0 0 ${0.005+0.010+0.015}" rpy="0 0 0" />
       <geometry>
         <cylinder radius="0.025" length="0.01"/>
@@ -56,6 +52,5 @@
     <xacro:if value="${tip_sensor == 'ubi'}">
       <collision>
-        <origin xyz="0 0 0.07375"
-            rpy="0 0 0"/>
+        <origin xyz="0 0 0.07375" rpy="0 0 0" />
         <geometry>
           <cylinder radius="0.0075" length="0.1445"/>
@@ -65,6 +60,5 @@
     <xacro:unless value="${tip_sensor == 'ubi'}">
       <collision>
-        <origin xyz="0 0 0.08875"
-            rpy="0 0 0"/>
+        <origin xyz="0 0 0.08875" rpy="0 0 0" />
         <geometry>
           <cylinder radius="0.0075" length="0.1475"/>
@@ -72,6 +66,5 @@
       </collision>
       <collision>
-        <origin xyz="0 0 0.1625"
-            rpy="0 0 0"/>
+        <origin xyz="0 0 0.1625" rpy="0 0 0" />
         <geometry>
           <sphere radius="0.0075"/>
@@ -88,6 +81,5 @@
     <link name="${prefix}ffdistal">
       <visual>
-        <origin xyz="0 0 0"
-            rpy="0 0 0"/>
+        <origin xyz="0 0 0" rpy="0 0 0" />
         <geometry>
           <mesh scale="0.001 0.001 0.001"
@@ -96,6 +88,5 @@
       </visual>
       <collision>
-        <origin xyz="0 0 0"
-            rpy="0 0 0"/>
+        <origin xyz="0 0 0" rpy="0 0 0" />
         <geometry>
           <mesh scale="0.001 0.001 0.001"
