Commit message: Added support for versions of tools with ATI sensor

File: agni_moveit_config/agni_generic_moveit_config/config/generic_bimanual_platform.srdf.xacro (robot description, xacro)
@@ -102,4 +102,9 @@
         <xacro:call macro="shadow_motor_joints" prefix="rh" />
       </xacro:if>
+      <xacro:if value="${TOOL_R == 'shadow_motor_right_ati'}" >
+        <link name="rh_ft_sensor_link" />
+        <joint name="rh_ft_tool_fixed_joint" />
+        <xacro:call macro="shadow_motor_joints" prefix="rh" />
+      </xacro:if>
       <!-- schunk hand -->
       <xacro:if value="${TOOL_R == 'schunk_hand_left'}" >
@@ -118,6 +123,13 @@
         <link name="rh_poking_stick" />
       </xacro:if>
+      <xacro:if value="${TOOL_R == 'poking_stick_rigid_ati'}" >
+        <link name="rh_ft_sensor_link" />
+        <link name="rh_poking_stick" />
+      </xacro:if>
       <xacro:if value="${TOOL_R == 'poking_stick_ubi'}" >
          <chain base_link="rh_poking_stick" tip_link="rh_ffdistal" />
+      </xacro:if>
+      <xacro:if value="${TOOL_R == 'poking_stick_ubi_ati'}" >
+         <chain base_link="rh_ft_sensor_link" tip_link="rh_ffdistal" />
       </xacro:if>
     </group>
@@ -133,4 +145,9 @@
         <xacro:call macro="shadow_motor_joints" prefix="rh" />
       </xacro:if>
+      <xacro:if value="${TOOL_L == 'shadow_motor_right_ati'}" >
+        <link name="rh_ft_sensor_link" />
+        <joint name="rh_ft_tool_fixed_joint" />
+        <xacro:call macro="shadow_motor_joints" prefix="rh" />
+      </xacro:if>
       <!-- schunk hand -->
       <xacro:if value="${TOOL_L == 'schunk_hand_left'}" >
@@ -149,6 +166,13 @@
           <link name="lh_poking_stick" />
       </xacro:if>
+      <xacro:if value="${TOOL_L == 'poking_stick_rigid_ati'}" >
+        <link name="lh_ft_sensor_link" />
+        <link name="lh_poking_stick" />
+      </xacro:if>
       <xacro:if value="${TOOL_L == 'poking_stick_ubi'}" >
          <chain base_link="lh_poking_stick" tip_link="lh_ffdistal" />
+      </xacro:if>
+      <xacro:if value="${TOOL_L == 'poking_stick_ubi_ati'}" >
+         <chain base_link="lh_ft_sensor_link" tip_link="lh_ffdistal" />
       </xacro:if>
     </group>

Commit message: Added link names explicitely in generic srdf (chain apparently skips fixed links when extracted)

File: agni_moveit_config/agni_generic_moveit_config/config/generic_bimanual_platform.srdf.xacro (robot description, xacro)
@@ -134,7 +134,12 @@
       </xacro:if>
       <xacro:if value="${TOOL_R == 'poking_stick_ubi'}" >
+         <link name="rh_poking_stick" />
+         <link name="rh_ffdistal" />
          <chain base_link="rh_poking_stick" tip_link="rh_ffdistal" />
       </xacro:if>
       <xacro:if value="${TOOL_R == 'poking_stick_ubi_ati'}" >
+         <link name="rh_ft_sensor_link" />
+         <link name="rh_poking_stick" />
+         <link name="rh_ffdistal" />
          <chain base_link="rh_ft_sensor_link" tip_link="rh_ffdistal" />
       </xacro:if>
@@ -183,7 +188,12 @@
       </xacro:if>
       <xacro:if value="${TOOL_L == 'poking_stick_ubi'}" >
+         <link name="lh_poking_stick" />
+         <link name="lh_ffdistal" />
          <chain base_link="lh_poking_stick" tip_link="lh_ffdistal" />
       </xacro:if>
       <xacro:if value="${TOOL_L == 'poking_stick_ubi_ati'}" >
+         <link name="lh_ft_sensor_link" />
+         <link name="lh_poking_stick" />
+         <link name="lh_ffdistal" />
          <chain base_link="lh_ft_sensor_link" tip_link="lh_ffdistal" />
       </xacro:if>

Commit message: Added support for schunk + ati

File: agni_moveit_config/agni_generic_moveit_config/config/generic_bimanual_platform.srdf.xacro (robot description, xacro)
@@ -120,4 +120,14 @@
         <xacro:call macro="schunk_hand_joints" prefix="rh" />
       </xacro:if>
+      <xacro:if value="${TOOL_R == 'schunk_hand_left_ati'}" >
+        <link name="lh_ft_sensor_link" />
+        <joint name="lh_ft_tool_fixed_joint" />
+        <xacro:call macro="schunk_hand_joints" prefix="lh" />
+      </xacro:if>
+      <xacro:if value="${TOOL_R == 'schunk_hand_right_ati'}" >
+        <link name="rh_ft_sensor_link" />
+        <joint name="rh_ft_tool_fixed_joint" />
+        <xacro:call macro="schunk_hand_joints" prefix="rh" />
+      </xacro:if>
       <!-- myrmex -->
       <xacro:if value="${TOOL_R == 'myrmex'}" >
@@ -172,4 +182,14 @@
       </xacro:if>
       <xacro:if value="${TOOL_L == 'schunk_hand_right'}" >
+        <xacro:call macro="schunk_hand_joints" prefix="rh" />
+      </xacro:if>
+      <xacro:if value="${TOOL_L == 'schunk_hand_left_ati'}" >
+        <link name="lh_ft_sensor_link" />
+        <joint name="lh_ft_tool_fixed_joint" />
+        <xacro:call macro="schunk_hand_joints" prefix="lh" />
+      </xacro:if>
+      <xacro:if value="${TOOL_L == 'schunk_hand_right_ati'}" >
+        <link name="rh_ft_sensor_link" />
+        <joint name="rh_ft_tool_fixed_joint" />
         <xacro:call macro="schunk_hand_joints" prefix="rh" />
       </xacro:if>
