Commit message: Added placement possibilities to myrmex_description

File: myrmex_description/robots/myrmex_board.urdf.xacro (robot description, xacro)
@@ -4,8 +4,10 @@
    <xacro:arg name="board_row_nb" default="3"/>
    <xacro:arg name="board_col_nb" default="3"/>
+   <xacro:arg name="pos_xyz" default="0 0 0"/>
+   <xacro:arg name="ori_rpy" default="0 0 0"/>
   <joint name="board_base_joint" type="fixed">
       <parent link="world" />
       <child link="board_base" />
-      <origin xyz="0 0 0" rpy="0 0 0"/>
+      <origin xyz="$(arg pos_xyz)" rpy="$(arg ori_rpy)"/>
   </joint>
    <link name="board_base">

Commit message: Fixed myrmex standalone to handle namespaces

File: myrmex_description/robots/myrmex_board.urdf.xacro (robot description, xacro)
@@ -6,4 +6,5 @@
    <xacro:arg name="pos_xyz" default="0 0 0"/>
    <xacro:arg name="ori_rpy" default="0 0 0"/>
+   <xacro:arg name="ns" default=""/>
   <joint name="board_base_joint" type="fixed">
       <parent link="world" />
@@ -34,7 +35,9 @@
     </link>
    <xacro:include filename="$(find myrmex_description)/models/myrmex_tactile_surface.urdf.xacro" />
-   <xacro:myrmex_tactile_surface prefix="" parent="board_base" size_x="$(arg board_row_nb)" size_y="$(arg board_col_nb)"
+   <xacro:myrmex_tactile_surface prefix="$(arg ns)" parent="board_base" size_x="$(arg board_row_nb)" size_y="$(arg board_col_nb)"
                                  foam_size_x="0.08" foam_size_y="0.08" />
-   <xacro:myrmex_tactile_markers parent="world" prefix="" channel="myrmex_sensor" size_x="$(arg board_row_nb)" size_y="$(arg board_col_nb)">
+   <xacro:property name="ns" value="$(arg ns)" />
+   <xacro:property name="prefix_" value="${ns + '_' if ns else ''}" />
+   <xacro:myrmex_tactile_markers parent="${prefix_}myrmex_foam" prefix="$(arg ns)" channel="myrmex_sensor" size_x="$(arg board_row_nb)" size_y="$(arg board_col_nb)">
       <origin xyz="0 0 0.001" rpy="0 0 0"/>
    </xacro:myrmex_tactile_markers>
