Commit message: Fixed myrmex orientation and rviz description

File: myrmex_description/robots/myrmex_2d_rig.urdf.xacro (robot description, xacro)
@@ -109,5 +109,5 @@
       <parent link="rig_hand" />
       <child link="rig_myrmex_quick_mount" />
-      <origin xyz="${-hand_len} 0 ${-hand_z_offset+0.03034}" rpy="0 ${-pi} 0"/>
+      <origin xyz="${-hand_len} 0 ${-hand_z_offset+0.03034}" rpy="0 ${-pi} ${pi/2.0}"/>
   </joint>
   <xacro:myrmex_quick_mount prefix="rig"/>
