Commit message: Updated myrmex to handle foam size and fixed myrmex board

File: myrmex_description/models/myrmex_tactile_surface.urdf.xacro (robot description, xacro)
@@ -1,5 +1,5 @@
 <?xml version="1.0"?>
 <robot name="myrmex_quick_mount" xmlns:xacro="http://www.ros.org/wiki/xacro">
-  <xacro:macro name="myrmex_tactile_surface" params="prefix:='' parent size_x:=1 size_y:=1">
+  <xacro:macro name="myrmex_tactile_surface" params="prefix:='' parent size_x:=1 size_y:=1 foam_size_x:=0.095 foam_size_y:=0.095 ">
     <xacro:property name="prefix_" value="${prefix + '_' if prefix else ''}" />
     <joint name="${prefix_}myrmex_bumper_joint" type="prismatic">
@@ -21,9 +21,11 @@
         <geometry>
           <xacro:if value="${1 if (size_x==1 and size_y==1) else 0}" >
-          <mesh scale="1.0 1.0 1.0"
+            <xacro:property name="scale_x" value="${foam_size_x/0.095}" />
+            <xacro:property name="scale_y" value="${foam_size_y/0.095}" />
+            <mesh scale="${scale_x} ${scale_y} 1.0"
                 filename="package://myrmex_description/models/meshes/myrmex_foam.stl"/>
           </xacro:if>
           <xacro:unless value="${1 if (size_x==1 and size_y==1) else 0}" >
-            <box size="${0.095*size_x} ${0.095*size_y} 0.006"/>
+            <box size="${foam_size_x*size_x} ${foam_size_y*size_y} 0.006"/>
           </xacro:unless>
         </geometry>
@@ -32,5 +34,5 @@
         <origin xyz="0 0 0" rpy="0 0 0"/>
         <geometry>
-          <box size="${0.095*size_x} ${0.095*size_y} 0.006"/>
+          <box size="${foam_size_x*size_x} ${foam_size_y*size_y} 0.006"/>
         </geometry>
       </collision>

File: myrmex_description/robots/myrmex_board.urdf.xacro (robot description, xacro)
@@ -4,6 +4,34 @@
    <xacro:arg name="board_row_nb" default="3"/>
    <xacro:arg name="board_col_nb" default="3"/>
+  <joint name="board_base_joint" type="fixed">
+      <parent link="world" />
+      <child link="board_base" />
+      <origin xyz="0 0 0" rpy="0 0 0"/>
+  </joint>
+   <link name="board_base">
+       <inertial>
+        <origin xyz="0 0 0.015" rpy="0 0 0" />
+        <mass value="0.400" />
+        <inertia ixx="0.0002" ixy="0.0" ixz="0.0"
+        iyy="0.0002" iyz="0.0" izz="0.0001" />
+      </inertial>
+      <xacro:property name="board_row_nb" value="$(arg board_row_nb)" />
+      <xacro:property name="board_col_nb" value="$(arg board_col_nb)" />
+      <visual>
+        <origin xyz="0.05 0 0.015" rpy="0 0 0"/>
+        <geometry>
+          <box size="${0.1 + board_row_nb*0.08} ${board_col_nb*0.08} 0.03"/>
+        </geometry>
+      </visual>
+      <collision>
+        <origin xyz="0.05 0 0.015" rpy="0 0 0"/>
+        <geometry>
+          <box size="${0.1 + board_row_nb*0.08} ${board_col_nb*0.08} 0.03"/>
+        </geometry>
+      </collision>
+    </link>
    <xacro:include filename="$(find myrmex_description)/models/myrmex_tactile_surface.urdf.xacro" />
-   <xacro:myrmex_tactile_surface prefix="" parent="world" size_x="$(arg board_row_nb)" size_y="$(arg board_col_nb)"/>
+   <xacro:myrmex_tactile_surface prefix="" parent="board_base" size_x="$(arg board_row_nb)" size_y="$(arg board_col_nb)"
+                                 foam_size_x="0.08" foam_size_y="0.08" />
    <xacro:myrmex_tactile_markers parent="world" prefix="" channel="myrmex_sensor" size_x="$(arg board_row_nb)" size_y="$(arg board_col_nb)">
       <origin xyz="0 0 0.001" rpy="0 0 0"/>

Commit message: Added possibility to name myrmex tactile sensors

File: myrmex_description/models/myrmex_tactile_surface.urdf.xacro (robot description, xacro)
@@ -58,5 +58,5 @@
     </gazebo>
   </xacro:macro>
-  <xacro:macro name="myrmex_tactile_markers" params="parent channel prefix:='' size_x:=1 size_y:=1 *origin">
+  <xacro:macro name="myrmex_tactile_markers" params="parent channel name:='myrmex_sensor' prefix:='' size_x:=1 size_y:=1 *origin">
     <xacro:property name="cell_size" value="0.005" />
     <xacro:property name="cell_spacing" value="0.005" />
@@ -65,5 +65,5 @@
     <xacro:property name="prefix_" value="${prefix + '_' if prefix else ''}" />
     <!-- tactile marker mapping description -->
-    <sensor name="${prefix_}myrmex_sensor" update_rate="100">
+    <sensor name="${prefix_}${name}" update_rate="100">
       <parent link="${parent}"/>
       <xacro:insert_block name="origin"/>
